Commit message: Address PR comments

File: irobot_create_description/urdf/bumper.xacro (robot description, xacro)
@@ -1,7 +1,7 @@
 <?xml version="1.0"?>
 <robot xmlns:xacro="http://ros.org/wiki/xacro">
-<xacro:macro name="simple_bumper" params="name:=bumper parent_link robot_type visual_mesh collision_mesh
+<xacro:macro name="bumper" params="name:=bumper parent_link robot_type visual_mesh collision_mesh
                                           *origin *inertial">
-  <joint name="${name}_joint" type="prismatic">
+  <joint name="${name}_joint" type="fixed">
     <parent link="${parent_link}"/>
     <child link="${name}_link"/>
@@ -23,5 +23,5 @@
     <xacro:insert_block name="inertial"/>
   </link>
-  <gazebo reference="bumper_link" >
+  <gazebo reference="${name}_link" >
     <mu1>0.1</mu1>
     <mu2>0.1</mu2>
@@ -30,11 +30,7 @@
     <maxContacts>10</maxContacts>
     <material>Gazebo/Green</material>
-    <sensor name='${name}_contact_sensor' type='contact'>
-      <always_on>true</always_on>
-      <update_rate>40</update_rate>
-      <contact>
-        <collision>${name}_link_collision</collision>
-      </contact>
-    </sensor>
+  </gazebo>
+  <gazebo reference="${name}_joint">
+    <preserveFixedJoint>true</preserveFixedJoint>
   </gazebo>
 </xacro:macro>

File: irobot_create_description/urdf/wheel.xacro (robot description, xacro)
@@ -22,5 +22,5 @@
       </geometry>
     </collision>
-    <xacro:inertial_cilinder mass="${wheel_mass}" radius="${wheel_radius}" length="${wheel_width}" />
+    <xacro:inertial_cylinder mass="${wheel_mass}" radius="${wheel_radius}" length="${wheel_width}" />
   </link>
   <gazebo reference="wheel_${name}_link">
