Commit message: Updated wheels and caster colors

File: irobot_create_description/urdf/caster.urdf.xacro (robot description, xacro)
@@ -20,4 +20,7 @@
     </collision>
   </link>
+  <gazebo reference="${name}_link">
+    <material>Gazebo/Grey</material>
+  </gazebo>
 </xacro:macro>
 </robot>

File: irobot_create_description/urdf/wheel.urdf.xacro (robot description, xacro)
@@ -32,4 +32,5 @@
     <minDepth>0.0001</minDepth>
     <maxVel>1.0</maxVel>
+    <material>Gazebo/Grey</material>
   </gazebo>
 </xacro:macro>

Commit message: Update robot models (#11)
* WIP: update robot meshes

* WIP: Improved collision and inertias

* Removed unnecessary wheel models

* Updated wheels and caster colors

* Updated colors for models in gazebo

File: irobot_create_description/urdf/caster.urdf.xacro (robot description, xacro)
@@ -20,4 +20,7 @@
     </collision>
   </link>
+  <gazebo reference="${name}_link">
+    <material>Gazebo/DarkGrey</material>
+  </gazebo>
 </xacro:macro>
 </robot>

File: irobot_create_description/urdf/create3.urdf.xacro (robot description, xacro)
@@ -7,7 +7,8 @@
   <!-- MECHANICAL PROPERTIES -->
   <xacro:property name="body_z_offset_cm"           value="-2.5" />
+  <xacro:property name="body_collision_z_offset_cm" value="-1" />
   <xacro:property name="body_mass_kg"               value="2.300" />
-  <xacro:property name="body_radius_cm"             value="16" />
-  <xacro:property name="body_length_cm"             value="4.8" />
+  <xacro:property name="body_radius_cm"             value="16.4" />
+  <xacro:property name="body_length_cm"             value="6" />
   <xacro:property name="bumper_mass_kg"             value="0.1" />
   <xacro:property name="bumper_offset_z_cm"         value="-2.5" />
@@ -18,4 +19,5 @@
   <xacro:property name="caster_position_y_cm"       value="0" />
   <xacro:property name="caster_position_z_cm"       value="-5.4" />
+  <xacro:property name="inertial_offset_x_cm"       value="1" />
   <!-- Create 3 base definitions-->
   <link name="base_footprint"/>
@@ -26,12 +28,11 @@
   <link name="base_link">
     <visual>
-      <origin xyz="0 0 ${body_z_offset_cm*cm2m}" rpy="0 0 ${-pi*3.0/2.0}"/>
+      <origin xyz="0 0 ${body_z_offset_cm*cm2m}" rpy="0 0 ${pi/2}"/>
       <geometry>
-        <mesh filename="file://$(find irobot_create_description)/meshes/body_collision.stl"
-          scale="0.001 0.001 0.001"/>
+        <mesh filename="file://$(find irobot_create_description)/meshes/body_visual.dae" />
       </geometry>
     </visual>
     <collision name="create3_base_collision">
-      <origin xyz="0 0 ${body_z_offset_cm*cm2m/2}"/>
+      <origin xyz="0 0 ${body_collision_z_offset_cm*cm2m}" rpy="0 0 ${pi/2}"/>
       <geometry>
         <cylinder length="${body_length_cm*cm2m}" radius="${body_radius_cm*cm2m}"/>
@@ -40,5 +41,5 @@
     <xacro:inertial_cylinder_with_pose mass="${body_mass_kg}" radius="${body_radius_cm*cm2m}"
       length="${body_length_cm*cm2m}">
-      <origin xyz="0 0 ${body_z_offset_cm*cm2m}"/>
+      <origin xyz="${inertial_offset_x_cm*cm2m} 0 ${body_collision_z_offset_cm*cm2m}"/>
     </xacro:inertial_cylinder_with_pose>
   </link>
@@ -47,7 +48,7 @@
       parent_link="base_link"
       robot_type="create3"
-      visual_mesh="file://$(find irobot_create_description)/meshes/bumper_collision.stl"
-      collision_mesh="file://$(find irobot_create_description)/meshes/bumper_collision.stl">
-    <origin xyz="0 0 ${bumper_offset_z_cm*cm2m}"/>
+      visual_mesh="file://$(find irobot_create_description)/meshes/bumper_visual.dae"
+      collision_mesh="file://$(find irobot_create_description)/meshes/bumper_collision.dae">
+    <origin xyz="0 0 ${bumper_offset_z_cm*cm2m}" rpy="0 0 ${pi/2}"/>
     <inertial>
         <origin xyz="${bumber_inertial_x_cm*cm2m} 0 ${bumper_offset_z_cm*cm2m}"/>

File: irobot_create_description/urdf/wheel.urdf.xacro (robot description, xacro)
@@ -32,4 +32,5 @@
     <minDepth>0.0001</minDepth>
     <maxVel>1.0</maxVel>
+    <material>Gazebo/DarkGrey</material>
   </gazebo>
 </xacro:macro>

Commit message: Fix movement in Rviz and add color to wheels

File: irobot_create_description/urdf/caster.urdf.xacro (robot description, xacro)
@@ -13,4 +13,6 @@
         <sphere radius="${radius_cm*cm2m}"/>
       </geometry>
+      <!-- Give black color to caster in Rviz -->
+      <xacro:insert_block name="material_black"/>
     </visual>
     <collision>

File: irobot_create_description/urdf/common_properties.urdf.xacro (robot description, xacro)
@@ -37,3 +37,9 @@
   <xacro:property name="mm2m"    value="${1/1000.0}"/>
   <xacro:property name="deg2rad" value="${pi/180}"/>
+  <!-- Material colors -->
+  <xacro:property name="material_black">
+    <material name="black">
+      <color rgba="0.1 0.1 0.1 1"/>
+    </material>
+  </xacro:property>
 </robot>

File: irobot_create_description/urdf/wheel.urdf.xacro (robot description, xacro)
@@ -16,4 +16,6 @@
         <cylinder length="${width_cm*cm2m}" radius="${radius_cm*cm2m}"/>
       </geometry>
+      <!-- Give black color to wheels in Rviz -->
+      <xacro:insert_block name="material_black"/>
     </visual>
     <collision>

Commit message: Make caster a separate model

File: irobot_create_description/urdf/caster.urdf.xacro (robot description, xacro)
@@ -2,5 +2,7 @@
 <robot xmlns:xacro="http://ros.org/wiki/xacro">
 <xacro:macro name="caster" params="name parent_link *origin">
-  <xacro:property name="radius_cm" value="1" />
+  <xacro:include filename="$(find irobot_create_description)/urdf/common_properties.urdf.xacro"/>
+  <xacro:property name="radius" value="${1*cm2m}" />
+  <xacro:property name="mass"   value="0.01"/>
   <joint name="${name}_joint" type="fixed">
     <parent link="${parent_link}"/>
@@ -11,5 +13,5 @@
     <visual>
       <geometry>
-        <sphere radius="${radius_cm*cm2m}"/>
+        <sphere radius="${radius}"/>
       </geometry>
       <!-- Give black color to caster in Rviz -->
@@ -18,10 +20,18 @@
     <collision>
       <geometry>
-        <sphere radius="${radius_cm*cm2m}"/>
+        <sphere radius="${radius}"/>
       </geometry>
     </collision>
+    <xacro:inertial_sphere mass="${mass}" diameter="${2*radius}"/>
   </link>
+  <gazebo reference="${name}_joint">
+    <preserveFixedJoint>true</preserveFixedJoint>
+  </gazebo>
   <gazebo reference="${name}_link">
     <material>Gazebo/DarkGrey</material>
+    <mu1>0.1</mu1>
+    <mu2>0.1</mu2>
+    <kp>1000000.0</kp>
+    <kd>1.0</kd>
   </gazebo>
 </xacro:macro>
