Commit message: Address PR comments

File: irobot_create_description/urdf/common_properties.urdf.xacro (robot description, xacro)
@@ -1,3 +1,4 @@
 <?xml version="1.0" ?>
+<<<<<<< HEAD
 <!-- Various useful macros -->
 <robot name="xacro_properties" xmlns:xacro="http://ros.org/wiki/xacro">
@@ -9,4 +10,17 @@
         iyy="${(1/12) * mass * (x*x + z*z)}" iyz="0.0"
         izz="${(1/12) * mass * (x*x + y*y)}" />
+=======
+<!--
+  Various useful macros
+ -->
+<robot name="xacro_properties" xmlns:xacro="http://ros.org/wiki/xacro">
+  <xacro:macro name="inertial_cuboid" params="mass x_length y_length z_length">
+    <inertial>
+      <mass value="${mass}" />
+      <origin xyz="0 0 0" />
+      <inertia ixx="${(1/12) * mass * (y_length*y_length + z_length*z_length)}" ixy="0.0" ixz="0.0"
+	iyy="${(1/12) * mass * (x_length*x_length + z_length*z_length)}" iyz="0.0"
+	izz="${(1/12) * mass * (x_length*x_length + y_length*y_length)}" />
+>>>>>>> Address PR comments
     </inertial>
   </xacro:macro>
@@ -16,6 +30,11 @@
       <origin xyz="0 0 0" />
       <inertia ixx="${(1/12) * mass * (3*radius*radius + length*length)}" ixy="0.0" ixz="0.0"
+<<<<<<< HEAD
         iyy="${(1/12) * mass * (3*radius*radius + length*length)}" iyz="0.0"
         izz="${(1/2) * mass * (radius*radius)}" />
+=======
+	iyy="${(1/12) * mass * (3*radius*radius + length*length)}" iyz="0.0"
+	izz="${(1/2) * mass * (radius*radius)}" />
+>>>>>>> Address PR comments
     </inertial>
   </xacro:macro>
@@ -25,4 +44,5 @@
       <mass value="${mass}" />
       <inertia ixx="${(1/12) * mass * (3*radius*radius + length*length)}" ixy="0.0" ixz="0.0"
+<<<<<<< HEAD
         iyy="${(1/12) * mass * (3*radius*radius + length*length)}" iyz="0.0"
         izz="${(1/2) * mass * (radius*radius)}" />
@@ -32,3 +52,9 @@
   <xacro:property name="cm2m" value="${1/100.0}"/>
   <xacro:property name="mm2m" value="${1/1000.0}"/>
+=======
+	iyy="${(1/12) * mass * (3*radius*radius + length*length)}" iyz="0.0"
+	izz="${(1/2) * mass * (radius*radius)}" />
+    </inertial>
+  </xacro:macro>
+>>>>>>> Address PR comments
 </robot>

Commit message: Gives files more appropriate names and makes macro of the caster wheel

File: irobot_create_description/urdf/common_properties.urdf.xacro (robot description, xacro)
@@ -4,11 +4,11 @@
  -->
 <robot name="xacro_properties" xmlns:xacro="http://ros.org/wiki/xacro">
-  <xacro:macro name="inertial_cuboid" params="mass x_length y_length z_length">
+  <xacro:macro name="inertial_cuboid" params="mass x y z">
     <inertial>
       <mass value="${mass}" />
       <origin xyz="0 0 0" />
-      <inertia ixx="${(1/12) * mass * (y_length*y_length + z_length*z_length)}" ixy="0.0" ixz="0.0"
-	iyy="${(1/12) * mass * (x_length*x_length + z_length*z_length)}" iyz="0.0"
-	izz="${(1/12) * mass * (x_length*x_length + y_length*y_length)}" />
+      <inertia ixx="${(1/12) * mass * (y*y + z*z)}" ixy="0.0" ixz="0.0"
+	iyy="${(1/12) * mass * (x*x + z*z)}" iyz="0.0"
+	izz="${(1/12) * mass * (x*x + y*y)}" />
     </inertial>
   </xacro:macro>

File: irobot_create_description/urdf/create3.urdf.xacro (robot description, xacro)
@@ -2,6 +2,7 @@
 <robot name="create3" xmlns:xacro="http://ros.org/wiki/xacro">
   <xacro:include filename="$(find irobot_create_description)/urdf/common_properties.urdf.xacro"/>
-  <xacro:include filename="$(find irobot_create_description)/urdf/bumper.xacro" />
-  <xacro:include filename="$(find irobot_create_description)/urdf/wheel_with_wheeldrop.xacro" />
+  <xacro:include filename="$(find irobot_create_description)/urdf/bumper.urdf.xacro" />
+  <xacro:include filename="$(find irobot_create_description)/urdf/wheel_with_wheeldrop.urdf.xacro" />
+  <xacro:include filename="$(find irobot_create_description)/urdf/caster.urdf.xacro" />
   <!-- MECHANICAL PROPERTIES -->
   <xacro:property name="body_z_offset" value="-0.025" /><!-- z offset from ground [m] -->
@@ -13,5 +14,4 @@
   <xacro:property name="wheel_height" value="-0.0275" /><!-- z [m] -->
   <xacro:property name="distance_between_wheels" value="0.233" /><!-- y [m] -->
-  <xacro:property name="caster_radius" value="0.01" /> <!-- [m] -->
   <xacro:property name="caster_position_x" value="0.125" /><!-- x [m] -->
   <xacro:property name="caster_position_y" value="0" /><!-- y [m] -->
@@ -60,20 +60,7 @@
     <origin xyz="0 ${-distance_between_wheels/2} ${wheel_height}" rpy="${-pi/2} 0 0"/>
   </xacro:wheel_with_wheeldrop>
-  <joint name="caster_joint" type="fixed">
-    <parent link="base_link"/>
-    <child link="caster_link"/>
+  <!-- Caster wheel -->
+  <xacro:caster name="front_caster" parent_link="base_link">
     <origin xyz="${caster_position_x} ${caster_position_y} ${caster_position_z}" rpy="${-pi/2} 0 0"/>
-  </joint>
-  <link name="caster_link">
-    <visual>
-      <geometry>
-        <sphere radius="${caster_radius}"/>
-      </geometry>
-    </visual>
-    <collision>
-      <geometry>
-        <sphere radius="${caster_radius}"/>
-      </geometry>
-    </collision>
-  </link>
+  </xacro:caster>
 </robot>

File: irobot_create_description/urdf/wheel_with_wheeldrop.urdf.xacro (robot description, xacro)
@@ -1,9 +1,6 @@
 <?xml version="1.0"?>
 <robot xmlns:xacro="http://ros.org/wiki/xacro">
-<xacro:include filename="$(find irobot_create_description)/urdf/wheel.xacro" />
+<xacro:include filename="$(find irobot_create_description)/urdf/wheel.urdf.xacro" />
 <xacro:macro name="wheel_with_wheeldrop" params="name parent_link *origin">
-  <xacro:property name="wheel_mass" value="0.2" /> <!-- [kg] -->
-  <xacro:property name="wheel_radius" value="0.03575" /> <!-- [m] -->
-  <xacro:property name="wheel_width" value="0.015" /> <!-- [m] -->
   <joint name="wheel_${name}_axle_joint" type="prismatic">
     <parent link="${parent_link}"/>
@@ -21,7 +18,7 @@
   <link name="wheel_${name}_axle_link">
       <xacro:inertial_cuboid mass="0.05"
-                             x_length="0.15"
-                             y_length="0.15"
-                             z_length="0.15"/>
+                             x="0.15"
+                             y="0.15"
+                             z="0.15"/>
   </link>
   <!-- Wheel definition -->

Commit message: Gives files more appropriate names and makes macro of the caster wheel

File: irobot_create_description/urdf/common_properties.urdf.xacro (robot description, xacro)
@@ -1,4 +1,3 @@
 <?xml version="1.0" ?>
-<<<<<<< HEAD
 <!-- Various useful macros -->
 <robot name="xacro_properties" xmlns:xacro="http://ros.org/wiki/xacro">
@@ -10,17 +9,4 @@
         iyy="${(1/12) * mass * (x*x + z*z)}" iyz="0.0"
         izz="${(1/12) * mass * (x*x + y*y)}" />
-=======
-<!--
-  Various useful macros
- -->
-<robot name="xacro_properties" xmlns:xacro="http://ros.org/wiki/xacro">
-  <xacro:macro name="inertial_cuboid" params="mass x_length y_length z_length">
-    <inertial>
-      <mass value="${mass}" />
-      <origin xyz="0 0 0" />
-      <inertia ixx="${(1/12) * mass * (y_length*y_length + z_length*z_length)}" ixy="0.0" ixz="0.0"
-	iyy="${(1/12) * mass * (x_length*x_length + z_length*z_length)}" iyz="0.0"
-	izz="${(1/12) * mass * (x_length*x_length + y_length*y_length)}" />
->>>>>>> Address PR comments
     </inertial>
   </xacro:macro>
@@ -30,11 +16,6 @@
       <origin xyz="0 0 0" />
       <inertia ixx="${(1/12) * mass * (3*radius*radius + length*length)}" ixy="0.0" ixz="0.0"
-<<<<<<< HEAD
         iyy="${(1/12) * mass * (3*radius*radius + length*length)}" iyz="0.0"
         izz="${(1/2) * mass * (radius*radius)}" />
-=======
-	iyy="${(1/12) * mass * (3*radius*radius + length*length)}" iyz="0.0"
-	izz="${(1/2) * mass * (radius*radius)}" />
->>>>>>> Address PR comments
     </inertial>
   </xacro:macro>
@@ -44,5 +25,4 @@
       <mass value="${mass}" />
       <inertia ixx="${(1/12) * mass * (3*radius*radius + length*length)}" ixy="0.0" ixz="0.0"
-<<<<<<< HEAD
         iyy="${(1/12) * mass * (3*radius*radius + length*length)}" iyz="0.0"
         izz="${(1/2) * mass * (radius*radius)}" />
@@ -52,9 +32,3 @@
   <xacro:property name="cm2m" value="${1/100.0}"/>
   <xacro:property name="mm2m" value="${1/1000.0}"/>
-=======
-	iyy="${(1/12) * mass * (3*radius*radius + length*length)}" iyz="0.0"
-	izz="${(1/2) * mass * (radius*radius)}" />
-    </inertial>
-  </xacro:macro>
->>>>>>> Address PR comments
 </robot>

File: irobot_create_description/urdf/create3.urdf.xacro (robot description, xacro)
@@ -15,7 +15,13 @@
   <xacro:property name="wheel_height_cm"            value="-2.75" />
   <xacro:property name="distance_between_wheels_cm" value="23.3" />
+<<<<<<< HEAD
   <xacro:property name="caster_position_x_cm"       value="12.5" />
   <xacro:property name="caster_position_y_cm"       value="0" />
   <xacro:property name="caster_position_z_cm"       value="-5.4" />
+=======
+  <xacro:property name="caster_position_x" value="0.125" /><!-- x [m] -->
+  <xacro:property name="caster_position_y" value="0" /><!-- y [m] -->
+  <xacro:property name="caster_position_z" value="-0.054" /><!-- z [m] -->
+>>>>>>> Gives files more appropriate names and makes macro of the caster wheel
   <!-- Create 3 base definitions-->
   <link name="base_footprint"/>
@@ -66,6 +72,10 @@
   <!-- Caster wheel -->
   <xacro:caster name="front_caster" parent_link="base_link">
+<<<<<<< HEAD
     <origin xyz="${caster_position_x_cm*cm2m} ${caster_position_y_cm*cm2m} ${caster_position_z_cm*cm2m}"
       rpy="${-pi/2} 0 0"/>
+=======
+    <origin xyz="${caster_position_x} ${caster_position_y} ${caster_position_z}" rpy="${-pi/2} 0 0"/>
+>>>>>>> Gives files more appropriate names and makes macro of the caster wheel
   </xacro:caster>
 </robot>

Commit message: xacro formatting changes and adds README specifying dependencies

File: irobot_create_description/urdf/common_properties.urdf.xacro (robot description, xacro)
@@ -1,6 +1,4 @@
 <?xml version="1.0" ?>
-<!--
-  Various useful macros
- -->
+<!-- Various useful macros -->
 <robot name="xacro_properties" xmlns:xacro="http://ros.org/wiki/xacro">
   <xacro:macro name="inertial_cuboid" params="mass x y z">

File: irobot_create_description/urdf/create3.urdf.xacro (robot description, xacro)
@@ -48,5 +48,5 @@
     <origin xyz="0 0 ${bumper_offset_z}"/>
     <inertial>
-      <origin xyz="0.08 0 ${bumper_offset_z + 0.01}"/>
+      <origin xyz="0.08 0 ${bumper_offset_z}"/>
       <mass value="${bumper_mass}"/>
       <inertia ixx="0.0013483753405" ixy="0.0000000454352" ixz="0.0000014434849" iyy="0.0002521736852" iyz="-0.0000000006721" izz="0.0015442525386"/>

File: irobot_create_description/urdf/wheel.urdf.xacro (robot description, xacro)
@@ -2,7 +2,7 @@
 <robot xmlns:xacro="http://ros.org/wiki/xacro">
 <xacro:macro name="wheel" params="name parent_link *origin">
-  <xacro:property name="wheel_mass" value="0.2" /> <!-- [kg] -->
+  <xacro:property name="wheel_mass"   value="0.2" /> <!-- [kg] -->
   <xacro:property name="wheel_radius" value="0.03575" /> <!-- [m] -->
-  <xacro:property name="wheel_width" value="0.015" /> <!-- [m] -->
+  <xacro:property name="wheel_width"  value="0.015" /> <!-- [m] -->
   <joint name="wheel_${name}_joint" type="continuous">
     <parent link="${parent_link}"/>

Commit message: Change variable names

File: irobot_create_description/urdf/common_properties.urdf.xacro (robot description, xacro)
@@ -31,3 +31,4 @@
   <!-- Conversion macros -->
   <xacro:property name="cm2m"    value="${1/100.0}"/>
+  <xacro:property name="mm2m"    value="${1/1000.0}"/>
 </robot>

File: irobot_create_description/urdf/wheel.urdf.xacro (robot description, xacro)
@@ -2,7 +2,7 @@
 <robot xmlns:xacro="http://ros.org/wiki/xacro">
 <xacro:macro name="wheel" params="name parent_link *origin">
-  <xacro:property name="wheel_mass_kg"   value="0.2" />
-  <xacro:property name="wheel_radius_cm" value="3.575" />
-  <xacro:property name="wheel_width_cm"  value="1.5" />
+  <xacro:property name="mass_kg"   value="0.2" />
+  <xacro:property name="radius_cm" value="3.575" />
+  <xacro:property name="width_cm"  value="1.5" />
   <joint name="wheel_${name}_joint" type="continuous">
     <parent link="${parent_link}"/>
@@ -14,14 +14,14 @@
     <visual>
       <geometry>
-        <cylinder length="${wheel_width_cm*cm2m}" radius="${wheel_radius_cm*cm2m}"/>
+        <cylinder length="${width_cm*cm2m}" radius="${radius_cm*cm2m}"/>
       </geometry>
     </visual>
     <collision>
       <geometry>
-        <cylinder length="${wheel_width_cm*cm2m}" radius="${wheel_radius_cm*cm2m}"/>
+        <cylinder length="${width_cm*cm2m}" radius="${radius_cm*cm2m}"/>
       </geometry>
     </collision>
-    <xacro:inertial_cylinder mass="${wheel_mass_kg}" radius="${wheel_radius_cm*cm2m}"
-      length="${wheel_width_cm*cm2m}" />
+    <xacro:inertial_cylinder mass="${mass_kg}" radius="${radius_cm*cm2m}"
+      length="${width_cm*cm2m}" />
   </link>
   <gazebo reference="wheel_${name}_link">

File: irobot_create_description/urdf/wheel_with_wheeldrop.urdf.xacro (robot description, xacro)
@@ -3,14 +3,14 @@
 <xacro:include filename="$(find irobot_create_description)/urdf/wheel.urdf.xacro" />
 <xacro:macro name="wheel_with_wheeldrop" params="name parent_link *origin">
-  <xacro:property name="wheel_drop_lower"             value="0" />
-  <xacro:property name="wheel_drop_upper"             value="0.03" />
-  <xacro:property name="wheel_drop_effort"            value="100" />
-  <xacro:property name="wheel_drop_vel"               value="1" />
-  <xacro:property name="wheel_drop_spring_stiffness"  value="300" />
-  <xacro:property name="wheel_drop_spring_reference"  value="0.03" />
-  <xacro:property name="wheel_axle_mass"              value="0.05" />
-  <xacro:property name="wheel_axle_x"                 value="0.15" />
-  <xacro:property name="wheel_axle_y"                 value="0.15" />
-  <xacro:property name="wheel_axle_z"                 value="0.15" />
+  <xacro:property name="lower_mm"          value="0" />
+  <xacro:property name="upper_mm"          value="30" />
+  <xacro:property name="effort"            value="100" />
+  <xacro:property name="velocity"          value="1" />
+  <xacro:property name="spring_stiffness"  value="300" />
+  <xacro:property name="spring_reference"  value="0.03" />
+  <xacro:property name="axle_mass"         value="0.05" />
+  <xacro:property name="axle_x"            value="0.15" />
+  <xacro:property name="axle_y"            value="0.15" />
+  <xacro:property name="axle_z"            value="0.15" />
   <joint name="wheel_${name}_axle_joint" type="prismatic">
     <parent link="${parent_link}"/>
@@ -18,16 +18,16 @@
     <xacro:insert_block name="origin"/>
     <axis xyz="0 1 0"/>
-    <limit lower="${wheel_drop_lower}" upper="${wheel_drop_upper}" effort="${wheel_drop_effort}"
-      velocity="${wheel_drop_vel}"/>
+    <limit lower="${lower_mm*mm2m}" upper="${upper_mm*mm2m}" effort="${effort}"
+      velocity="${velocity}"/>
   </joint>
   <!-- Gazebo parameters to simulate a spring -->
   <gazebo reference="wheel_${name}_axle_joint">
     <implicitSpringDamper>true</implicitSpringDamper>
-    <springStiffness>${wheel_drop_spring_stiffness}</springStiffness>
-    <springReference>${wheel_drop_spring_reference}</springReference>
+    <springStiffness>${spring_stiffness}</springStiffness>
+    <springReference>${spring_reference}</springReference>
   </gazebo>
   <link name="wheel_${name}_axle_link">
-    <xacro:inertial_cuboid mass="${wheel_axle_mass}" x="${wheel_axle_x}" y="${wheel_axle_y}"
-      z="${wheel_axle_z}"/>
+    <xacro:inertial_cuboid mass="${axle_mass}" x="${axle_x}" y="${axle_y}"
+      z="${axle_z}"/>
   </link>
   <!-- Wheel definition -->

Commit message: Apply suggestions from linters

File: irobot_create_description/urdf/common_properties.urdf.xacro (robot description, xacro)
@@ -30,5 +30,5 @@
   </xacro:macro>
   <!-- Conversion macros -->
-  <xacro:property name="cm2m"    value="${1/100.0}"/>
-  <xacro:property name="mm2m"    value="${1/1000.0}"/>
+  <xacro:property name="cm2m" value="${1/100.0}"/>
+  <xacro:property name="mm2m" value="${1/1000.0}"/>
 </robot>

File: irobot_create_description/urdf/wheel_with_wheeldrop.urdf.xacro (robot description, xacro)
@@ -3,14 +3,14 @@
 <xacro:include filename="$(find irobot_create_description)/urdf/wheel.urdf.xacro" />
 <xacro:macro name="wheel_with_wheeldrop" params="name parent_link *origin">
-  <xacro:property name="lower_mm"          value="0" />
-  <xacro:property name="upper_mm"          value="30" />
-  <xacro:property name="effort"            value="100" />
-  <xacro:property name="velocity"          value="1" />
-  <xacro:property name="spring_stiffness"  value="300" />
-  <xacro:property name="spring_reference"  value="0.03" />
-  <xacro:property name="axle_mass"         value="0.05" />
-  <xacro:property name="axle_x"            value="0.15" />
-  <xacro:property name="axle_y"            value="0.15" />
-  <xacro:property name="axle_z"            value="0.15" />
+  <xacro:property name="lower_mm"         value="0" />
+  <xacro:property name="upper_mm"         value="30" />
+  <xacro:property name="effort"           value="100" />
+  <xacro:property name="velocity"         value="1" />
+  <xacro:property name="spring_stiffness" value="300" />
+  <xacro:property name="spring_reference" value="0.03" />
+  <xacro:property name="axle_mass"        value="0.05" />
+  <xacro:property name="axle_x"           value="0.15" />
+  <xacro:property name="axle_y"           value="0.15" />
+  <xacro:property name="axle_z"           value="0.15" />
   <joint name="wheel_${name}_axle_joint" type="prismatic">
     <parent link="${parent_link}"/>

Commit message: Improve common_properties xacro

File: irobot_create_description/urdf/common_properties.urdf.xacro (robot description, xacro)
@@ -2,8 +2,8 @@
 <!-- Various useful macros -->
 <robot name="xacro_properties" xmlns:xacro="http://ros.org/wiki/xacro">
-  <xacro:macro name="inertial_cuboid" params="mass x y z">
+  <xacro:macro name="inertial_cuboid_with_pose" params="mass x y z *origin">
     <inertial>
       <mass value="${mass}" />
-      <origin xyz="0 0 0" />
+      <xacro:insert_block name="origin"/>
       <inertia ixx="${(1/12) * mass * (y*y + z*z)}" ixy="0.0" ixz="0.0"
         iyy="${(1/12) * mass * (x*x + z*z)}" iyz="0.0"
@@ -11,12 +11,8 @@
     </inertial>
   </xacro:macro>
-  <xacro:macro name="inertial_cylinder" params="mass radius length">
-    <inertial>
-      <mass value="${mass}"/>
+  <xacro:macro name="inertial_cuboid" params="mass x y z">
+    <xacro:inertial_cuboid_with_pose mass="${mass}" x="${x}" y="${y}" z="${z}">
       <origin xyz="0 0 0" />
-      <inertia ixx="${(1/12) * mass * (3*radius*radius + length*length)}" ixy="0.0" ixz="0.0"
-        iyy="${(1/12) * mass * (3*radius*radius + length*length)}" iyz="0.0"
-        izz="${(1/2) * mass * (radius*radius)}" />
-    </inertial>
+    </xacro:inertial_cuboid_with_pose>
   </xacro:macro>
   <xacro:macro name="inertial_cylinder_with_pose" params="mass radius length *origin">
@@ -29,4 +25,9 @@
     </inertial>
   </xacro:macro>
+  <xacro:macro name="inertial_cylinder" params="mass radius length">
+    <xacro:inertial_cylinder_with_pose mass="${mass}" radius="${radius}" length="${length}">
+      <origin xyz="0 0 0" />
+    </xacro:inertial_cylinder_with_pose>
+  </xacro:macro>
   <!-- Conversion macros -->
   <xacro:property name="cm2m" value="${1/100.0}"/>

Commit message: Simplify dock xacro

File: irobot_create_description/urdf/common_properties.urdf.xacro (robot description, xacro)
@@ -31,5 +31,6 @@
   </xacro:macro>
   <!-- Conversion macros -->
-  <xacro:property name="cm2m" value="${1/100.0}"/>
-  <xacro:property name="mm2m" value="${1/1000.0}"/>
+  <xacro:property name="cm2m"    value="${1/100.0}"/>
+  <xacro:property name="mm2m"    value="${1/1000.0}"/>
+  <xacro:property name="deg2rad" value="${pi/180}"/>
 </robot>

File: irobot_create_description/urdf/dock/standard.urdf.xacro (robot description, xacro)
@@ -34,13 +34,10 @@
   <xacro:property name="buoy_y" value="0.005"/>
   <xacro:property name="buoy_z" value="${0.065 - (z_offset_mm*mm2m)}"/>
-  <xacro:property name="halo_x" value="-0.052"/>
-  <xacro:property name="halo_z" value="${0.095 - (z_offset_mm*mm2m)}"/>
-  <xacro:property name="halo_name" value="halo"/>
-  <xacro:property name="green_buoy_name" value="green_buoy"/>
-  <xacro:property name="red_buoy_name" value="red_buoy"/>
+  <xacro:property name="halo_name"        value="halo"/>
+  <xacro:property name="green_buoy_name"  value="green_buoy"/>
+  <xacro:property name="red_buoy_name"    value="red_buoy"/>
   <xacro:property name="yellow_buoy_name" value="yellow_buoy"/>
-  <xacro:property name="buoy_central_aperture"  value="${10/180 * pi}"/>
-  <xacro:property name="buoy_lateral_angle_yaw" value="${10/180 * pi}"/>
-  <xacro:property name="buoy_lateral_aperture"  value="${30/180 * pi}"/>
+  <xacro:property name="buoy_lateral_angle_yaw" value="${10*deg2rad}"/>
+  <xacro:property name="buoy_lateral_aperture"  value="${30*deg2rad}"/>
   <!-- Green IR emitter -->
   <xacro:ir_emitter name="${green_buoy_name}"
@@ -62,5 +59,5 @@
   <xacro:ir_emitter name="${yellow_buoy_name}"
                     code="172"
-                    aperture="${buoy_central_aperture}"
+                    aperture="${10*deg2rad}"
                     range="1.2192">
     <origin xyz="${buoy_x} 0 ${buoy_z}"/>
@@ -71,5 +68,5 @@
                     aperture="360"
                     range="0.6096">
-    <origin xyz="${halo_x} 0 ${halo_z}"/>
+    <origin xyz="-0.052 0 ${0.095 - (z_offset_mm*mm2m)}"/>
   </xacro:ir_emitter>
   <xacro:property name="real_behavior" value="$(arg real_behavior)"/>
