Commit message: Add docking station (#6)
* Improve common_properties xacro

* Use dock.launch.py

* Add standard dock spawner

* Add dock meshes

* Add dock URDF xacros

* Simplify IR emitter Xacro

* Simplify dock xacro

* Fix Ament Flake8

* Use primitive instead of mesh for dock's collision model

* Add ament_pycodestyle to CI

* Fix ament_pycodestyle

* Add pyflakes

* Add mypy static linting to CI

* Add ending commas

* fixup! Add ending commas

File: irobot_create_description/urdf/common_properties.urdf.xacro (robot description, xacro)
@@ -2,8 +2,8 @@
 <!-- Various useful macros -->
 <robot name="xacro_properties" xmlns:xacro="http://ros.org/wiki/xacro">
-  <xacro:macro name="inertial_cuboid" params="mass x y z">
+  <xacro:macro name="inertial_cuboid_with_pose" params="mass x y z *origin">
     <inertial>
       <mass value="${mass}" />
-      <origin xyz="0 0 0" />
+      <xacro:insert_block name="origin"/>
       <inertia ixx="${(1/12) * mass * (y*y + z*z)}" ixy="0.0" ixz="0.0"
         iyy="${(1/12) * mass * (x*x + z*z)}" iyz="0.0"
@@ -11,12 +11,8 @@
     </inertial>
   </xacro:macro>
-  <xacro:macro name="inertial_cylinder" params="mass radius length">
-    <inertial>
-      <mass value="${mass}"/>
+  <xacro:macro name="inertial_cuboid" params="mass x y z">
+    <xacro:inertial_cuboid_with_pose mass="${mass}" x="${x}" y="${y}" z="${z}">
       <origin xyz="0 0 0" />
-      <inertia ixx="${(1/12) * mass * (3*radius*radius + length*length)}" ixy="0.0" ixz="0.0"
-        iyy="${(1/12) * mass * (3*radius*radius + length*length)}" iyz="0.0"
-        izz="${(1/2) * mass * (radius*radius)}" />
-    </inertial>
+    </xacro:inertial_cuboid_with_pose>
   </xacro:macro>
   <xacro:macro name="inertial_cylinder_with_pose" params="mass radius length *origin">
@@ -29,6 +25,12 @@
     </inertial>
   </xacro:macro>
+  <xacro:macro name="inertial_cylinder" params="mass radius length">
+    <xacro:inertial_cylinder_with_pose mass="${mass}" radius="${radius}" length="${length}">
+      <origin xyz="0 0 0" />
+    </xacro:inertial_cylinder_with_pose>
+  </xacro:macro>
   <!-- Conversion macros -->
-  <xacro:property name="cm2m" value="${1/100.0}"/>
-  <xacro:property name="mm2m" value="${1/1000.0}"/>
+  <xacro:property name="cm2m"    value="${1/100.0}"/>
+  <xacro:property name="mm2m"    value="${1/1000.0}"/>
+  <xacro:property name="deg2rad" value="${pi/180}"/>
 </robot>

Commit message: Add a few useful macros

File: irobot_create_description/urdf/common_properties.urdf.xacro (robot description, xacro)
@@ -29,4 +29,6 @@
       <origin xyz="0 0 0" />
     </xacro:inertial_cylinder_with_pose>
+  <xacro:macro name="inertial_dummy">
+    <xacro:inertial_cuboid mass="0.01" x="0.01" y="0.01" z="0.01"/>
   </xacro:macro>
   <xacro:macro name="inertial_dummy">
@@ -36,4 +38,4 @@
   <xacro:property name="cm2m"    value="${1/100.0}"/>
   <xacro:property name="mm2m"    value="${1/1000.0}"/>
-  <xacro:property name="deg2rad" value="${pi/180}"/>
+  <xacro:property name="deg2rad" value="${pi/180.0}"/>
 </robot>

Commit message: fixup! Add a few useful macros

File: irobot_create_description/urdf/common_properties.urdf.xacro (robot description, xacro)
@@ -29,4 +29,5 @@
       <origin xyz="0 0 0" />
     </xacro:inertial_cylinder_with_pose>
+  </xacro:macro>
   <xacro:macro name="inertial_dummy">
     <xacro:inertial_cuboid mass="0.01" x="0.01" y="0.01" z="0.01"/>

Commit message: Uses inertial_dummy

File: irobot_create_description/urdf/common_properties.urdf.xacro (robot description, xacro)
@@ -30,4 +30,7 @@
     </xacro:inertial_cylinder_with_pose>
   </xacro:macro>
+  <xacro:macro name="inertial_dummy">
+    <xacro:inertial_cuboid mass="0.01" x="0.01" y="0.01" z="0.01"/>
+  </xacro:macro>
   <!-- Conversion macros -->
   <xacro:property name="cm2m"    value="${1/100.0}"/>

File: irobot_create_description/urdf/sensors/mouse.urdf.xacro (robot description, xacro)
@@ -2,8 +2,4 @@
 <robot xmlns:xacro="http://ros.org/wiki/xacro">
   <xacro:macro name="mouse" params="name:=mouse parent_link *origin update_rate" >
-    <!-- Sensor settings -->
-    <xacro:property name="mass" value="0.1" />
-    <xacro:property name="length" value="0.008" /> <!-- Length -->
-    <xacro:property name="radius" value="0.01" /> <!-- Radius -->
     <joint name="${name}_joint" type="fixed">
       <xacro:insert_block name="origin"/>
@@ -12,5 +8,5 @@
     </joint>
     <link name="${name}">
-      <xacro:inertial_cylinder mass="${mass}" length="${length}" radius="${radius}" />
+      <xacro:inertial_dummy />
     </link>
     <gazebo>

Commit message: Add IR intensity sensors (#13)
* Add a few useful macros

* Add IR intensity sensors to Create 3

* Fix warning in WD sensors

* Add IR intensity plugins

* Add IR intensity xacro

* fixup! Add a few useful macros

* Fix linter

* Fix range detection

* Move IR sensors behind the bumpers

* Clean up

* Fix linter

* Rename namespaces

* Address comments

* Move minimum range to Gazebo Helpers

* Change variable usage

* fixup! Change variable usage

* Fix grammar typos

* Fix IR intensity drawing

* Move ir_intensity xacro to sensors directory

* Set always_on to true

* fixup! Fix grammar typos

File: irobot_create_description/urdf/common_properties.urdf.xacro (robot description, xacro)
@@ -33,7 +33,10 @@
     <xacro:inertial_cuboid mass="0.01" x="0.01" y="0.01" z="0.01"/>
   </xacro:macro>
+  <xacro:macro name="inertial_dummy">
+    <xacro:inertial_cuboid mass="0.01" x="0.01" y="0.01" z="0.01"/>
+  </xacro:macro>
   <!-- Conversion macros -->
   <xacro:property name="cm2m"    value="${1/100.0}"/>
   <xacro:property name="mm2m"    value="${1/1000.0}"/>
-  <xacro:property name="deg2rad" value="${pi/180}"/>
+  <xacro:property name="deg2rad" value="${pi/180.0}"/>
 </robot>

File: irobot_create_description/urdf/create3.urdf.xacro (robot description, xacro)
@@ -4,4 +4,5 @@
   <xacro:include filename="$(find irobot_create_description)/urdf/caster.urdf.xacro" />
   <xacro:include filename="$(find irobot_create_description)/urdf/common_properties.urdf.xacro"/>
+  <xacro:include filename="$(find irobot_create_description)/urdf/sensors/ir_intensity.urdf.xacro" />
   <xacro:include filename="$(find irobot_create_description)/urdf/sensors/optical_mouse.urdf.xacro"/>
   <xacro:include filename="$(find irobot_create_description)/urdf/wheel_with_wheeldrop.urdf.xacro" />
@@ -82,3 +83,39 @@
     <origin xyz="0.1015 0.087 -0.055" rpy="0 0 ${-pi/4}"/>
   </xacro:optical_mouse>
+  <!-- IR intensity sensors -->
+  <xacro:property name="ir_intensity_z_pos" value="${-0.7*cm2m}"/>
+  <!--
+  The robot uses 7 IR sensors in the front to execute a wall-following action
+  or reduce the speed when it detects something in front for safety reasons.
+  The arrangement of the sensors is defined in the following schema of the top
+  view of the robot:
+                          Front view
+                              |
+                              V
+                        front_center_left
+                front_left            front_center_right
+            left                                    front_right
+  side_left                                                   right
+  -->
+  <xacro:ir_intensity name="front_center_left">
+    <origin xyz="0.1540 0 ${ir_intensity_z_pos}"/>
+  </xacro:ir_intensity>
+  <xacro:ir_intensity name="front_center_right">
+    <origin xyz="0.1396 -0.0651 ${ir_intensity_z_pos}" rpy="0 0 -0.436"/>
+  </xacro:ir_intensity>
+  <xacro:ir_intensity name="front_left">
+    <origin xyz="0.1396 0.0651 ${ir_intensity_z_pos}" rpy="0 0 0.436"/>
+  </xacro:ir_intensity>
+  <xacro:ir_intensity name="front_right">
+    <origin xyz="0.0990 -0.1180 ${ir_intensity_z_pos}" rpy="0 0 -0.873"/>
+  </xacro:ir_intensity>
+  <xacro:ir_intensity name="left">
+    <origin xyz="0.0990 0.1180 ${ir_intensity_z_pos}" rpy="0 0 0.873"/>
+  </xacro:ir_intensity>
+  <xacro:ir_intensity name="right">
+    <origin xyz="0.0399 -0.1488 ${ir_intensity_z_pos}" rpy="0 0 -1.309"/>
+  </xacro:ir_intensity>
+  <xacro:ir_intensity name="side_left">
+    <origin xyz="0.0399 0.1488 ${ir_intensity_z_pos}" rpy="0 0 1.309"/>
+  </xacro:ir_intensity>
 </robot>

Commit message: Fix movement in Rviz and add color to wheels (#18)
* Fix movement in Rviz and add color to wheels

* updates rviz configuration

* Adds Dock and TF visualization

* link_name property for std dock link

* Flake8 error fixed

* rename variables

* Fix locales issue in Rviz

* Fix flake8

File: irobot_create_description/urdf/common_properties.urdf.xacro (robot description, xacro)
@@ -40,3 +40,9 @@
   <xacro:property name="mm2m"    value="${1/1000.0}"/>
   <xacro:property name="deg2rad" value="${pi/180.0}"/>
+  <!-- Material colors -->
+  <xacro:property name="material_black">
+    <material name="black">
+      <color rgba="0.1 0.1 0.1 1"/>
+    </material>
+  </xacro:property>
 </robot>

File: irobot_create_description/urdf/dock/standard.urdf.xacro (robot description, xacro)
@@ -4,5 +4,6 @@
   <xacro:include filename="$(find irobot_create_description)/urdf/dock/ir_emitter.urdf.xacro"/>
   <xacro:property name="z_offset_mm" value="4.6"/>
-  <link name="base_link">
+  <xacro:property name="link_name" value="std_dock_link"/>
+  <link name="${link_name}">
     <visual>
       <origin xyz="0 0 ${z_offset_mm*mm2m}"/>
@@ -19,5 +20,5 @@
     </collision>
   </link>
-  <gazebo reference="base_link">
+  <gazebo reference="${link_name}">
     <mu1>1.0</mu1>
     <mu2>1.0</mu2>
@@ -37,4 +38,5 @@
   <!-- Green IR emitter -->
   <xacro:ir_emitter name="${green_buoy_name}"
+                    parent="${link_name}"
                     code="164"
                     aperture="${buoy_lateral_aperture}"
@@ -45,4 +47,5 @@
   <!-- Red IR emitter -->
   <xacro:ir_emitter name="${red_buoy_name}"
+                    parent="${link_name}"
                     code="168"
                     aperture="${buoy_lateral_aperture}"
@@ -53,4 +56,5 @@
   <!-- Yellow IR emitter -->
   <xacro:ir_emitter name="${yellow_buoy_name}"
+                    parent="${link_name}"
                     code="172"
                     aperture="${10*deg2rad}"
@@ -60,4 +64,5 @@
   <!-- Halo IR emitter -->
   <xacro:ir_emitter name="${halo_name}"
+                    parent="${link_name}"
                     code="161"
                     aperture="360"

Commit message: Add inertial_sphere, remove duplicated inertial_dummy and add in2m convertion

File: irobot_create_description/urdf/common_properties.urdf.xacro (robot description, xacro)
@@ -30,6 +30,11 @@
     </xacro:inertial_cylinder_with_pose>
   </xacro:macro>
-  <xacro:macro name="inertial_dummy">
-    <xacro:inertial_cuboid mass="0.01" x="0.01" y="0.01" z="0.01"/>
+  <xacro:macro name="inertial_sphere" params="mass diameter">
+    <inertial>
+      <mass value="${mass}" />
+      <inertia ixx="${(2/5) * mass * ( (diameter*0.5) * (diameter*0.5) )}" ixy="0.0" ixz="0.0"
+	             iyy="${(2/5) * mass * ( (diameter*0.5) * (diameter*0.5) )}" iyz="0.0"
+	             izz="${(2/5) * mass * ( (diameter*0.5) * (diameter*0.5) )}" />
+    </inertial>
   </xacro:macro>
   <xacro:macro name="inertial_dummy">
@@ -39,4 +44,5 @@
   <xacro:property name="cm2m"    value="${1/100.0}"/>
   <xacro:property name="mm2m"    value="${1/1000.0}"/>
+  <xacro:property name="in2m"    value="0.0254"/>
   <xacro:property name="deg2rad" value="${pi/180.0}"/>
   <!-- Material colors -->
