Commit message: Adds diffdrive controller (#4)
* diffdrive control package

* removes unnecessary dependency

* Adds missing dependencies

* code cleanup

* comment hard to understand code

* address review comments

* updates control.yaml

* included into irobot_create_gazebo and launched from there

* fix flake 8 erros

* applies 'safety enabled' controller parameters to robot

* uses joint_state_publisher instead of joint_state_publisher_gui

* Address comments

* doubled the cmd_vel_timeout

* republish node

* Address comments

* Adds QoS parameter

* Add resource directory

* creates irobot_create_toolbox package

* changes order of node execution

* same name convention to variables

* correct flake8 errors

* more flake 8 fixes

* new line at end of gitignore

* flake8

* flake8

* replace subscription by underscore

* rename QoS to qos

* add dependency rcl_interfaces

* add test_depends

* get qos and message type by inspecting publisher

* adds uncrustify

* fix flake 8

* updates .gitignore

* check_published_topic moved to init

* Adds the correct version of uncrustify and makes republisher output debug.

* Fix merge conflicts

* Fix uncrustify failures

* Update irobot_create_toolbox/irobot_create_toolbox/topic_republisher.py

Co-authored-by: Emiliano Borghi <creativa_eborghi@irobot.com>

* Add comments to explain functionality

* removes uncrustify because collides with clang_format

* Obtain qos and msg_type from subscriber

* Adds docstrings

* Subscription instead of subscriber

* docstring how to use the tool

Co-authored-by: Emiliano Borghi <creativa_eborghi@irobot.com>

File: irobot_create_description/urdf/wheel.urdf.xacro (robot description, xacro)
@@ -34,4 +34,12 @@
     <material>Gazebo/DarkGrey</material>
   </gazebo>
+  <ros2_control name="${name}_wheel_system" type="system">
+      <hardware>
+        <plugin>gazebo_ros2_control/GazeboSystem</plugin>
+      </hardware>
+      <joint name="wheel_${name}_joint">
+        <command_interface name="velocity" />
+      </joint>
+  </ros2_control>
 </xacro:macro>
 </robot>

Commit message: Clean up wheel and wheel drops

File: irobot_create_description/urdf/wheel.urdf.xacro (robot description, xacro)
@@ -2,17 +2,19 @@
 <robot xmlns:xacro="http://ros.org/wiki/xacro">
 <xacro:macro name="wheel" params="name parent_link *origin">
-  <xacro:property name="mass_kg"   value="0.2" />
-  <xacro:property name="radius_cm" value="3.575" />
-  <xacro:property name="width_cm"  value="1.5" />
-  <joint name="wheel_${name}_joint" type="continuous">
+  <xacro:property name="mass"   value="0.2" />
+  <xacro:property name="radius" value="${3.575*cm2m}" />
+  <xacro:property name="width"  value="${1.5*cm2m}" />
+  <xacro:property name="wheel_link_name"  value="wheel_${name}"/>
+  <xacro:property name="wheel_joint_name" value="${wheel_link_name}_joint"/>
+  <joint name="${wheel_joint_name}" type="continuous">
     <parent link="${parent_link}"/>
-    <child link="wheel_${name}_link"/>
+    <child link="${wheel_link_name}"/>
     <xacro:insert_block name="origin"/>
     <axis xyz="0 0 1"/>
   </joint>
-  <link name="wheel_${name}_link">
+  <link name="${wheel_link_name}">
     <visual>
       <geometry>
-        <cylinder length="${width_cm*cm2m}" radius="${radius_cm*cm2m}"/>
+        <cylinder length="${width}" radius="${radius}"/>
       </geometry>
       <!-- Give black color to wheels in Rviz -->
@@ -21,11 +23,11 @@
     <collision>
       <geometry>
-        <cylinder length="${width_cm*cm2m}" radius="${radius_cm*cm2m}"/>
+        <cylinder length="${width}" radius="${radius}"/>
       </geometry>
     </collision>
-    <xacro:inertial_cylinder mass="${mass_kg}" radius="${radius_cm*cm2m}"
-      length="${width_cm*cm2m}" />
+    <xacro:inertial_cylinder mass="${mass}" radius="${radius}"
+      length="${width}" />
   </link>
-  <gazebo reference="wheel_${name}_link">
+  <gazebo reference="${wheel_link_name}">
     <mu1>1.0</mu1>
     <mu2>1.0</mu2>
@@ -36,12 +38,12 @@
     <material>Gazebo/DarkGrey</material>
   </gazebo>
-  <ros2_control name="${name}_wheel_system" type="system">
-      <hardware>
-        <plugin>gazebo_ros2_control/GazeboSystem</plugin>
-      </hardware>
-      <joint name="wheel_${name}_joint">
-        <state_interface name="position" />
-        <command_interface name="velocity" />
-      </joint>
+  <ros2_control name="${wheel_link_name}_controller" type="system">
+    <hardware>
+      <plugin>gazebo_ros2_control/GazeboSystem</plugin>
+    </hardware>
+    <joint name="${wheel_joint_name}">
+      <state_interface name="position" />
+      <command_interface name="velocity" />
+    </joint>
   </ros2_control>
 </xacro:macro>

File: irobot_create_description/urdf/wheel_with_wheeldrop.urdf.xacro (robot description, xacro)
@@ -9,5 +9,5 @@
   </xacro:wheel_drop>
   <!-- Wheel definition -->
-  <xacro:wheel name="${name}" parent_link="wheel_${name}_axle_link">
+  <xacro:wheel name="${name}" parent_link="wheel_drop_${name}">
     <origin xyz="0 0 0" rpy="0 0 0"/>
   </xacro:wheel>

Commit message: Rename wheel joint and link

File: irobot_create_description/urdf/wheel.urdf.xacro (robot description, xacro)
@@ -5,5 +5,5 @@
   <xacro:property name="radius" value="${3.575*cm2m}" />
   <xacro:property name="width"  value="${1.5*cm2m}" />
-  <xacro:property name="wheel_link_name"  value="wheel_${name}"/>
+  <xacro:property name="wheel_link_name"  value="${name}_wheel"/>
   <xacro:property name="wheel_joint_name" value="${wheel_link_name}_joint"/>
   <joint name="${wheel_joint_name}" type="continuous">
