Commit message: Removes extra comments

File: irobot_create_description/urdf/button.urdf.xacro (robot description, xacro)
@@ -7,7 +7,5 @@
     <xacro:insert_block name="origin"/>
   </joint>
-  <link name="${name}">
-    <!-- <xacro:inertial_dummy/> -->
-  </link>
+  <link name="${name}"/>
 </xacro:macro>
 </robot>

File: irobot_create_description/urdf/create3.urdf.xacro (robot description, xacro)
@@ -45,5 +45,4 @@
   </link>
   <!-- Bumper -->
-  <!-- name="bump_front_center" -->
   <xacro:bumper
       visual_mesh="file://$(find irobot_create_description)/meshes/bumper_visual.dae"
