Commit message: Address comments

File: irobot_create_description/urdf/bumper.urdf.xacro (robot description, xacro)
@@ -2,11 +2,9 @@
 <robot xmlns:xacro="http://ros.org/wiki/xacro">
 <xacro:macro name="bumper" params="name:=bumper parent_link robot_type visual_mesh collision_mesh
-                                          *origin *inertial">
+  *origin *inertial">
   <joint name="${name}_joint" type="fixed">
     <parent link="${parent_link}"/>
     <child link="${name}_link"/>
-    <axis xyz="0 1 0"/>
     <xacro:insert_block name="origin"/>
-    <limit lower="0" upper="0" velocity="0.01" effort="30"/>
   </joint>
   <link name="${name}_link">
@@ -29,5 +27,4 @@
     <minDepth>0.001</minDepth>
     <maxContacts>10</maxContacts>
-    <material>Gazebo/Green</material>
   </gazebo>
   <gazebo reference="${name}_joint">

File: irobot_create_description/urdf/common_properties.urdf.xacro (robot description, xacro)
@@ -7,6 +7,6 @@
       <origin xyz="0 0 0" />
       <inertia ixx="${(1/12) * mass * (y*y + z*z)}" ixy="0.0" ixz="0.0"
-	iyy="${(1/12) * mass * (x*x + z*z)}" iyz="0.0"
-	izz="${(1/12) * mass * (x*x + y*y)}" />
+        iyy="${(1/12) * mass * (x*x + z*z)}" iyz="0.0"
+        izz="${(1/12) * mass * (x*x + y*y)}" />
     </inertial>
   </xacro:macro>
@@ -16,6 +16,6 @@
       <origin xyz="0 0 0" />
       <inertia ixx="${(1/12) * mass * (3*radius*radius + length*length)}" ixy="0.0" ixz="0.0"
-	iyy="${(1/12) * mass * (3*radius*radius + length*length)}" iyz="0.0"
-	izz="${(1/2) * mass * (radius*radius)}" />
+        iyy="${(1/12) * mass * (3*radius*radius + length*length)}" iyz="0.0"
+        izz="${(1/2) * mass * (radius*radius)}" />
     </inertial>
   </xacro:macro>
@@ -25,6 +25,6 @@
       <mass value="${mass}" />
       <inertia ixx="${(1/12) * mass * (3*radius*radius + length*length)}" ixy="0.0" ixz="0.0"
-	iyy="${(1/12) * mass * (3*radius*radius + length*length)}" iyz="0.0"
-	izz="${(1/2) * mass * (radius*radius)}" />
+        iyy="${(1/12) * mass * (3*radius*radius + length*length)}" iyz="0.0"
+        izz="${(1/2) * mass * (radius*radius)}" />
     </inertial>
   </xacro:macro>

File: irobot_create_description/urdf/create3.urdf.xacro (robot description, xacro)
@@ -6,15 +6,15 @@
   <xacro:include filename="$(find irobot_create_description)/urdf/caster.urdf.xacro" />
   <!-- MECHANICAL PROPERTIES -->
-  <xacro:property name="body_z_offset" value="-0.025" /><!-- z offset from ground [m] -->
-  <xacro:property name="body_mass" value="2.300" />
-  <xacro:property name="body_radius" value="0.16" />
-  <xacro:property name="body_length" value="0.048" />
-  <xacro:property name="bumper_mass" value="0.1" /> <!-- [kg] -->
-  <xacro:property name="bumper_offset_z" value="-0.025" /><!-- [m] -->
-  <xacro:property name="wheel_height" value="-0.0275" /><!-- z [m] -->
-  <xacro:property name="distance_between_wheels" value="0.233" /><!-- y [m] -->
-  <xacro:property name="caster_position_x" value="0.125" /><!-- x [m] -->
-  <xacro:property name="caster_position_y" value="0" /><!-- y [m] -->
-  <xacro:property name="caster_position_z" value="-0.054" /><!-- z [m] -->
+  <xacro:property name="body_z_offset"           value="-0.025" />  <!-- z offset from ground [m] -->
+  <xacro:property name="body_mass"               value="2.300" />   <!-- [kg] -->
+  <xacro:property name="body_radius"             value="0.16" />    <!-- [m] -->
+  <xacro:property name="body_length"             value="0.048" />   <!-- [m] -->
+  <xacro:property name="bumper_mass"             value="0.1" />     <!-- [kg] -->
+  <xacro:property name="bumper_offset_z"         value="-0.025" />  <!-- [m] -->
+  <xacro:property name="wheel_height"            value="-0.0275" /> <!-- z [m] -->
+  <xacro:property name="distance_between_wheels" value="0.233" />   <!-- y [m] -->
+  <xacro:property name="caster_position_x"       value="0.125" />   <!-- x [m] -->
+  <xacro:property name="caster_position_y"       value="0" />       <!-- y [m] -->
+  <xacro:property name="caster_position_z"       value="-0.054" />  <!-- z [m] -->
   <!-- Create 3 base definitions-->
   <link name="base_footprint"/>
@@ -31,5 +31,5 @@
     </visual>
     <collision name="create3_base_collision">
-      <origin xyz="-0.005 0 ${(body_z_offset/2.) + 0.01}"/>
+      <origin xyz="-0.005 0 ${body_z_offset/2.}"/>
       <geometry>
         <cylinder length="${body_length}" radius="${body_radius}"/>
@@ -50,8 +50,9 @@
       <origin xyz="0.08 0 ${bumper_offset_z}"/>
       <mass value="${bumper_mass}"/>
-      <inertia ixx="0.0013483753405" ixy="0.0000000454352" ixz="0.0000014434849" iyy="0.0002521736852" iyz="-0.0000000006721" izz="0.0015442525386"/>
+      <inertia ixx="0.0013483753405" ixy="0.0000000454352" ixz="0.0000014434849" iyy="0.0002521736852"
+        iyz="-0.0000000006721" izz="0.0015442525386"/>
     </inertial>
   </xacro:bumper>
-  <!-- Wheel with mechanical wheel drop -->
+  <!-- Wheels with mechanical wheel drop -->
   <xacro:wheel_with_wheeldrop name="left" parent_link="base_link">
     <origin xyz="0 ${distance_between_wheels/2} ${wheel_height}" rpy="${-pi/2} 0 0"/>

File: irobot_create_description/urdf/wheel.urdf.xacro (robot description, xacro)
@@ -2,7 +2,7 @@
 <robot xmlns:xacro="http://ros.org/wiki/xacro">
 <xacro:macro name="wheel" params="name parent_link *origin">
-  <xacro:property name="wheel_mass"   value="0.2" /> <!-- [kg] -->
-  <xacro:property name="wheel_radius" value="0.03575" /> <!-- [m] -->
-  <xacro:property name="wheel_width"  value="0.015" /> <!-- [m] -->
+  <xacro:property name="wheel_mass"   value="0.2" />      <!-- [kg] -->
+  <xacro:property name="wheel_radius" value="0.03575" />  <!-- [m] -->
+  <xacro:property name="wheel_width"  value="0.015" />    <!-- [m] -->
   <joint name="wheel_${name}_joint" type="continuous">
     <parent link="${parent_link}"/>
@@ -14,5 +14,5 @@
     <visual>
       <geometry>
-          <cylinder length="${wheel_width}" radius="${wheel_radius}"/>
+        <cylinder length="${wheel_width}" radius="${wheel_radius}"/>
       </geometry>
     </visual>

File: irobot_create_description/urdf/wheel_with_wheeldrop.urdf.xacro (robot description, xacro)
@@ -17,8 +17,5 @@
   </gazebo>
   <link name="wheel_${name}_axle_link">
-      <xacro:inertial_cuboid mass="0.05"
-                             x="0.15"
-                             y="0.15"
-                             z="0.15"/>
+    <xacro:inertial_cuboid mass="0.05" x="0.15" y="0.15" z="0.15"/>
   </link>
   <!-- Wheel definition -->

Commit message: Reformats xacro files and simplifies CMakeLists

File: irobot_create_description/urdf/bumper.urdf.xacro (robot description, xacro)
@@ -22,4 +22,5 @@
   </link>
   <gazebo reference="${name}_link" >
+    <material>Gazebo/Green</material>
     <mu1>0.1</mu1>
     <mu2>0.1</mu2>

File: irobot_create_description/urdf/caster.urdf.xacro (robot description, xacro)
@@ -2,5 +2,5 @@
 <robot xmlns:xacro="http://ros.org/wiki/xacro">
 <xacro:macro name="caster" params="name parent_link *origin">
-  <xacro:property name="radius" value="0.01" /> <!-- [m] -->
+  <xacro:property name="radius_cm" value="1" />
   <joint name="${name}_joint" type="fixed">
     <parent link="${parent_link}"/>
@@ -11,10 +11,10 @@
     <visual>
       <geometry>
-        <sphere radius="${radius}"/>
+        <sphere radius="${radius_cm*cm2m}"/>
       </geometry>
     </visual>
     <collision>
       <geometry>
-        <sphere radius="${radius}"/>
+        <sphere radius="${radius_cm*cm2m}"/>
       </geometry>
     </collision>

File: irobot_create_description/urdf/common_properties.urdf.xacro (robot description, xacro)
@@ -29,3 +29,5 @@
     </inertial>
   </xacro:macro>
+  <!-- Conversion macros -->
+  <xacro:property name="cm2m"    value="${1/100.0}"/>
 </robot>

File: irobot_create_description/urdf/create3.urdf.xacro (robot description, xacro)
@@ -6,15 +6,15 @@
   <xacro:include filename="$(find irobot_create_description)/urdf/caster.urdf.xacro" />
   <!-- MECHANICAL PROPERTIES -->
-  <xacro:property name="body_z_offset"           value="-0.025" />  <!-- z offset from ground [m] -->
-  <xacro:property name="body_mass"               value="2.300" />   <!-- [kg] -->
-  <xacro:property name="body_radius"             value="0.16" />    <!-- [m] -->
-  <xacro:property name="body_length"             value="0.048" />   <!-- [m] -->
-  <xacro:property name="bumper_mass"             value="0.1" />     <!-- [kg] -->
-  <xacro:property name="bumper_offset_z"         value="-0.025" />  <!-- [m] -->
-  <xacro:property name="wheel_height"            value="-0.0275" /> <!-- z [m] -->
-  <xacro:property name="distance_between_wheels" value="0.233" />   <!-- y [m] -->
-  <xacro:property name="caster_position_x"       value="0.125" />   <!-- x [m] -->
-  <xacro:property name="caster_position_y"       value="0" />       <!-- y [m] -->
-  <xacro:property name="caster_position_z"       value="-0.054" />  <!-- z [m] -->
+  <xacro:property name="body_z_offset_cm"           value="-2.5" />
+  <xacro:property name="body_mass_kg"              value="2.300" />
+  <xacro:property name="body_radius_cm"             value="16" />
+  <xacro:property name="body_length_cm"             value="4.8" />
+  <xacro:property name="bumper_mass_kg"            value="0.1" />
+  <xacro:property name="bumper_offset_z_cm"         value="-2.5" />
+  <xacro:property name="wheel_height_cm"            value="-2.75" />
+  <xacro:property name="distance_between_wheels_cm" value="23.3" />
+  <xacro:property name="caster_position_x_cm"       value="12.5" />
+  <xacro:property name="caster_position_y_cm"       value="0" />
+  <xacro:property name="caster_position_z_cm"       value="-5.4" />
   <!-- Create 3 base definitions-->
   <link name="base_footprint"/>
@@ -25,17 +25,17 @@
   <link name="base_link">
     <visual>
-      <origin xyz="0 0 ${body_z_offset}" rpy="0 0 ${-pi*3.0/2.0}"/>
+      <origin xyz="0 0 ${body_z_offset_cm*cm2m}" rpy="0 0 ${-pi*3.0/2.0}"/>
       <geometry>
-        <mesh filename="package://irobot_create_description/meshes/body_collision.stl" scale="0.001 0.001 0.001"/>
+        <mesh filename="file://$(find irobot_create_description)/meshes/body_collision.stl" scale="0.001 0.001 0.001"/>
       </geometry>
     </visual>
     <collision name="create3_base_collision">
-      <origin xyz="-0.005 0 ${body_z_offset/2.}"/>
+      <origin xyz="-0.005 0 ${body_z_offset_cm*cm2m/2.}"/>
       <geometry>
-        <cylinder length="${body_length}" radius="${body_radius}"/>
+        <cylinder length="${body_length_cm*cm2m}" radius="${body_radius_cm*cm2m}"/>
       </geometry>
     </collision>
-    <xacro:inertial_cylinder_with_pose mass="${body_mass}" radius="${body_radius}" length="${body_length}">
-      <origin xyz="0 0 ${body_z_offset - 0.02}"/>
+    <xacro:inertial_cylinder_with_pose mass="${body_mass_kg}" radius="${body_radius_cm*cm2m}" length="${body_length_cm*cm2m}">
+      <origin xyz="0 0 ${body_z_offset_cm*cm2m}"/>
     </xacro:inertial_cylinder_with_pose>
   </link>
@@ -44,24 +44,25 @@
       parent_link="base_link"
       robot_type="create3"
-      visual_mesh="package://irobot_create_description/meshes/bumper_collision.stl"
-      collision_mesh="package://irobot_create_description/meshes/bumper_collision.stl">
-    <origin xyz="0 0 ${bumper_offset_z}"/>
+      visual_mesh="file://$(find irobot_create_description)/meshes/bumper_collision.stl"
+      collision_mesh="file://$(find irobot_create_description)/meshes/bumper_collision.stl">
+    <origin xyz="0 0 ${bumper_offset_z_cm*cm2m}"/>
     <inertial>
-      <origin xyz="0.08 0 ${bumper_offset_z}"/>
-      <mass value="${bumper_mass}"/>
-      <inertia ixx="0.0013483753405" ixy="0.0000000454352" ixz="0.0000014434849" iyy="0.0002521736852"
-        iyz="-0.0000000006721" izz="0.0015442525386"/>
-    </inertial>
+        <origin xyz="0.08 0 ${bumper_offset_z_cm*cm2m}"/>
+        <mass value="${bumper_mass_kg}"/>
+        <inertia ixx="0.0013483753405" ixy="0.0000000454352" ixz="0.0000014434849" iyy="0.0002521736852"
+          iyz="-0.0000000006721" izz="0.0015442525386"/>
+      </inertial>
   </xacro:bumper>
   <!-- Wheels with mechanical wheel drop -->
   <xacro:wheel_with_wheeldrop name="left" parent_link="base_link">
-    <origin xyz="0 ${distance_between_wheels/2} ${wheel_height}" rpy="${-pi/2} 0 0"/>
+    <origin xyz="0 ${distance_between_wheels_cm*cm2m/2} ${wheel_height_cm*cm2m}" rpy="${-pi/2} 0 0"/>
   </xacro:wheel_with_wheeldrop>
   <xacro:wheel_with_wheeldrop name="right" parent_link="base_link">
-    <origin xyz="0 ${-distance_between_wheels/2} ${wheel_height}" rpy="${-pi/2} 0 0"/>
+    <origin xyz="0 ${-distance_between_wheels_cm*cm2m/2} ${wheel_height_cm*cm2m}" rpy="${-pi/2} 0 0"/>
   </xacro:wheel_with_wheeldrop>
   <!-- Caster wheel -->
   <xacro:caster name="front_caster" parent_link="base_link">
-    <origin xyz="${caster_position_x} ${caster_position_y} ${caster_position_z}" rpy="${-pi/2} 0 0"/>
+    <origin xyz="${caster_position_x_cm*cm2m} ${caster_position_y_cm*cm2m} ${caster_position_z_cm*cm2m}"
+      rpy="${-pi/2} 0 0"/>
   </xacro:caster>
 </robot>

File: irobot_create_description/urdf/wheel.urdf.xacro (robot description, xacro)
@@ -2,7 +2,7 @@
 <robot xmlns:xacro="http://ros.org/wiki/xacro">
 <xacro:macro name="wheel" params="name parent_link *origin">
-  <xacro:property name="wheel_mass"   value="0.2" />      <!-- [kg] -->
-  <xacro:property name="wheel_radius" value="0.03575" />  <!-- [m] -->
-  <xacro:property name="wheel_width"  value="0.015" />    <!-- [m] -->
+  <xacro:property name="wheel_mass_kg"   value="0.2" />
+  <xacro:property name="wheel_radius_cm" value="3.575" />
+  <xacro:property name="wheel_width_cm"  value="1.5" />
   <joint name="wheel_${name}_joint" type="continuous">
     <parent link="${parent_link}"/>
@@ -14,13 +14,14 @@
     <visual>
       <geometry>
-        <cylinder length="${wheel_width}" radius="${wheel_radius}"/>
+        <cylinder length="${wheel_width_cm*cm2m}" radius="${wheel_radius_cm*cm2m}"/>
       </geometry>
     </visual>
     <collision>
       <geometry>
-        <cylinder length="${wheel_width}" radius="${wheel_radius}"/>
+        <cylinder length="${wheel_width_cm*cm2m}" radius="${wheel_radius_cm*cm2m}"/>
       </geometry>
     </collision>
-    <xacro:inertial_cylinder mass="${wheel_mass}" radius="${wheel_radius}" length="${wheel_width}" />
+    <xacro:inertial_cylinder mass="${wheel_mass_kg}" radius="${wheel_radius_cm*cm2m}"
+      length="${wheel_width_cm*cm2m}" />
   </link>
   <gazebo reference="wheel_${name}_link">

Commit message: Updated colors for models in gazebo

File: irobot_create_description/urdf/bumper.urdf.xacro (robot description, xacro)
@@ -22,5 +22,4 @@
   </link>
   <gazebo reference="${name}_link" >
-    <material>Gazebo/Green</material>
     <mu1>0.1</mu1>
     <mu2>0.1</mu2>
@@ -28,4 +27,5 @@
     <minDepth>0.001</minDepth>
     <maxContacts>10</maxContacts>
+    <material>Gazebo/DarkGrey</material>
   </gazebo>
   <gazebo reference="${name}_joint">

File: irobot_create_description/urdf/caster.urdf.xacro (robot description, xacro)
@@ -21,5 +21,5 @@
   </link>
   <gazebo reference="${name}_link">
-    <material>Gazebo/Grey</material>
+    <material>Gazebo/DarkGrey</material>
   </gazebo>
 </xacro:macro>

File: irobot_create_description/urdf/wheel.urdf.xacro (robot description, xacro)
@@ -32,5 +32,5 @@
     <minDepth>0.0001</minDepth>
     <maxVel>1.0</maxVel>
-    <material>Gazebo/Grey</material>
+    <material>Gazebo/DarkGrey</material>
   </gazebo>
 </xacro:macro>

Commit message: rename optical mouse in xacros

File: irobot_create_description/urdf/bumper.urdf.xacro (robot description, xacro)
@@ -1,5 +1,5 @@
 <?xml version="1.0"?>
 <robot xmlns:xacro="http://ros.org/wiki/xacro">
-<xacro:macro name="bumper" params="name:=bumper parent_link robot_type visual_mesh collision_mesh
+<xacro:macro name="bumper" params="name:=bumper parent_link visual_mesh collision_mesh
   *origin *inertial">
   <joint name="${name}_joint" type="fixed">

File: irobot_create_description/urdf/create3.urdf.xacro (robot description, xacro)
@@ -4,5 +4,5 @@
   <xacro:include filename="$(find irobot_create_description)/urdf/caster.urdf.xacro" />
   <xacro:include filename="$(find irobot_create_description)/urdf/common_properties.urdf.xacro"/>
-  <xacro:include filename="$(find irobot_create_description)/urdf/sensors/optical_mouse.urdf.xacro"/>
+  <xacro:include filename="$(find irobot_create_description)/urdf/sensors/mouse.urdf.xacro"/>
   <xacro:include filename="$(find irobot_create_description)/urdf/wheel_with_wheeldrop.urdf.xacro" />
   <!-- MECHANICAL PROPERTIES -->
@@ -22,4 +22,5 @@
   <xacro:property name="inertial_offset_x_cm"       value="1" />
   <xacro:property name="wheel_drop_offset_z_mm"     value="3.5"/>
+  <xacro:property name="wheel_drop_z"               value="${wheel_height_cm*cm2m + wheel_drop_offset_z_mm*mm2m}"/>
   <xacro:property name="mouse_update_rate"          value="62" />
   <!-- Create 3 base definitions-->
@@ -50,5 +51,4 @@
   <xacro:bumper
       parent_link="base_link"
-      robot_type="create3"
       visual_mesh="file://$(find irobot_create_description)/meshes/bumper_visual.dae"
       collision_mesh="file://$(find irobot_create_description)/meshes/bumper_collision.dae">
@@ -62,5 +62,4 @@
   </xacro:bumper>
   <!-- Wheels with mechanical wheel drop -->
-  <xacro:property name="wheel_drop_z" value="${wheel_height_cm*cm2m + wheel_drop_offset_z_mm*mm2m}"/>
   <xacro:wheel_with_wheeldrop name="left">
     <origin xyz="0 ${distance_between_wheels_cm*cm2m/2} ${wheel_drop_z}" rpy="${-pi/2} 0 0"/>
@@ -80,12 +79,9 @@
   </gazebo>
   <!-- Optical mouse -->
-  <xacro:optical_mouse name="optical_mouse"
-                      parent="base_link"
-                      ros_topic="optical_mouse"
-                      visualize="true"
-                      noise_mean="0.0"
-                      noise_var="0.0"
-                      mouse_seed="0.0" update_rate="${mouse_update_rate}">
-  <origin xyz="0.1015 0.087 -0.055" rpy="0 0 ${-pi/4}"/>
-</xacro:optical_mouse>
+  <xacro:mouse
+      parent_link="base_link"
+      mouse_seed="0.0"
+      update_rate="${mouse_update_rate}">
+    <origin xyz="0.1015 0.087 -0.055" rpy="0 0 ${-pi/4}"/>
+  </xacro:mouse>
 </robot>

File: irobot_create_description/urdf/sensors/mouse.urdf.xacro (robot description, xacro)
@@ -1,6 +1,6 @@
 <?xml version="1.0"?>
 <robot xmlns:xacro="http://ros.org/wiki/xacro">
-  <xacro:macro name="optical_mouse" params="name parent *origin ros_topic visualize noise_mean:=0
-                                            noise_var:=0 mouse_seed update_rate" >
+  <xacro:macro name="mouse" params="name:=mouse parent_link *origin visualize:=true noise_mean:=0.0
+                                            noise_var:=0.0 mouse_seed:=0.0 update_rate" >
     <!-- Sensor settings -->
     <xacro:property name="mass" value="0.1" />
@@ -9,10 +9,10 @@
     <!-- Visualization settings -->
     <xacro:property name="color" value="Red" />
-    <joint name="optical_mouse_joint" type="fixed">
+    <joint name="mouse_joint" type="fixed">
       <xacro:insert_block name="origin"/>
-      <parent link="${parent}"/>
-      <child link="optical_mouse_${name}_link"/>
+      <parent link="${parent_link}"/>
+      <child link="${name}"/>
     </joint>
-    <link name="optical_mouse_${name}_link">
+    <link name="${name}">
       <xacro:if value="${visualize}">
         <visual>
@@ -30,5 +30,5 @@
         </ros>
         <update_rate>${update_rate}</update_rate>
-        <link>optical_mouse_${name}_link</link>
+        <link>${name}</link>
         <gaussian_mean>${noise_mean}</gaussian_mean>
         <gaussian_var>${noise_var}</gaussian_var>
@@ -39,8 +39,8 @@
       </plugin>
     </gazebo>
-    <gazebo reference="optical_mouse_${name}_link" >
+    <gazebo reference="o${name}" >
       <material>Gazebo/${color}</material>
     </gazebo>
-    <gazebo reference="optical_mouse_joint" >
+    <gazebo reference="mouse_joint" >
       <preserveFixedJoint>true</preserveFixedJoint>
     </gazebo>

Commit message: Added bumper plugin

File: irobot_create_description/urdf/bumper.urdf.xacro (robot description, xacro)
@@ -28,4 +28,12 @@
     <maxContacts>10</maxContacts>
     <material>Gazebo/DarkGrey</material>
+    <sensor name='${name}_contact_sensor' type='contact'>
+      <always_on>true</always_on>
+      <update_rate>62</update_rate>
+      <contact>
+        <collision>${name}_link_collision</collision>
+      </contact>
+      <plugin name="bumper_controller" filename="libgazebo_ros_irobot_bumper.so"/>
+    </sensor>
   </gazebo>
   <gazebo reference="${name}_joint">

Commit message: Addressed peer review comments

File: irobot_create_description/urdf/bumper.urdf.xacro (robot description, xacro)
@@ -1,5 +1,5 @@
 <?xml version="1.0"?>
 <robot xmlns:xacro="http://ros.org/wiki/xacro">
-<xacro:macro name="bumper" params="name:=bumper parent_link visual_mesh collision_mesh
+<xacro:macro name="bumper" params="name:=bumper parent_link update_rate:=62.0 visual_mesh collision_mesh
   *origin *inertial">
   <joint name="${name}_joint" type="fixed">
@@ -30,5 +30,5 @@
     <sensor name='${name}_contact_sensor' type='contact'>
       <always_on>true</always_on>
-      <update_rate>62</update_rate>
+      <update_rate>${update_rate}</update_rate>
       <contact>
         <collision>${name}_link_collision</collision>

Commit message: Implement bumper contact sensor (#15)
* Added bumper plugin

* Fixed rebase-related problems

* Fixed github actions failures

* Remove unnecessary identifier from log's msg

* Addressed peer review comments

* Removed log directory from commits

* Addressed Rodri's comments

* Applied ament-clang-format fixes

* Updated iterator with find_if

* Make clang format happy again

* Adressed peer review comments

* Addressed peer review comments

* Use find_if everywhere

* Update topic name

* Applied clang format fixes

* Addressed peer review comments

* Fix typo

File: irobot_create_description/urdf/bumper.urdf.xacro (robot description, xacro)
@@ -1,5 +1,5 @@
 <?xml version="1.0"?>
 <robot xmlns:xacro="http://ros.org/wiki/xacro">
-<xacro:macro name="bumper" params="name:=bumper parent_link visual_mesh collision_mesh
+<xacro:macro name="bumper" params="name:=bumper parent_link update_rate:=62.0 visual_mesh collision_mesh
   *origin *inertial">
   <joint name="${name}_joint" type="fixed">
@@ -28,4 +28,17 @@
     <maxContacts>10</maxContacts>
     <material>Gazebo/DarkGrey</material>
+    <sensor name='${name}_contact_sensor' type='contact'>
+      <always_on>true</always_on>
+      <update_rate>${update_rate}</update_rate>
+      <contact>
+        <collision>${name}_link_collision</collision>
+      </contact>
+      <plugin name="${name}_plugin" filename="libgazebo_ros_create_bumper.so">
+        <ros>
+          <namespace>/</namespace>
+          <remapping>~/out:=bumper/event</remapping>
+        </ros>
+      </plugin>
+    </sensor>
   </gazebo>
   <gazebo reference="${name}_joint">
