Commit message: Rename tf frames to match the real robot model

File: irobot_create_description/urdf/bumper.urdf.xacro (robot description, xacro)
@@ -1,12 +1,27 @@
 <?xml version="1.0"?>
 <robot xmlns:xacro="http://ros.org/wiki/xacro">
-<xacro:macro name="bumper" params="name:=bumper parent_link update_rate:=62.0 visual_mesh collision_mesh
+<!--
+  The robot has 5 bumper sensors in the front but for the simulation
+  only the center one is being used, so the remaining 4 bumpers are
+  created as 'dummy bumpers'.
+ -->
+<xacro:macro name="dummy_bumper" params="name parent_link:=base_link *origin">
+  <joint name="${name}_joint" type="fixed">
+    <parent link="${parent_link}"/>
+    <child link="${name}"/>
+    <xacro:insert_block name="origin"/>
+  </joint>
+  <link name="${name}">
+    <xacro:inertial_dummy/>
+  </link>
+</xacro:macro>
+<xacro:macro name="bumper" params="name parent_link:=base_link update_rate:=62.0 visual_mesh collision_mesh
   *origin *inertial">
   <joint name="${name}_joint" type="fixed">
     <parent link="${parent_link}"/>
-    <child link="${name}_link"/>
+    <child link="${name}"/>
     <xacro:insert_block name="origin"/>
   </joint>
-  <link name="${name}_link">
+  <link name="${name}">
     <visual>
       <geometry>
@@ -21,5 +36,5 @@
     <xacro:insert_block name="inertial"/>
   </link>
-  <gazebo reference="${name}_link" >
+  <gazebo reference="${name}" >
     <mu1>0.1</mu1>
     <mu2>0.1</mu2>
@@ -45,4 +60,20 @@
     <preserveFixedJoint>true</preserveFixedJoint>
   </gazebo>
+  <xacro:dummy_bumper
+      name="bump_front_left">
+      <origin xyz="0.02345 -0.0875 0.025" rpy="0 0 0.5235985"/>
+  </xacro:dummy_bumper>
+  <xacro:dummy_bumper
+      name="bump_front_right">
+      <origin xyz="0.02345 0.0875 0.025" rpy="0 0 -0.5235985"/>
+  </xacro:dummy_bumper>
+  <xacro:dummy_bumper
+      name="bump_left">
+      <origin xyz="0.0875 -0.15155 0.025" rpy="0 0 1.047193"/>
+  </xacro:dummy_bumper>
+  <xacro:dummy_bumper
+      name="bump_right">
+      <origin xyz="0.0875 0.15155 0.025" rpy="0 0 -1.047193"/>
+  </xacro:dummy_bumper>
 </xacro:macro>
 </robot>

File: irobot_create_description/urdf/create3.urdf.xacro (robot description, xacro)
@@ -2,4 +2,5 @@
 <robot name="create3" xmlns:xacro="http://ros.org/wiki/xacro">
   <xacro:include filename="$(find irobot_create_description)/urdf/bumper.urdf.xacro" />
+  <xacro:include filename="$(find irobot_create_description)/urdf/button.urdf.xacro" />
   <xacro:include filename="$(find irobot_create_description)/urdf/caster.urdf.xacro" />
   <xacro:include filename="$(find irobot_create_description)/urdf/common_properties.urdf.xacro"/>
@@ -10,26 +11,20 @@
   <xacro:include filename="$(find irobot_create_description)/urdf/wheel_with_wheeldrop.urdf.xacro" />
   <!-- MECHANICAL PROPERTIES -->
-  <xacro:property name="body_z_offset"           value="${-2.5*cm2m}" />
-  <xacro:property name="body_collision_z_offset" value="${-1*cm2m}" />
+  <xacro:property name="body_z_offset"           value="${4.1*cm2m}" />
+  <xacro:property name="body_collision_z_offset" value="${1*cm2m}" />
   <xacro:property name="body_mass"               value="2.300" />
   <xacro:property name="body_radius"             value="${16.4*cm2m}" />
   <xacro:property name="body_length"             value="${6*cm2m}" />
   <xacro:property name="bumper_mass"             value="0.1" />
-  <xacro:property name="bumper_offset_z"         value="${-2.5*cm2m}" />
+  <xacro:property name="bumper_offset_z"         value="${4.1*cm2m}" />
   <xacro:property name="bumber_inertial_x"       value="${8*cm2m}" />
   <xacro:property name="bumper_inertial_z"       value="${2*cm2m}"/>
-  <xacro:property name="wheel_height"            value="${-2.75*cm2m}" />
+  <xacro:property name="wheel_height"            value="${3.85*cm2m}" />
   <xacro:property name="distance_between_wheels" value="${23.3*cm2m}" />
   <xacro:property name="caster_position_x"       value="${12.5*cm2m}" />
-  <xacro:property name="caster_position_z"       value="${-5.4*cm2m}" />
-  <xacro:property name="wheel_drop_offset_z"     value="${3.5*mm2m}"/>
+  <xacro:property name="caster_position_z"       value="${1.2*cm2m}" />
+  <xacro:property name="wheel_drop_offset_z"     value="${3.1*mm2m}"/>
   <xacro:property name="wheel_drop_z"            value="${wheel_height + wheel_drop_offset_z}"/>
-  <!-- Create 3 base definitions-->
-  <link name="base_footprint"/>
-  <joint name="base_footprint_joint" type="fixed">
-    <origin xyz="0 0 0.066" rpy="0 0.013 0"/>
-    <parent link="base_footprint"/>
-    <child link="base_link" />
-  </joint>
+  <!-- Create 3 base definition-->
   <link name="base_link">
     <visual>
@@ -40,5 +35,5 @@
     </visual>
     <collision name="create3_base_collision">
-      <origin xyz="0 0 ${body_collision_z_offset}" rpy="0 0 ${pi/2}"/>
+      <origin xyz="0 0 ${body_z_offset + body_collision_z_offset}" rpy="0 0 ${pi/2}"/>
       <geometry>
         <cylinder length="${body_length}" radius="${body_radius}"/>
@@ -51,5 +46,5 @@
   <!-- Bumper -->
   <xacro:bumper
-      parent_link="base_link"
+      name="bump_front_center"
       visual_mesh="file://$(find irobot_create_description)/meshes/bumper_visual.dae"
       collision_mesh="file://$(find irobot_create_description)/meshes/bumper_collision.dae">
@@ -71,5 +66,5 @@
   <!-- Caster wheel -->
   <xacro:caster name="front_caster" parent_link="base_link">
-    <origin xyz="${caster_position_x} 0 ${caster_position_z}" rpy="${-pi/2} 0 0"/>
+    <origin xyz="${caster_position_x} 0 ${caster_position_z}" rpy="${-pi/2} ${pi} 0"/>
   </xacro:caster>
   <!-- IMU -->
@@ -148,3 +143,16 @@
     <origin xyz="0.0399 0.1488 ${ir_intensity_z_pos}" rpy="0 0 1.309"/>
   </xacro:ir_intensity>
+  <!-- Buttons -->
+  <xacro:button
+      name="button_1">
+      <origin xyz="0.06 0.37 0.08" rpy="0 -1.5707963 0"/>
+  </xacro:button>
+  <xacro:button
+      name="button_2">
+      <origin xyz="0.06 -0.37 0.08" rpy="0 -1.5707963 0"/>
+  </xacro:button>
+  <xacro:button
+      name="button_power">
+      <origin xyz="0.06 0 0.08" rpy="0 -1.5707963 0"/>
+  </xacro:button>
 </robot>

File: irobot_create_description/urdf/wheel.urdf.xacro (robot description, xacro)
@@ -5,5 +5,5 @@
   <xacro:property name="radius" value="${3.575*cm2m}" />
   <xacro:property name="width"  value="${1.5*cm2m}" />
-  <xacro:property name="wheel_link_name"  value="${name}_wheel"/>
+  <xacro:property name="wheel_link_name"  value="_${name}_wheel"/>
   <xacro:property name="wheel_joint_name" value="${wheel_link_name}_joint"/>
   <joint name="${wheel_joint_name}" type="continuous">

File: irobot_create_description/urdf/wheel_drop.urdf.xacro (robot description, xacro)
@@ -8,5 +8,5 @@
   <xacro:property name="wd_mass" value="0.05"/>
   <xacro:property name="update_rate"   value="62" />
-  <xacro:property name="wd_link_name"  value="wheel_drop_${name}"/>
+  <xacro:property name="wd_link_name"  value="${name}_wheel"/>
   <xacro:property name="wd_joint_name" value="${wd_link_name}_joint"/>
   <joint name="${wd_joint_name}" type="prismatic">

File: irobot_create_description/urdf/wheel_with_wheeldrop.urdf.xacro (robot description, xacro)
@@ -9,5 +9,5 @@
   </xacro:wheel_drop>
   <!-- Wheel definition -->
-  <xacro:wheel name="${name}" parent_link="wheel_drop_${name}">
+  <xacro:wheel name="${name}" parent_link="${name}_wheel">
     <origin xyz="0 0 0" rpy="0 0 0"/>
   </xacro:wheel>

Commit message: Addressed comments.

File: irobot_create_description/urdf/bumper.urdf.xacro (robot description, xacro)
@@ -1,27 +1,26 @@
 <?xml version="1.0"?>
 <robot xmlns:xacro="http://ros.org/wiki/xacro">
-<!--
-  The robot has 5 bumper sensors in the front but for the simulation
-  only the center one is being used, so the remaining 4 bumpers are
-  created as 'dummy bumpers'.
- -->
-<xacro:macro name="dummy_bumper" params="name parent_link:=base_link *origin">
-  <joint name="${name}_joint" type="fixed">
+<!-- The robot has a bumper with 5 contact sensors. The center one is
+functional, while the 4 remaining ones are created as dummy links. -->
+<xacro:macro name="dummy_bumper_zone" params="name parent_link:=base_link *origin">
+  <xacro:property name="link_name" value="${name}"/>
+  <xacro:property name="joint_name" value="${name}_joint"/>
+  <joint name="${joint_name}" type="fixed">
     <parent link="${parent_link}"/>
-    <child link="${name}"/>
+    <child link="${link_name}"/>
     <xacro:insert_block name="origin"/>
   </joint>
-  <link name="${name}">
-    <xacro:inertial_dummy/>
-  </link>
+  <link name="${link_name}"/>
 </xacro:macro>
-<xacro:macro name="bumper" params="name parent_link:=base_link update_rate:=62.0 visual_mesh collision_mesh
+<xacro:macro name="bumper" params="name:=bump_front_center parent_link:=base_link update_rate:=62.0 visual_mesh collision_mesh
   *origin *inertial">
-  <joint name="${name}_joint" type="fixed">
+  <xacro:property name="link_name" value="${name}"/>
+  <xacro:property name="joint_name" value="${name}_joint"/>
+  <joint name="${joint_name}" type="fixed">
     <parent link="${parent_link}"/>
-    <child link="${name}"/>
+    <child link="${link_name}"/>
     <xacro:insert_block name="origin"/>
   </joint>
-  <link name="${name}">
+  <link name="${link_name}">
     <visual>
       <geometry>
@@ -57,23 +56,23 @@
     </sensor>
   </gazebo>
-  <gazebo reference="${name}_joint">
+  <gazebo reference="${joint_name}">
     <preserveFixedJoint>true</preserveFixedJoint>
   </gazebo>
-  <xacro:dummy_bumper
+  <xacro:dummy_bumper_zone
       name="bump_front_left">
       <origin xyz="0.02345 -0.0875 0.025" rpy="0 0 0.5235985"/>
-  </xacro:dummy_bumper>
-  <xacro:dummy_bumper
+  </xacro:dummy_bumper_zone>
+  <xacro:dummy_bumper_zone
       name="bump_front_right">
       <origin xyz="0.02345 0.0875 0.025" rpy="0 0 -0.5235985"/>
-  </xacro:dummy_bumper>
-  <xacro:dummy_bumper
+  </xacro:dummy_bumper_zone>
+  <xacro:dummy_bumper_zone
       name="bump_left">
       <origin xyz="0.0875 -0.15155 0.025" rpy="0 0 1.047193"/>
-  </xacro:dummy_bumper>
-  <xacro:dummy_bumper
+  </xacro:dummy_bumper_zone>
+  <xacro:dummy_bumper_zone
       name="bump_right">
       <origin xyz="0.0875 0.15155 0.025" rpy="0 0 -1.047193"/>
-  </xacro:dummy_bumper>
+  </xacro:dummy_bumper_zone>
 </xacro:macro>
 </robot>

File: irobot_create_description/urdf/button.urdf.xacro (robot description, xacro)
@@ -8,5 +8,5 @@
   </joint>
   <link name="${name}">
-    <xacro:inertial_dummy/>
+    <!-- <xacro:inertial_dummy/> -->
   </link>
 </xacro:macro>

File: irobot_create_description/urdf/create3.urdf.xacro (robot description, xacro)
@@ -45,6 +45,6 @@
   </link>
   <!-- Bumper -->
+  <!-- name="bump_front_center" -->
   <xacro:bumper
-      name="bump_front_center"
       visual_mesh="file://$(find irobot_create_description)/meshes/bumper_visual.dae"
       collision_mesh="file://$(find irobot_create_description)/meshes/bumper_collision.dae">
@@ -66,5 +66,5 @@
   <!-- Caster wheel -->
   <xacro:caster name="front_caster" parent_link="base_link">
-    <origin xyz="${caster_position_x} 0 ${caster_position_z}" rpy="${-pi/2} ${pi} 0"/>
+    <origin xyz="${caster_position_x} 0 ${caster_position_z}" rpy="${-pi/2} 0 0"/>
   </xacro:caster>
   <!-- IMU -->
@@ -146,13 +146,13 @@
   <xacro:button
       name="button_1">
-      <origin xyz="0.06 0.37 0.08" rpy="0 -1.5707963 0"/>
+      <origin xyz="0.06 0.37 0.08" rpy="0 ${-pi/2} 0"/>
   </xacro:button>
   <xacro:button
       name="button_2">
-      <origin xyz="0.06 -0.37 0.08" rpy="0 -1.5707963 0"/>
+      <origin xyz="0.06 -0.37 0.08" rpy="0 ${-pi/2} 0"/>
   </xacro:button>
   <xacro:button
       name="button_power">
-      <origin xyz="0.06 0 0.08" rpy="0 -1.5707963 0"/>
+      <origin xyz="0.06 0 0.08" rpy="0 ${-pi/2} 0"/>
   </xacro:button>
 </robot>

File: irobot_create_description/urdf/wheel.urdf.xacro (robot description, xacro)
@@ -5,5 +5,5 @@
   <xacro:property name="radius" value="${3.575*cm2m}" />
   <xacro:property name="width"  value="${1.5*cm2m}" />
-  <xacro:property name="wheel_link_name"  value="_${name}_wheel"/>
+  <xacro:property name="wheel_link_name"  value="${name}_wheel"/>
   <xacro:property name="wheel_joint_name" value="${wheel_link_name}_joint"/>
   <joint name="${wheel_joint_name}" type="continuous">

File: irobot_create_description/urdf/wheel_drop.urdf.xacro (robot description, xacro)
@@ -8,5 +8,5 @@
   <xacro:property name="wd_mass" value="0.05"/>
   <xacro:property name="update_rate"   value="62" />
-  <xacro:property name="wd_link_name"  value="${name}_wheel"/>
+  <xacro:property name="wd_link_name"  value="wheel_drop_${name}"/>
   <xacro:property name="wd_joint_name" value="${wd_link_name}_joint"/>
   <joint name="${wd_joint_name}" type="prismatic">

File: irobot_create_description/urdf/wheel_with_wheeldrop.urdf.xacro (robot description, xacro)
@@ -9,5 +9,5 @@
   </xacro:wheel_drop>
   <!-- Wheel definition -->
-  <xacro:wheel name="${name}" parent_link="${name}_wheel">
+  <xacro:wheel name="${name}" parent_link="wheel_drop_${name}">
     <origin xyz="0 0 0" rpy="0 0 0"/>
   </xacro:wheel>

Commit message: Rename tf frame to match the real robot model (#63)
* Rename tf frames to match the real robot model

* Addressed comments.

* Removes extra comments

* Updates the positions of the cliff sensors. This also solves the trigger error.

* Corrects the cliff sensors position.

* Changes the min range of the cliff sensors.

File: irobot_create_description/urdf/bumper.urdf.xacro (robot description, xacro)
@@ -1,12 +1,26 @@
 <?xml version="1.0"?>
 <robot xmlns:xacro="http://ros.org/wiki/xacro">
-<xacro:macro name="bumper" params="name:=bumper parent_link update_rate:=62.0 visual_mesh collision_mesh
-  *origin *inertial">
-  <joint name="${name}_joint" type="fixed">
+<!-- The robot has a bumper with 5 contact sensors. The center one is
+functional, while the 4 remaining ones are created as dummy links. -->
+<xacro:macro name="dummy_bumper_zone" params="name parent_link:=base_link *origin">
+  <xacro:property name="link_name" value="${name}"/>
+  <xacro:property name="joint_name" value="${name}_joint"/>
+  <joint name="${joint_name}" type="fixed">
     <parent link="${parent_link}"/>
-    <child link="${name}_link"/>
+    <child link="${link_name}"/>
     <xacro:insert_block name="origin"/>
   </joint>
-  <link name="${name}_link">
+  <link name="${link_name}"/>
+</xacro:macro>
+<xacro:macro name="bumper" params="name:=bump_front_center parent_link:=base_link update_rate:=62.0 visual_mesh collision_mesh
+  *origin *inertial">
+  <xacro:property name="link_name" value="${name}"/>
+  <xacro:property name="joint_name" value="${name}_joint"/>
+  <joint name="${joint_name}" type="fixed">
+    <parent link="${parent_link}"/>
+    <child link="${link_name}"/>
+    <xacro:insert_block name="origin"/>
+  </joint>
+  <link name="${link_name}">
     <visual>
       <geometry>
@@ -21,5 +35,5 @@
     <xacro:insert_block name="inertial"/>
   </link>
-  <gazebo reference="${name}_link" >
+  <gazebo reference="${name}" >
     <mu1>0.1</mu1>
     <mu2>0.1</mu2>
@@ -42,7 +56,23 @@
     </sensor>
   </gazebo>
-  <gazebo reference="${name}_joint">
+  <gazebo reference="${joint_name}">
     <preserveFixedJoint>true</preserveFixedJoint>
   </gazebo>
+  <xacro:dummy_bumper_zone
+      name="bump_front_left">
+      <origin xyz="0.02345 -0.0875 0.025" rpy="0 0 0.5235985"/>
+  </xacro:dummy_bumper_zone>
+  <xacro:dummy_bumper_zone
+      name="bump_front_right">
+      <origin xyz="0.02345 0.0875 0.025" rpy="0 0 -0.5235985"/>
+  </xacro:dummy_bumper_zone>
+  <xacro:dummy_bumper_zone
+      name="bump_left">
+      <origin xyz="0.0875 -0.15155 0.025" rpy="0 0 1.047193"/>
+  </xacro:dummy_bumper_zone>
+  <xacro:dummy_bumper_zone
+      name="bump_right">
+      <origin xyz="0.0875 0.15155 0.025" rpy="0 0 -1.047193"/>
+  </xacro:dummy_bumper_zone>
 </xacro:macro>
 </robot>

File: irobot_create_description/urdf/create3.urdf.xacro (robot description, xacro)
@@ -2,4 +2,5 @@
 <robot name="create3" xmlns:xacro="http://ros.org/wiki/xacro">
   <xacro:include filename="$(find irobot_create_description)/urdf/bumper.urdf.xacro" />
+  <xacro:include filename="$(find irobot_create_description)/urdf/button.urdf.xacro" />
   <xacro:include filename="$(find irobot_create_description)/urdf/caster.urdf.xacro" />
   <xacro:include filename="$(find irobot_create_description)/urdf/common_properties.urdf.xacro"/>
@@ -10,26 +11,20 @@
   <xacro:include filename="$(find irobot_create_description)/urdf/wheel_with_wheeldrop.urdf.xacro" />
   <!-- MECHANICAL PROPERTIES -->
-  <xacro:property name="body_z_offset"           value="${-2.5*cm2m}" />
-  <xacro:property name="body_collision_z_offset" value="${-1*cm2m}" />
+  <xacro:property name="body_z_offset"           value="${4.1*cm2m}" />
+  <xacro:property name="body_collision_z_offset" value="${1*cm2m}" />
   <xacro:property name="body_mass"               value="2.300" />
   <xacro:property name="body_radius"             value="${16.4*cm2m}" />
   <xacro:property name="body_length"             value="${6*cm2m}" />
   <xacro:property name="bumper_mass"             value="0.1" />
-  <xacro:property name="bumper_offset_z"         value="${-2.5*cm2m}" />
+  <xacro:property name="bumper_offset_z"         value="${4.1*cm2m}" />
   <xacro:property name="bumber_inertial_x"       value="${8*cm2m}" />
   <xacro:property name="bumper_inertial_z"       value="${2*cm2m}"/>
-  <xacro:property name="wheel_height"            value="${-2.75*cm2m}" />
+  <xacro:property name="wheel_height"            value="${3.85*cm2m}" />
   <xacro:property name="distance_between_wheels" value="${23.3*cm2m}" />
   <xacro:property name="caster_position_x"       value="${12.5*cm2m}" />
-  <xacro:property name="caster_position_z"       value="${-5.4*cm2m}" />
-  <xacro:property name="wheel_drop_offset_z"     value="${3.5*mm2m}"/>
+  <xacro:property name="caster_position_z"       value="${1.2*cm2m}" />
+  <xacro:property name="wheel_drop_offset_z"     value="${3.1*mm2m}"/>
   <xacro:property name="wheel_drop_z"            value="${wheel_height + wheel_drop_offset_z}"/>
-  <!-- Create 3 base definitions-->
-  <link name="base_footprint"/>
-  <joint name="base_footprint_joint" type="fixed">
-    <origin xyz="0 0 0.066" rpy="0 0.013 0"/>
-    <parent link="base_footprint"/>
-    <child link="base_link" />
-  </joint>
+  <!-- Create 3 base definition-->
   <link name="base_link">
     <visual>
@@ -40,5 +35,5 @@
     </visual>
     <collision name="create3_base_collision">
-      <origin xyz="0 0 ${body_collision_z_offset}" rpy="0 0 ${pi/2}"/>
+      <origin xyz="0 0 ${body_z_offset + body_collision_z_offset}" rpy="0 0 ${pi/2}"/>
       <geometry>
         <cylinder length="${body_length}" radius="${body_radius}"/>
@@ -51,5 +46,4 @@
   <!-- Bumper -->
   <xacro:bumper
-      parent_link="base_link"
       visual_mesh="file://$(find irobot_create_description)/meshes/bumper_visual.dae"
       collision_mesh="file://$(find irobot_create_description)/meshes/bumper_collision.dae">
@@ -87,11 +81,11 @@
   </xacro:optical_mouse>
   <!-- Cliffs sensors -->
-  <xacro:property name="cliff_z"  value="${-4.5*cm2m}" />
-  <xacro:property name="cliff_center_x" value="${5.9*cm2m}"/>
-  <xacro:property name="cliff_center_y" value="${14.6*cm2m}"/>
+  <xacro:property name="cliff_z"  value="${2.1*cm2m}" />
+  <xacro:property name="cliff_center_x" value="${16*cm2m}"/>
+  <xacro:property name="cliff_center_y" value="${4.5*cm2m}"/>
   <xacro:property name="cliff_center_pitch" value="${80*deg2rad}"/>
   <xacro:property name="cliff_center_yaw" value="${65.3*deg2rad}"/>
-  <xacro:property name="cliff_back_x" value="${-6.5*cm2m}"/>
-  <xacro:property name="cliff_back_y" value="${14.5*cm2m}"/>
+  <xacro:property name="cliff_back_x" value="${6*cm2m}"/>
+  <xacro:property name="cliff_back_y" value="${-14.5*cm2m}"/>
   <xacro:property name="cliff_back_pitch" value="${80*deg2rad}"/>
   <xacro:property name="cliff_back_yaw" value="${167.4*deg2rad}"/>
@@ -148,3 +142,16 @@
     <origin xyz="0.0399 0.1488 ${ir_intensity_z_pos}" rpy="0 0 1.309"/>
   </xacro:ir_intensity>
+  <!-- Buttons -->
+  <xacro:button
+      name="button_1">
+      <origin xyz="0.06 0.37 0.08" rpy="0 ${-pi/2} 0"/>
+  </xacro:button>
+  <xacro:button
+      name="button_2">
+      <origin xyz="0.06 -0.37 0.08" rpy="0 ${-pi/2} 0"/>
+  </xacro:button>
+  <xacro:button
+      name="button_power">
+      <origin xyz="0.06 0 0.08" rpy="0 ${-pi/2} 0"/>
+  </xacro:button>
 </robot>
