Commit message: fix bumper and cliffs

File: irobot_create_description/urdf/bumper.urdf.xacro (robot description, xacro)
@@ -46,5 +46,5 @@
       <update_rate>${update_rate}</update_rate>
       <contact>
-        <collision>${name}_link_collision</collision>
+        <collision>${link_name}_collision</collision>
       </contact>
       <plugin name="${name}_plugin" filename="libgazebo_ros_create_bumper.so">

File: irobot_create_description/urdf/create3.urdf.xacro (robot description, xacro)
@@ -88,5 +88,5 @@
   </xacro:optical_mouse>
   <!-- Cliffs sensors -->
-  <xacro:property name="cliff_z"  value="${2.1*cm2m}" />
+  <xacro:property name="cliff_z"  value="${-4.5*cm2m}" />
   <xacro:property name="cliff_center_x" value="${16*cm2m}"/>
   <xacro:property name="cliff_center_y" value="${4.5*cm2m}"/>
@@ -165,8 +165,7 @@
   <xacro:property name="ir_omni_fov_rad" value="${220.0*deg2rad}"/>
   <xacro:property name="ir_front_facing_fov_rad" value="${pi/2}"/>
-  <xacro:ir_opcode_receivers robot_model_name="${robot_model_name}" dock_model_name="${dock_model_name}" emitter_link_name="${emitter_link_name}" sensor_0_range="0.01" sensor_0_fov="${ir_omni_fov_rad}"
-    sensor_1_range="0.5" sensor_1_fov="${ir_front_facing_fov_rad}" visualize="true" >
-    <origin xyz="0.153 0 0.035"/>
-  </xacro:ir_opcode_receivers>
+  <xacro:ir_opcode_receivers robot_model_name="${robot_model_name}" dock_model_name="${dock_model_name}"
+    emitter_link_name="${emitter_link_name}" sensor_0_range="0.01" sensor_0_fov="${ir_omni_fov_rad}"
+    sensor_1_range="0.5" sensor_1_fov="${ir_front_facing_fov_rad}" >
   <!-- Dock status -->
   <gazebo>

File: irobot_create_description/urdf/dock/standard.urdf.xacro (robot description, xacro)
@@ -34,6 +34,5 @@
                     parent="${link_name}"
                     aperture="${buoy_lateral_aperture}"
-                    range="1.0"
-                    visualize="true">
+                    range="1.0">
     <origin xyz="${buoy_x} 0 ${buoy_z}"
             rpy="0 0 ${- buoy_lateral_angle_yaw}"/>
@@ -43,6 +42,5 @@
                     parent="${link_name}"
                     aperture="${buoy_lateral_aperture}"
-                    range="1.0"
-                    visualize="true">
+                    range="1.0">
     <origin xyz="${buoy_x} 0 ${buoy_z}"
             rpy="0 0 ${buoy_lateral_angle_yaw}"/>
@@ -52,6 +50,5 @@
                     parent="${link_name}"
                     aperture="${10*deg2rad}"
-                    range="1.0"
-                    visualize="true">
+                    range="1.0">
     <origin xyz="${buoy_x} 0 ${buoy_z}"/>
   </xacro:ir_emitter>
@@ -60,6 +57,5 @@
                     parent="${link_name}"
                     aperture="360"
-                    range="0.6096"
-                    visualize="true">
+                    range="0.6096">
     <origin xyz="${buoy_x} 0 ${0.095 - z_offset}"/>
   </xacro:ir_emitter>
