Commit message: License moved to root and other minor comments addressed

File: irobot_create_description/urdf/create3.urdf.xacro (robot description, xacro)
@@ -13,11 +13,8 @@
   <xacro:property name="wheel_height" value="-0.0275" /><!-- z [m] -->
   <xacro:property name="distance_between_wheels" value="0.233" /><!-- y [m] -->
-  <xacro:property name="caster_mass" value="0.1" /> <!-- [kg] -->
   <xacro:property name="caster_radius" value="0.01" /> <!-- [m] -->
-  <xacro:property name="caster_width" value="0.018" /> <!-- [m] -->
   <xacro:property name="caster_position_x" value="0.125" /><!-- x [m] -->
   <xacro:property name="caster_position_y" value="0" /><!-- y [m] -->
   <xacro:property name="caster_position_z" value="-0.054" /><!-- z [m] -->
-  <xacro:property name="robot_type" value="create3" />
   <!-- Create 3 base definitions-->
   <link name="base_footprint"/>
@@ -33,5 +30,5 @@
       </geometry>
     </visual>
-    <collision name = "create3_base_collision">
+    <collision name="create3_base_collision">
       <origin xyz="-0.005 0 ${(body_z_offset/2.) + 0.01}"/>
       <geometry>
@@ -46,5 +43,5 @@
   <xacro:bumper
       parent_link="base_link"
-      robot_type="${robot_type}"
+      robot_type="create3"
       visual_mesh="file://meshes/bumper_collision.stl"
       collision_mesh="file://meshes/bumper_collision.stl">
@@ -56,5 +53,4 @@
     </inertial>
   </xacro:bumper>
-  <!-- Wheel configuration -->
   <!-- Wheel with mechanical wheel drop -->
   <xacro:wheel_with_wheeldrop name="left" parent_link="base_link">

Commit message: Removes traces of gazebo and launches robot in RViz only

File: irobot_create_description/urdf/create3.urdf.xacro (robot description, xacro)
@@ -27,5 +27,5 @@
       <origin xyz="0 0 ${body_z_offset}" rpy="0 0 ${-pi*3.0/2.0}"/>
       <geometry>
-        <mesh filename="file://meshes/body_collision.stl" scale="0.001 0.001 0.001"/>
+        <mesh filename="package://irobot_create_description/meshes/body_collision.stl" scale="0.001 0.001 0.001"/>
       </geometry>
     </visual>
@@ -44,6 +44,6 @@
       parent_link="base_link"
       robot_type="create3"
-      visual_mesh="file://meshes/bumper_collision.stl"
-      collision_mesh="file://meshes/bumper_collision.stl">
+      visual_mesh="package://irobot_create_description/meshes/bumper_collision.stl"
+      collision_mesh="package://irobot_create_description/meshes/bumper_collision.stl">
     <origin xyz="0 0 ${bumper_offset_z}"/>
     <inertial>
@@ -60,16 +60,4 @@
     <origin xyz="0 ${-distance_between_wheels/2} ${wheel_height}" rpy="${-pi/2} 0 0"/>
   </xacro:wheel_with_wheeldrop>
-  <gazebo>
-      <plugin name="wheels_joint_states" filename="libgazebo_ros_joint_state_publisher.so">
-        <joint_name>wheel_right_joint</joint_name>
-        <joint_name>wheel_left_joint</joint_name>
-      </plugin>
-  </gazebo>
-  <gazebo>
-      <plugin name="wheel_drop_joint_states" filename="libgazebo_ros_joint_state_publisher.so">
-        <joint_name>wheel_right_axle_joint</joint_name>
-        <joint_name>wheel_left_axle_joint</joint_name>
-      </plugin>
-  </gazebo>
   <joint name="caster_joint" type="fixed">
     <parent link="base_link"/>

Commit message: xacro formatting changes and adds README specifying dependencies

File: irobot_create_description/urdf/create3.urdf.xacro (robot description, xacro)
@@ -15,13 +15,7 @@
   <xacro:property name="wheel_height_cm"            value="-2.75" />
   <xacro:property name="distance_between_wheels_cm" value="23.3" />
-<<<<<<< HEAD
   <xacro:property name="caster_position_x_cm"       value="12.5" />
   <xacro:property name="caster_position_y_cm"       value="0" />
   <xacro:property name="caster_position_z_cm"       value="-5.4" />
-=======
-  <xacro:property name="caster_position_x" value="0.125" /><!-- x [m] -->
-  <xacro:property name="caster_position_y" value="0" /><!-- y [m] -->
-  <xacro:property name="caster_position_z" value="-0.054" /><!-- z [m] -->
->>>>>>> Gives files more appropriate names and makes macro of the caster wheel
   <!-- Create 3 base definitions-->
   <link name="base_footprint"/>
@@ -72,10 +66,6 @@
   <!-- Caster wheel -->
   <xacro:caster name="front_caster" parent_link="base_link">
-<<<<<<< HEAD
     <origin xyz="${caster_position_x_cm*cm2m} ${caster_position_y_cm*cm2m} ${caster_position_z_cm*cm2m}"
       rpy="${-pi/2} 0 0"/>
-=======
-    <origin xyz="${caster_position_x} ${caster_position_y} ${caster_position_z}" rpy="${-pi/2} 0 0"/>
->>>>>>> Gives files more appropriate names and makes macro of the caster wheel
   </xacro:caster>
 </robot>

Commit message: creates numeric variables in xacro files

File: irobot_create_description/urdf/create3.urdf.xacro (robot description, xacro)
@@ -7,9 +7,10 @@
   <!-- MECHANICAL PROPERTIES -->
   <xacro:property name="body_z_offset_cm"           value="-2.5" />
-  <xacro:property name="body_mass_kg"              value="2.300" />
+  <xacro:property name="body_mass_kg"               value="2.300" />
   <xacro:property name="body_radius_cm"             value="16" />
   <xacro:property name="body_length_cm"             value="4.8" />
-  <xacro:property name="bumper_mass_kg"            value="0.1" />
+  <xacro:property name="bumper_mass_kg"             value="0.1" />
   <xacro:property name="bumper_offset_z_cm"         value="-2.5" />
+  <xacro:property name="bumber_inertial_x_cm"       value="8" />
   <xacro:property name="wheel_height_cm"            value="-2.75" />
   <xacro:property name="distance_between_wheels_cm" value="23.3" />
@@ -27,14 +28,16 @@
       <origin xyz="0 0 ${body_z_offset_cm*cm2m}" rpy="0 0 ${-pi*3.0/2.0}"/>
       <geometry>
-        <mesh filename="file://$(find irobot_create_description)/meshes/body_collision.stl" scale="0.001 0.001 0.001"/>
+        <mesh filename="file://$(find irobot_create_description)/meshes/body_collision.stl"
+          scale="0.001 0.001 0.001"/>
       </geometry>
     </visual>
     <collision name="create3_base_collision">
-      <origin xyz="-0.005 0 ${body_z_offset_cm*cm2m/2.}"/>
+      <origin xyz="0 0 ${body_z_offset_cm*cm2m/2}"/>
       <geometry>
         <cylinder length="${body_length_cm*cm2m}" radius="${body_radius_cm*cm2m}"/>
       </geometry>
     </collision>
-    <xacro:inertial_cylinder_with_pose mass="${body_mass_kg}" radius="${body_radius_cm*cm2m}" length="${body_length_cm*cm2m}">
+    <xacro:inertial_cylinder_with_pose mass="${body_mass_kg}" radius="${body_radius_cm*cm2m}"
+      length="${body_length_cm*cm2m}">
       <origin xyz="0 0 ${body_z_offset_cm*cm2m}"/>
     </xacro:inertial_cylinder_with_pose>
@@ -48,5 +51,5 @@
     <origin xyz="0 0 ${bumper_offset_z_cm*cm2m}"/>
     <inertial>
-        <origin xyz="0.08 0 ${bumper_offset_z_cm*cm2m}"/>
+        <origin xyz="${bumber_inertial_x_cm*cm2m} 0 ${bumper_offset_z_cm*cm2m}"/>
         <mass value="${bumper_mass_kg}"/>
         <inertia ixx="0.0013483753405" ixy="0.0000000454352" ixz="0.0000014434849" iyy="0.0002521736852"

File: irobot_create_description/urdf/wheel_with_wheeldrop.urdf.xacro (robot description, xacro)
@@ -3,4 +3,14 @@
 <xacro:include filename="$(find irobot_create_description)/urdf/wheel.urdf.xacro" />
 <xacro:macro name="wheel_with_wheeldrop" params="name parent_link *origin">
+  <xacro:property name="wheel_drop_lower"             value="0" />
+  <xacro:property name="wheel_drop_upper"             value="0.03" />
+  <xacro:property name="wheel_drop_effort"            value="100" />
+  <xacro:property name="wheel_drop_vel"               value="1" />
+  <xacro:property name="wheel_drop_spring_stiffness"  value="300" />
+  <xacro:property name="wheel_drop_spring_reference"  value="0.03" />
+  <xacro:property name="wheel_axle_mass"              value="0.05" />
+  <xacro:property name="wheel_axle_x"                 value="0.15" />
+  <xacro:property name="wheel_axle_y"                 value="0.15" />
+  <xacro:property name="wheel_axle_z"                 value="0.15" />
   <joint name="wheel_${name}_axle_joint" type="prismatic">
     <parent link="${parent_link}"/>
@@ -8,14 +18,16 @@
     <xacro:insert_block name="origin"/>
     <axis xyz="0 1 0"/>
-    <limit lower="0.0" upper="0.03" effort="100" velocity="1"/>
+    <limit lower="${wheel_drop_lower}" upper="${wheel_drop_upper}" effort="${wheel_drop_effort}"
+      velocity="${wheel_drop_vel}"/>
   </joint>
   <!-- Gazebo parameters to simulate a spring -->
   <gazebo reference="wheel_${name}_axle_joint">
     <implicitSpringDamper>true</implicitSpringDamper>
-    <springStiffness>300</springStiffness>
-    <springReference>0.03</springReference>
+    <springStiffness>${wheel_drop_spring_stiffness}</springStiffness>
+    <springReference>${wheel_drop_spring_reference}</springReference>
   </gazebo>
   <link name="wheel_${name}_axle_link">
-    <xacro:inertial_cuboid mass="0.05" x="0.15" y="0.15" z="0.15"/>
+    <xacro:inertial_cuboid mass="${wheel_axle_mass}" x="${wheel_axle_x}" y="${wheel_axle_y}"
+      z="${wheel_axle_z}"/>
   </link>
   <!-- Wheel definition -->

Commit message: diffdrive control package

File: irobot_create_description/urdf/create3.urdf.xacro (robot description, xacro)
@@ -72,3 +72,8 @@
       rpy="${-pi/2} 0 0"/>
   </xacro:caster>
+  <gazebo>
+    <plugin name="gazebo_ros2_control" filename="libgazebo_ros2_control.so">
+      <parameters> $(find irobot_create_control)/config/control.yaml </parameters>
+    </plugin>
+  </gazebo>
 </robot>

File: irobot_create_description/urdf/wheel.urdf.xacro (robot description, xacro)
@@ -34,4 +34,13 @@
     <material>Gazebo/DarkGrey</material>
   </gazebo>
+  <ros2_control name="${name}_wheel_system" type="system">
+      <hardware>
+        <plugin>gazebo_ros2_control/GazeboSystem</plugin>
+      </hardware>
+      <joint name="wheel_${name}_joint">
+        <command_interface name="velocity" />
+        <state_interface name="position"/>
+      </joint>
+  </ros2_control>
 </xacro:macro>
 </robot>

Commit message: Adds mouse sensor plugin

File: irobot_create_description/urdf/create3.urdf.xacro (robot description, xacro)
@@ -5,4 +5,5 @@
   <xacro:include filename="$(find irobot_create_description)/urdf/common_properties.urdf.xacro"/>
   <xacro:include filename="$(find irobot_create_description)/urdf/wheel_with_wheeldrop.urdf.xacro" />
+  <xacro:include filename="$(find irobot_create_description)/urdf/sensors/optical_mouse.urdf.xacro"/>
   <!-- MECHANICAL PROPERTIES -->
   <xacro:property name="body_z_offset_cm"           value="-2.5" />
@@ -77,3 +78,13 @@
     </plugin>
   </gazebo>
+  <!-- Optical mouse -->
+  <xacro:optical_mouse name="optical_mouse"
+                      parent="base_link"
+                      ros_topic="optical_mouse"
+                      visualize="true"
+                      noise_mean="0.0"
+                      noise_var="0.0"
+                      mouse_seed="0.0" sensor_rotation="${pi/4}" resolution="492" update_rate="80">
+  <origin xyz="0.1015 0.087 -0.055"/>
+</xacro:optical_mouse>
 </robot>

Commit message: updates publish rate

File: irobot_create_description/urdf/create3.urdf.xacro (robot description, xacro)
@@ -22,4 +22,6 @@
   <xacro:property name="inertial_offset_x_cm"       value="1" />
   <xacro:property name="wheel_drop_offset_z_mm"     value="3.5"/>
+  <xacro:property name="mouse_resolution"           value="492" />
+  <xacro:property name="mouse_update_rate"          value="62" />
   <!-- Create 3 base definitions-->
   <link name="base_footprint"/>
@@ -85,5 +87,5 @@
                       noise_mean="0.0"
                       noise_var="0.0"
-                      mouse_seed="0.0" sensor_rotation="${pi/4}" resolution="492" update_rate="80">
+                      mouse_seed="0.0" sensor_rotation="${pi/4}" resolution="${mouse_resolution}" update_rate="${mouse_update_rate}">
   <origin xyz="0.1015 0.087 -0.055"/>
 </xacro:optical_mouse>

Commit message: WIP: update robot meshes

File: irobot_create_description/urdf/create3.urdf.xacro (robot description, xacro)
@@ -26,12 +26,11 @@
   <link name="base_link">
     <visual>
-      <origin xyz="0 0 ${body_z_offset_cm*cm2m}" rpy="0 0 ${-pi*3.0/2.0}"/>
+      <origin xyz="0 0 ${body_z_offset_cm*cm2m}" rpy="0 0 ${pi/2}"/>
       <geometry>
-        <mesh filename="file://$(find irobot_create_description)/meshes/body_collision.stl"
-          scale="0.001 0.001 0.001"/>
+        <mesh filename="file://$(find irobot_create_description)/meshes/body_visual.dae" />
       </geometry>
     </visual>
     <collision name="create3_base_collision">
-      <origin xyz="0 0 ${body_z_offset_cm*cm2m/2}"/>
+      <origin xyz="0 0 ${body_z_offset_cm*cm2m}" rpy="0 0 ${pi/2}"/>
       <geometry>
         <cylinder length="${body_length_cm*cm2m}" radius="${body_radius_cm*cm2m}"/>
@@ -47,7 +46,7 @@
       parent_link="base_link"
       robot_type="create3"
-      visual_mesh="file://$(find irobot_create_description)/meshes/bumper_collision.stl"
-      collision_mesh="file://$(find irobot_create_description)/meshes/bumper_collision.stl">
-    <origin xyz="0 0 ${bumper_offset_z_cm*cm2m}"/>
+      visual_mesh="file://$(find irobot_create_description)/meshes/bumper_visual.dae"
+      collision_mesh="file://$(find irobot_create_description)/meshes/bumper_collision.dae">
+    <origin xyz="0 0 ${bumper_offset_z_cm*cm2m}" rpy="0 0 ${pi/2}"/>
     <inertial>
         <origin xyz="${bumber_inertial_x_cm*cm2m} 0 ${bumper_offset_z_cm*cm2m}"/>

Commit message: WIP: Improved collision and inertias

File: irobot_create_description/urdf/create3.urdf.xacro (robot description, xacro)
@@ -7,7 +7,8 @@
   <!-- MECHANICAL PROPERTIES -->
   <xacro:property name="body_z_offset_cm"           value="-2.5" />
+  <xacro:property name="body_collision_z_offset_cm" value="-1" />
   <xacro:property name="body_mass_kg"               value="2.300" />
-  <xacro:property name="body_radius_cm"             value="16" />
-  <xacro:property name="body_length_cm"             value="4.8" />
+  <xacro:property name="body_radius_cm"             value="16.4" />
+  <xacro:property name="body_length_cm"             value="6" />
   <xacro:property name="bumper_mass_kg"             value="0.1" />
   <xacro:property name="bumper_offset_z_cm"         value="-2.5" />
@@ -18,4 +19,5 @@
   <xacro:property name="caster_position_y_cm"       value="0" />
   <xacro:property name="caster_position_z_cm"       value="-5.4" />
+  <xacro:property name="inertial_offset_x_cm"       value="1" />
   <!-- Create 3 base definitions-->
   <link name="base_footprint"/>
@@ -32,5 +34,5 @@
     </visual>
     <collision name="create3_base_collision">
-      <origin xyz="0 0 ${body_z_offset_cm*cm2m}" rpy="0 0 ${pi/2}"/>
+      <origin xyz="0 0 ${body_collision_z_offset_cm*cm2m}" rpy="0 0 ${pi/2}"/>
       <geometry>
         <cylinder length="${body_length_cm*cm2m}" radius="${body_radius_cm*cm2m}"/>
@@ -39,5 +41,5 @@
     <xacro:inertial_cylinder_with_pose mass="${body_mass_kg}" radius="${body_radius_cm*cm2m}"
       length="${body_length_cm*cm2m}">
-      <origin xyz="0 0 ${body_z_offset_cm*cm2m}"/>
+      <origin xyz="${inertial_offset_x_cm*cm2m} 0 ${body_collision_z_offset_cm*cm2m}"/>
     </xacro:inertial_cylinder_with_pose>
   </link>

Commit message: Use realistic wheeldrop model

File: irobot_create_description/urdf/create3.urdf.xacro (robot description, xacro)
@@ -1,8 +1,8 @@
 <?xml version="1.0" ?>
 <robot name="create3" xmlns:xacro="http://ros.org/wiki/xacro">
+  <xacro:include filename="$(find irobot_create_description)/urdf/bumper.urdf.xacro" />
+  <xacro:include filename="$(find irobot_create_description)/urdf/caster.urdf.xacro" />
   <xacro:include filename="$(find irobot_create_description)/urdf/common_properties.urdf.xacro"/>
-  <xacro:include filename="$(find irobot_create_description)/urdf/bumper.urdf.xacro" />
   <xacro:include filename="$(find irobot_create_description)/urdf/wheel_with_wheeldrop.urdf.xacro" />
-  <xacro:include filename="$(find irobot_create_description)/urdf/caster.urdf.xacro" />
   <!-- MECHANICAL PROPERTIES -->
   <xacro:property name="body_z_offset_cm"           value="-2.5" />
@@ -59,8 +59,8 @@
   </xacro:bumper>
   <!-- Wheels with mechanical wheel drop -->
-  <xacro:wheel_with_wheeldrop name="left" parent_link="base_link">
+  <xacro:wheel_with_wheeldrop name="left">
     <origin xyz="0 ${distance_between_wheels_cm*cm2m/2} ${wheel_height_cm*cm2m}" rpy="${-pi/2} 0 0"/>
   </xacro:wheel_with_wheeldrop>
-  <xacro:wheel_with_wheeldrop name="right" parent_link="base_link">
+  <xacro:wheel_with_wheeldrop name="right">
     <origin xyz="0 ${-distance_between_wheels_cm*cm2m/2} ${wheel_height_cm*cm2m}" rpy="${-pi/2} 0 0"/>
   </xacro:wheel_with_wheeldrop>

File: irobot_create_description/urdf/wheel_with_wheeldrop.urdf.xacro (robot description, xacro)
@@ -1,34 +1,11 @@
 <?xml version="1.0"?>
 <robot xmlns:xacro="http://ros.org/wiki/xacro">
-<xacro:include filename="$(find irobot_create_description)/urdf/wheel.urdf.xacro" />
-<xacro:macro name="wheel_with_wheeldrop" params="name parent_link *origin">
-  <xacro:property name="lower_mm"         value="0" />
-  <xacro:property name="upper_mm"         value="30" />
-  <xacro:property name="effort"           value="100" />
-  <xacro:property name="velocity"         value="1" />
-  <xacro:property name="spring_stiffness" value="300" />
-  <xacro:property name="spring_reference" value="0.03" />
-  <xacro:property name="axle_mass"        value="0.05" />
-  <xacro:property name="axle_x"           value="0.15" />
-  <xacro:property name="axle_y"           value="0.15" />
-  <xacro:property name="axle_z"           value="0.15" />
-  <joint name="wheel_${name}_axle_joint" type="prismatic">
-    <parent link="${parent_link}"/>
-    <child link="wheel_${name}_axle_link"/>
+<xacro:macro name="wheel_with_wheeldrop" params="name parent_link:=base_link *origin">
+  <xacro:include filename="$(find irobot_create_description)/urdf/wheel.urdf.xacro" />
+  <xacro:include filename="$(find irobot_create_description)/urdf/wheel_drop.urdf.xacro" />
+  <!-- Wheel Drop definition -->
+  <xacro:wheel_drop name="${name}" parent="${parent_link}">
     <xacro:insert_block name="origin"/>
-    <axis xyz="0 1 0"/>
-    <limit lower="${lower_mm*mm2m}" upper="${upper_mm*mm2m}" effort="${effort}"
-      velocity="${velocity}"/>
-  </joint>
-  <!-- Gazebo parameters to simulate a spring -->
-  <gazebo reference="wheel_${name}_axle_joint">
-    <implicitSpringDamper>true</implicitSpringDamper>
-    <springStiffness>${spring_stiffness}</springStiffness>
-    <springReference>${spring_reference}</springReference>
-  </gazebo>
-  <link name="wheel_${name}_axle_link">
-    <xacro:inertial_cuboid mass="${axle_mass}" x="${axle_x}" y="${axle_y}"
-      z="${axle_z}"/>
-  </link>
+  </xacro:wheel_drop>
   <!-- Wheel definition -->
   <xacro:wheel name="${name}" parent_link="wheel_${name}_axle_link">

Commit message: Fix body inclination offset

File: irobot_create_description/urdf/create3.urdf.xacro (robot description, xacro)
@@ -20,4 +20,5 @@
   <xacro:property name="caster_position_z_cm"       value="-5.4" />
   <xacro:property name="inertial_offset_x_cm"       value="1" />
+  <xacro:property name="wheel_drop_offset_z_mm"     value="3.5"/>
   <!-- Create 3 base definitions-->
   <link name="base_footprint"/>
@@ -59,9 +60,10 @@
   </xacro:bumper>
   <!-- Wheels with mechanical wheel drop -->
+  <xacro:property name="wheel_drop_z" value="${wheel_height_cm*cm2m + wheel_drop_offset_z_mm*mm2m}"/>
   <xacro:wheel_with_wheeldrop name="left">
-    <origin xyz="0 ${distance_between_wheels_cm*cm2m/2} ${wheel_height_cm*cm2m}" rpy="${-pi/2} 0 0"/>
+    <origin xyz="0 ${distance_between_wheels_cm*cm2m/2} ${wheel_drop_z}" rpy="${-pi/2} 0 0"/>
   </xacro:wheel_with_wheeldrop>
   <xacro:wheel_with_wheeldrop name="right">
-    <origin xyz="0 ${-distance_between_wheels_cm*cm2m/2} ${wheel_height_cm*cm2m}" rpy="${-pi/2} 0 0"/>
+    <origin xyz="0 ${-distance_between_wheels_cm*cm2m/2} ${wheel_drop_z}" rpy="${-pi/2} 0 0"/>
   </xacro:wheel_with_wheeldrop>
   <!-- Caster wheel -->
