Commit message: Use realistic wheel drop model (#8)
* Use realistic wheeldrop model

* Rename parent argument to parent_link

* Add wheel drop plugin

* Enable C++ linter

* Fix linter

* Create irobot_create_gazebo_plugins

* Add env hooks

* Fix reminiscents of irobot_create_gazebo_plugins

* Address Alexis' comments

* Use 62 Hz by default

* Fix body inclination offset

* Fix plugin installation

* Remove env-hooks

* Address Rodri's comment

Add urdf cliff sensor to create3

Add cliff plugin

Addressed Emi and Rodr's comments

Enable linter

Address Emi Rodri and Alexis comments

Update irobot_create_description/urdf/cliffs_sensor.urdf.xacro

Co-authored-by: Emiliano Borghi <emiliano.borghi@gmail.com>

Address more comments

Update cliff sensor links and added to the create3

Fix remapping warning

Update ament checks  and emi comments

Addressed Emi's comments

Address more Emi's commment

Update cliff topic

Address Emi's functions

Improve the code with Emi comments

File: irobot_create_description/urdf/create3.urdf.xacro (robot description, xacro)
@@ -3,4 +3,5 @@
   <xacro:include filename="$(find irobot_create_description)/urdf/bumper.urdf.xacro" />
   <xacro:include filename="$(find irobot_create_description)/urdf/caster.urdf.xacro" />
+  <xacro:include filename="$(find irobot_create_description)/urdf/cliff_sensor.urdf.xacro"/>
   <xacro:include filename="$(find irobot_create_description)/urdf/common_properties.urdf.xacro"/>
   <xacro:include filename="$(find irobot_create_description)/urdf/sensors/optical_mouse.urdf.xacro"/>
@@ -82,3 +83,29 @@
     <origin xyz="0.1015 0.087 -0.055" rpy="0 0 ${-pi/4}"/>
   </xacro:optical_mouse>
+  <!-- Cliffs sensors -->
+  <xacro:property name="cliff_z"        value="${-4.5*cm2m}" />
+  <xacro:property name="cliff_center_x" value="${5.9*cm2m}"/>
+  <xacro:property name="cliff_center_y" value="${14.6*cm2m}"/>
+  <xacro:property name="cliff_center_P" value="${80*deg2rad}"/>
+  <xacro:property name="cliff_center_Y" value="${65.3*deg2rad}"/>
+  <xacro:property name="cliff_back_x" value="${-6.5*cm2m}"/>
+  <xacro:property name="cliff_back_y" value="${14.5*cm2m}"/>
+  <xacro:property name="cliff_back_P" value="${80*deg2rad}"/>
+  <xacro:property name="cliff_back_Y" value="${167.4*deg2rad}"/>
+  <xacro:cliff_sensor name="side_left">
+    <origin xyz="${cliff_back_x} ${cliff_back_y} ${cliff_z}"
+            rpy="0 ${cliff_back_P} ${cliff_back_Y}"/>
+  </xacro:cliff_sensor>
+  <xacro:cliff_sensor name="side_right">
+    <origin xyz="${cliff_back_x} ${- cliff_back_y} ${cliff_z}"
+            rpy="0 ${cliff_back_P} ${- cliff_back_Y}"/>
+  </xacro:cliff_sensor>
+  <xacro:cliff_sensor name="front_left">
+    <origin xyz="${cliff_center_x} ${cliff_center_y} ${cliff_z}"
+            rpy="0 ${cliff_center_P} ${cliff_center_Y}"/>
+  </xacro:cliff_sensor>
+  <xacro:cliff_sensor name="front_right">
+    <origin xyz="${cliff_center_x} ${- cliff_center_y} ${cliff_z}"
+            rpy="0 ${cliff_center_P} ${- cliff_center_Y}"/>
+  </xacro:cliff_sensor>
 </robot>

File: irobot_create_description/urdf/wheel_drop.urdf.xacro (robot description, xacro)
@@ -32,5 +32,9 @@
       <ros>
         <namespace>wheel_drop</namespace>
+<<<<<<< HEAD
         <argument>~/out:=${name}_wheel/event</argument>
+=======
+        <remapping>~/out:=${name}_wheel/event</remapping>
+>>>>>>> Use realistic wheel drop model (#8)
       </ros>
       <updateRate>${update_rate}</updateRate>

Commit message: Use realistic wheel drop model (#8)
* Use realistic wheeldrop model

* Rename parent argument to parent_link

* Add wheel drop plugin

* Enable C++ linter

* Fix linter

* Create irobot_create_gazebo_plugins

* Add env hooks

* Fix reminiscents of irobot_create_gazebo_plugins

* Address Alexis' comments

* Use 62 Hz by default

* Fix body inclination offset

* Fix plugin installation

* Remove env-hooks

* Address Rodri's comment

File: irobot_create_description/urdf/create3.urdf.xacro (robot description, xacro)
@@ -1,8 +1,8 @@
 <?xml version="1.0" ?>
 <robot name="create3" xmlns:xacro="http://ros.org/wiki/xacro">
+  <xacro:include filename="$(find irobot_create_description)/urdf/bumper.urdf.xacro" />
+  <xacro:include filename="$(find irobot_create_description)/urdf/caster.urdf.xacro" />
   <xacro:include filename="$(find irobot_create_description)/urdf/common_properties.urdf.xacro"/>
-  <xacro:include filename="$(find irobot_create_description)/urdf/bumper.urdf.xacro" />
   <xacro:include filename="$(find irobot_create_description)/urdf/wheel_with_wheeldrop.urdf.xacro" />
-  <xacro:include filename="$(find irobot_create_description)/urdf/caster.urdf.xacro" />
   <!-- MECHANICAL PROPERTIES -->
   <xacro:property name="body_z_offset_cm"           value="-2.5" />
@@ -20,4 +20,5 @@
   <xacro:property name="caster_position_z_cm"       value="-5.4" />
   <xacro:property name="inertial_offset_x_cm"       value="1" />
+  <xacro:property name="wheel_drop_offset_z_mm"     value="3.5"/>
   <!-- Create 3 base definitions-->
   <link name="base_footprint"/>
@@ -59,9 +60,10 @@
   </xacro:bumper>
   <!-- Wheels with mechanical wheel drop -->
-  <xacro:wheel_with_wheeldrop name="left" parent_link="base_link">
-    <origin xyz="0 ${distance_between_wheels_cm*cm2m/2} ${wheel_height_cm*cm2m}" rpy="${-pi/2} 0 0"/>
+  <xacro:property name="wheel_drop_z" value="${wheel_height_cm*cm2m + wheel_drop_offset_z_mm*mm2m}"/>
+  <xacro:wheel_with_wheeldrop name="left">
+    <origin xyz="0 ${distance_between_wheels_cm*cm2m/2} ${wheel_drop_z}" rpy="${-pi/2} 0 0"/>
   </xacro:wheel_with_wheeldrop>
-  <xacro:wheel_with_wheeldrop name="right" parent_link="base_link">
-    <origin xyz="0 ${-distance_between_wheels_cm*cm2m/2} ${wheel_height_cm*cm2m}" rpy="${-pi/2} 0 0"/>
+  <xacro:wheel_with_wheeldrop name="right">
+    <origin xyz="0 ${-distance_between_wheels_cm*cm2m/2} ${wheel_drop_z}" rpy="${-pi/2} 0 0"/>
   </xacro:wheel_with_wheeldrop>
   <!-- Caster wheel -->

File: irobot_create_description/urdf/wheel_with_wheeldrop.urdf.xacro (robot description, xacro)
@@ -1,34 +1,11 @@
 <?xml version="1.0"?>
 <robot xmlns:xacro="http://ros.org/wiki/xacro">
-<xacro:include filename="$(find irobot_create_description)/urdf/wheel.urdf.xacro" />
-<xacro:macro name="wheel_with_wheeldrop" params="name parent_link *origin">
-  <xacro:property name="lower_mm"         value="0" />
-  <xacro:property name="upper_mm"         value="30" />
-  <xacro:property name="effort"           value="100" />
-  <xacro:property name="velocity"         value="1" />
-  <xacro:property name="spring_stiffness" value="300" />
-  <xacro:property name="spring_reference" value="0.03" />
-  <xacro:property name="axle_mass"        value="0.05" />
-  <xacro:property name="axle_x"           value="0.15" />
-  <xacro:property name="axle_y"           value="0.15" />
-  <xacro:property name="axle_z"           value="0.15" />
-  <joint name="wheel_${name}_axle_joint" type="prismatic">
-    <parent link="${parent_link}"/>
-    <child link="wheel_${name}_axle_link"/>
+<xacro:macro name="wheel_with_wheeldrop" params="name parent_link:=base_link *origin">
+  <xacro:include filename="$(find irobot_create_description)/urdf/wheel.urdf.xacro" />
+  <xacro:include filename="$(find irobot_create_description)/urdf/wheel_drop.urdf.xacro" />
+  <!-- Wheel Drop definition -->
+  <xacro:wheel_drop name="${name}" parent_link="${parent_link}">
     <xacro:insert_block name="origin"/>
-    <axis xyz="0 1 0"/>
-    <limit lower="${lower_mm*mm2m}" upper="${upper_mm*mm2m}" effort="${effort}"
-      velocity="${velocity}"/>
-  </joint>
-  <!-- Gazebo parameters to simulate a spring -->
-  <gazebo reference="wheel_${name}_axle_joint">
-    <implicitSpringDamper>true</implicitSpringDamper>
-    <springStiffness>${spring_stiffness}</springStiffness>
-    <springReference>${spring_reference}</springReference>
-  </gazebo>
-  <link name="wheel_${name}_axle_link">
-    <xacro:inertial_cuboid mass="${axle_mass}" x="${axle_x}" y="${axle_y}"
-      z="${axle_z}"/>
-  </link>
+  </xacro:wheel_drop>
   <!-- Wheel definition -->
   <xacro:wheel name="${name}" parent_link="wheel_${name}_axle_link">

Commit message: applies mouse improvements

File: irobot_create_description/urdf/create3.urdf.xacro (robot description, xacro)
@@ -22,5 +22,4 @@
   <xacro:property name="inertial_offset_x_cm"       value="1" />
   <xacro:property name="wheel_drop_offset_z_mm"     value="3.5"/>
-  <xacro:property name="mouse_resolution"           value="492" />
   <xacro:property name="mouse_update_rate"          value="62" />
   <!-- Create 3 base definitions-->
@@ -87,6 +86,6 @@
                       noise_mean="0.0"
                       noise_var="0.0"
-                      mouse_seed="0.0" sensor_rotation="${pi/4}" resolution="${mouse_resolution}" update_rate="${mouse_update_rate}">
-  <origin xyz="0.1015 0.087 -0.055"/>
+                      mouse_seed="0.0" update_rate="${mouse_update_rate}">
+  <origin xyz="0.1015 0.087 -0.055" rpy="0 0 ${-pi/4}"/>
 </xacro:optical_mouse>
 </robot>

File: irobot_create_description/urdf/sensors/optical_mouse.urdf.xacro (robot description, xacro)
@@ -1,6 +1,6 @@
 <?xml version="1.0"?>
 <robot xmlns:xacro="http://ros.org/wiki/xacro">
-  <xacro:macro name="optical_mouse" params="name parent *origin ros_topic visualize sensor_rotation
-                                            noise_mean:=0 noise_var:=0 mouse_seed resolution update_rate" >
+  <xacro:macro name="optical_mouse" params="name parent *origin ros_topic visualize noise_mean:=0
+                                            noise_var:=0 mouse_seed update_rate" >
     <!-- Sensor settings -->
     <xacro:property name="mass" value="0.1" />
@@ -9,7 +9,5 @@
     <!-- Visualization settings -->
     <xacro:property name="color" value="Red" />
-    <joint name="optical_mouse_joint" type="revolute">
-      <axis xyz="0 1 0" />
-      <limit effort="1000.0" lower="0.0" upper="0.0" velocity="0.0"/>
+    <joint name="optical_mouse_joint" type="fixed">
       <xacro:insert_block name="origin"/>
       <parent link="${parent}"/>
@@ -33,6 +31,4 @@
         <update_rate>${update_rate}</update_rate>
         <link>optical_mouse_${name}_link</link>
-        <resolution>${resolution}</resolution>
-        <sensor_rotation>${sensor_rotation}</sensor_rotation>
         <gaussian_mean>${noise_mean}</gaussian_mean>
         <gaussian_var>${noise_var}</gaussian_var>
@@ -46,4 +42,7 @@
       <material>Gazebo/${color}</material>
     </gazebo>
+    <gazebo reference="optical_mouse_joint" >
+      <preserveFixedJoint>true</preserveFixedJoint>
+    </gazebo>
   </xacro:macro>
 </robot>

Commit message: Add IR intensity sensors to Create 3

File: irobot_create_description/urdf/create3.urdf.xacro (robot description, xacro)
@@ -4,4 +4,5 @@
   <xacro:include filename="$(find irobot_create_description)/urdf/caster.urdf.xacro" />
   <xacro:include filename="$(find irobot_create_description)/urdf/common_properties.urdf.xacro"/>
+  <xacro:include filename="$(find irobot_create_description)/urdf/ir_intensity.urdf.xacro" />
   <xacro:include filename="$(find irobot_create_description)/urdf/sensors/optical_mouse.urdf.xacro"/>
   <xacro:include filename="$(find irobot_create_description)/urdf/wheel_with_wheeldrop.urdf.xacro" />
@@ -82,3 +83,26 @@
     <origin xyz="0.1015 0.087 -0.055" rpy="0 0 ${-pi/4}"/>
   </xacro:optical_mouse>
+  <!-- IR intensity sensors -->
+  <xacro:property name="ir_intensity_z_pos_cm" value="3"/>
+  <xacro:ir_intensity name="front_center_left">
+    <origin xyz="0.1540 -0.0000 ${ir_intensity_z_pos_cm*cm2m}"/>
+  </xacro:ir_intensity>
+  <xacro:ir_intensity name="front_center_right">
+    <origin xyz="0.1396 -0.0651 ${ir_intensity_z_pos_cm*cm2m}" rpy="0 0 -0.436"/>
+  </xacro:ir_intensity>
+  <xacro:ir_intensity name="front_left">
+    <origin xyz="0.1396 0.0651 ${ir_intensity_z_pos_cm*cm2m}" rpy="0 0 0.436"/>
+  </xacro:ir_intensity>
+  <xacro:ir_intensity name="front_right">
+    <origin xyz="0.0990 -0.1180 ${ir_intensity_z_pos_cm*cm2m}" rpy="0 0 -0.873"/>
+  </xacro:ir_intensity>
+  <xacro:ir_intensity name="left">
+    <origin xyz="0.0990 0.1180 ${ir_intensity_z_pos_cm*cm2m}" rpy="0 0 0.873"/>
+  </xacro:ir_intensity>
+  <xacro:ir_intensity name="right">
+    <origin xyz="0.0399 -0.1488 ${ir_intensity_z_pos_cm*cm2m}" rpy="0 0 -1.309"/>
+  </xacro:ir_intensity>
+  <xacro:ir_intensity name="side_left">
+    <origin xyz="0.0399 0.1488 ${ir_intensity_z_pos_cm*cm2m}" rpy="0 0 1.309"/>
+  </xacro:ir_intensity>
 </robot>

Commit message: Move IR sensors behind the bumpers

File: irobot_create_description/urdf/create3.urdf.xacro (robot description, xacro)
@@ -84,5 +84,5 @@
   </xacro:optical_mouse>
   <!-- IR intensity sensors -->
-  <xacro:property name="ir_intensity_z_pos_cm" value="3"/>
+  <xacro:property name="ir_intensity_z_pos_cm" value="-0.7"/>
   <xacro:ir_intensity name="front_center_left">
     <origin xyz="0.1540 -0.0000 ${ir_intensity_z_pos_cm*cm2m}"/>

File: irobot_create_description/urdf/ir_intensity.urdf.xacro (robot description, xacro)
@@ -5,5 +5,5 @@
                params="name parent:=base_link
                        update_rate:=62.0 fov:=${10*deg2rad}
-                       min_range:=${5*mm2m} max_range:=${20*cm2m}
+                       min_range:=${25*mm2m} max_range:=${20*cm2m}
                        visualize:=true *origin" >
     <xacro:property name="link_name" value="ir_intensity_${name}"/>

Commit message: Address comments

File: irobot_create_description/urdf/create3.urdf.xacro (robot description, xacro)
@@ -81,5 +81,4 @@
   <xacro:mouse
       parent_link="base_link"
-      mouse_seed="0.0"
       update_rate="${mouse_update_rate}">
     <origin xyz="0.1015 0.087 -0.055" rpy="0 0 ${-pi/4}"/>

File: irobot_create_description/urdf/sensors/mouse.urdf.xacro (robot description, xacro)
@@ -1,13 +1,10 @@
 <?xml version="1.0"?>
 <robot xmlns:xacro="http://ros.org/wiki/xacro">
-  <xacro:macro name="mouse" params="name:=mouse parent_link *origin visualize:=true noise_mean:=0.0
-                                            noise_var:=0.0 mouse_seed:=0.0 update_rate" >
+  <xacro:macro name="mouse" params="name:=mouse parent_link *origin update_rate" >
     <!-- Sensor settings -->
     <xacro:property name="mass" value="0.1" />
     <xacro:property name="length" value="0.008" /> <!-- Length -->
     <xacro:property name="radius" value="0.01" /> <!-- Radius -->
-    <!-- Visualization settings -->
-    <xacro:property name="color" value="Red" />
-    <joint name="mouse_joint" type="fixed">
+    <joint name="${name}_joint" type="fixed">
       <xacro:insert_block name="origin"/>
       <parent link="${parent_link}"/>
@@ -15,15 +12,8 @@
     </joint>
     <link name="${name}">
-      <xacro:if value="${visualize}">
-        <visual>
-          <geometry>
-            <cylinder length="${length}" radius="${radius}" />
-          </geometry>
-        </visual>
-      </xacro:if>
       <xacro:inertial_cylinder mass="${mass}" length="${length}" radius="${radius}" />
     </link>
     <gazebo>
-      <plugin name="gazebo_ros_optical_mouse" filename="libgazebo_ros_create_optical_mouse.so">
+      <plugin name="${name}_plugin" filename="libgazebo_ros_create_optical_mouse.so">
         <ros>
           <namespace>/</namespace>
@@ -31,16 +21,7 @@
         <update_rate>${update_rate}</update_rate>
         <link>${name}</link>
-        <gaussian_mean>${noise_mean}</gaussian_mean>
-        <gaussian_var>${noise_var}</gaussian_var>
-        <xacro:if value="${mouse_seed > 0}">
-          <!-- Only pass the value if it's possitive. Otherwise, use random. -->
-          <mouse_seed>${mouse_seed}</mouse_seed>
-        </xacro:if>
       </plugin>
     </gazebo>
-    <gazebo reference="o${name}" >
-      <material>Gazebo/${color}</material>
-    </gazebo>
-    <gazebo reference="mouse_joint" >
+    <gazebo reference="${name}_joint" >
       <preserveFixedJoint>true</preserveFixedJoint>
     </gazebo>

Commit message: Fix spawn pose of the robot

File: irobot_create_description/urdf/create3.urdf.xacro (robot description, xacro)
@@ -24,4 +24,5 @@
   <link name="base_footprint"/>
   <joint name="base_footprint_joint" type="fixed">
+    <origin xyz="0 0 0.065594" rpy="0 0.012796 0"/>
     <parent link="base_footprint"/>
     <child link="base_link" />

Commit message: Address comments

File: irobot_create_description/urdf/create3.urdf.xacro (robot description, xacro)
@@ -85,6 +85,19 @@
   <!-- IR intensity sensors -->
   <xacro:property name="ir_intensity_z_pos_cm" value="-0.7"/>
+  <!--
+  The robot uses 7 IR sensors in the front to execute a wall-following action
+  or reduce the speed when it detects something in front for safety reasons.
+  The arrangement of the sensors is defined in the following schema of the top
+  view of the robot:
+                          Front view
+                              |
+                              V
+                        front_center_left
+                front_left            front_right
+            left                                 right
+  side_left                                           side_right
+  -->
   <xacro:ir_intensity name="front_center_left">
-    <origin xyz="0.1540 -0.0000 ${ir_intensity_z_pos_cm*cm2m}"/>
+    <origin xyz="0.1540 0 ${ir_intensity_z_pos_cm*cm2m}"/>
   </xacro:ir_intensity>
   <xacro:ir_intensity name="front_center_right">

File: irobot_create_description/urdf/ir_intensity.urdf.xacro (robot description, xacro)
@@ -5,6 +5,6 @@
                params="name parent:=base_link
                        update_rate:=62.0 fov:=${10*deg2rad}
-                       min_range:=${25*mm2m} max_range:=${20*cm2m}
-                       visualize:=true *origin" >
+                       min_range:=${25*mm2m} max_range:=${200*mm2m}
+                       visualize:=false *origin" >
     <xacro:property name="link_name" value="ir_intensity_${name}"/>
     <joint name="${link_name}_joint" type="fixed">
@@ -44,4 +44,5 @@
           </range>
         </ray>
+        <!-- Noise is currently disabled -->
         <noise>
           <type>gaussian</type>

Commit message: default values for update rate and parent link

File: irobot_create_description/urdf/create3.urdf.xacro (robot description, xacro)
@@ -23,5 +23,4 @@
   <xacro:property name="wheel_drop_offset_z_mm"     value="3.5"/>
   <xacro:property name="wheel_drop_z"               value="${wheel_height_cm*cm2m + wheel_drop_offset_z_mm*mm2m}"/>
-  <xacro:property name="mouse_update_rate"          value="62" />
   <!-- Create 3 base definitions-->
   <link name="base_footprint"/>
@@ -78,8 +77,6 @@
     </plugin>
   </gazebo>
-  <!-- Optical mouse -->
-  <xacro:mouse
-      parent_link="base_link"
-      update_rate="${mouse_update_rate}">
+  <!-- mouse -->
+  <xacro:mouse>
     <origin xyz="0.1015 0.087 -0.055" rpy="0 0 ${-pi/4}"/>
   </xacro:mouse>

File: irobot_create_description/urdf/sensors/mouse.urdf.xacro (robot description, xacro)
@@ -1,5 +1,5 @@
 <?xml version="1.0"?>
 <robot xmlns:xacro="http://ros.org/wiki/xacro">
-  <xacro:macro name="mouse" params="name:=mouse parent_link *origin update_rate" >
+  <xacro:macro name="mouse" params="name:=mouse parent_link:=base_link *origin update_rate:=62" >
     <joint name="${name}_joint" type="fixed">
       <xacro:insert_block name="origin"/>

Commit message: renames mouse xacro to optical_mouse

File: irobot_create_description/urdf/create3.urdf.xacro (robot description, xacro)
@@ -4,5 +4,5 @@
   <xacro:include filename="$(find irobot_create_description)/urdf/caster.urdf.xacro" />
   <xacro:include filename="$(find irobot_create_description)/urdf/common_properties.urdf.xacro"/>
-  <xacro:include filename="$(find irobot_create_description)/urdf/sensors/mouse.urdf.xacro"/>
+  <xacro:include filename="$(find irobot_create_description)/urdf/sensors/optical_mouse.urdf.xacro"/>
   <xacro:include filename="$(find irobot_create_description)/urdf/wheel_with_wheeldrop.urdf.xacro" />
   <!-- MECHANICAL PROPERTIES -->
@@ -78,6 +78,6 @@
   </gazebo>
   <!-- mouse -->
-  <xacro:mouse>
+  <xacro:optical_mouse>
     <origin xyz="0.1015 0.087 -0.055" rpy="0 0 ${-pi/4}"/>
-  </xacro:mouse>
+  </xacro:optical_mouse>
 </robot>

File: irobot_create_description/urdf/sensors/optical_mouse.urdf.xacro (robot description, xacro)
@@ -1,5 +1,5 @@
 <?xml version="1.0"?>
 <robot xmlns:xacro="http://ros.org/wiki/xacro">
-  <xacro:macro name="mouse" params="name:=mouse parent_link:=base_link *origin update_rate:=62" >
+  <xacro:macro name="optical_mouse" params="name:=mouse parent_link:=base_link *origin update_rate:=62" >
     <joint name="${name}_joint" type="fixed">
       <xacro:insert_block name="origin"/>

Commit message: Round offset values to third decimal
Co-authored-by: Emiliano Borghi <creativa_eborghi@irobot.com>

File: irobot_create_description/urdf/create3.urdf.xacro (robot description, xacro)
@@ -24,5 +24,5 @@
   <link name="base_footprint"/>
   <joint name="base_footprint_joint" type="fixed">
-    <origin xyz="0 0 0.065594" rpy="0 0.012796 0"/>
+    <origin xyz="0 0 0.066" rpy="0 0.013 0"/>
     <parent link="base_footprint"/>
     <child link="base_link" />

Commit message: Adds IMU sensor

File: irobot_create_description/urdf/create3.urdf.xacro (robot description, xacro)
@@ -7,4 +7,5 @@
   <xacro:include filename="$(find irobot_create_description)/urdf/sensors/optical_mouse.urdf.xacro"/>
   <xacro:include filename="$(find irobot_create_description)/urdf/wheel_with_wheeldrop.urdf.xacro" />
+  <xacro:include filename="$(find irobot_create_description)/urdf/sensors/imu.urdf.xacro" />
   <!-- MECHANICAL PROPERTIES -->
   <xacro:property name="body_z_offset_cm"           value="-2.5" />
@@ -74,4 +75,8 @@
       rpy="${-pi/2} 0 0"/>
   </xacro:caster>
+  <!-- IMU -->
+  <xacro:imu_sensor>
+  <origin xyz="0.050613 0.043673 0.0202"/>
+</xacro:imu_sensor>
   <gazebo>
     <plugin name="gazebo_ros2_control" filename="libgazebo_ros2_control.so">
