Commit message: Change variable usage

File: irobot_create_description/urdf/create3.urdf.xacro (robot description, xacro)
@@ -84,5 +84,5 @@
   </xacro:optical_mouse>
   <!-- IR intensity sensors -->
-  <xacro:property name="ir_intensity_z_pos_cm" value="-0.7"/>
+  <xacro:property name="ir_intensity_z_pos" value="-0.7*cm2m"/>
   <!--
   The robot uses 7 IR sensors in the front to execute a wall-following action
@@ -99,23 +99,23 @@
   -->
   <xacro:ir_intensity name="front_center_left">
-    <origin xyz="0.1540 0 ${ir_intensity_z_pos_cm*cm2m}"/>
+    <origin xyz="0.1540 0 ${ir_intensity_z_pos}"/>
   </xacro:ir_intensity>
   <xacro:ir_intensity name="front_center_right">
-    <origin xyz="0.1396 -0.0651 ${ir_intensity_z_pos_cm*cm2m}" rpy="0 0 -0.436"/>
+    <origin xyz="0.1396 -0.0651 ${ir_intensity_z_pos}" rpy="0 0 -0.436"/>
   </xacro:ir_intensity>
   <xacro:ir_intensity name="front_left">
-    <origin xyz="0.1396 0.0651 ${ir_intensity_z_pos_cm*cm2m}" rpy="0 0 0.436"/>
+    <origin xyz="0.1396 0.0651 ${ir_intensity_z_pos}" rpy="0 0 0.436"/>
   </xacro:ir_intensity>
   <xacro:ir_intensity name="front_right">
-    <origin xyz="0.0990 -0.1180 ${ir_intensity_z_pos_cm*cm2m}" rpy="0 0 -0.873"/>
+    <origin xyz="0.0990 -0.1180 ${ir_intensity_z_pos}" rpy="0 0 -0.873"/>
   </xacro:ir_intensity>
   <xacro:ir_intensity name="left">
-    <origin xyz="0.0990 0.1180 ${ir_intensity_z_pos_cm*cm2m}" rpy="0 0 0.873"/>
+    <origin xyz="0.0990 0.1180 ${ir_intensity_z_pos}" rpy="0 0 0.873"/>
   </xacro:ir_intensity>
   <xacro:ir_intensity name="right">
-    <origin xyz="0.0399 -0.1488 ${ir_intensity_z_pos_cm*cm2m}" rpy="0 0 -1.309"/>
+    <origin xyz="0.0399 -0.1488 ${ir_intensity_z_pos}" rpy="0 0 -1.309"/>
   </xacro:ir_intensity>
   <xacro:ir_intensity name="side_left">
-    <origin xyz="0.0399 0.1488 ${ir_intensity_z_pos_cm*cm2m}" rpy="0 0 1.309"/>
+    <origin xyz="0.0399 0.1488 ${ir_intensity_z_pos}" rpy="0 0 1.309"/>
   </xacro:ir_intensity>
 </robot>

Commit message: minor changes

File: irobot_create_description/urdf/create3.urdf.xacro (robot description, xacro)
@@ -77,6 +77,6 @@
   <!-- IMU -->
   <xacro:imu_sensor>
-  <origin xyz="0.050613 0.043673 0.0202"/>
-</xacro:imu_sensor>
+    <origin xyz="0.050613 0.043673 0.0202"/>
+  </xacro:imu_sensor>
   <gazebo>
     <plugin name="gazebo_ros2_control" filename="libgazebo_ros2_control.so">

Commit message: sets frame_id to mouse

File: irobot_create_description/urdf/create3.urdf.xacro (robot description, xacro)
@@ -77,5 +77,5 @@
     </plugin>
   </gazebo>
-  <!-- mouse -->
+  <!-- Mouse -->
   <xacro:optical_mouse>
     <origin xyz="0.1015 0.087 -0.055" rpy="0 0 ${-pi/4}"/>

File: irobot_create_description/urdf/sensors/optical_mouse.urdf.xacro (robot description, xacro)
@@ -1,5 +1,5 @@
 <?xml version="1.0"?>
 <robot xmlns:xacro="http://ros.org/wiki/xacro">
-  <xacro:macro name="optical_mouse" params="name:=mouse parent_link:=base_link *origin update_rate:=62" >
+  <xacro:macro name="optical_mouse" params="name:=mouse parent_link:=base_link update_rate:=62 *origin" >
     <joint name="${name}_joint" type="fixed">
       <xacro:insert_block name="origin"/>

Commit message: Fix spawn pose of the robot (#16)
* Fix spawn pose of the robot

* Round offset values to third decimal

Co-authored-by: Emiliano Borghi <creativa_eborghi@irobot.com>

File: irobot_create_description/urdf/create3.urdf.xacro (robot description, xacro)
@@ -24,4 +24,5 @@
   <link name="base_footprint"/>
   <joint name="base_footprint_joint" type="fixed">
+    <origin xyz="0 0 0.066" rpy="0 0.013 0"/>
     <parent link="base_footprint"/>
     <child link="base_link" />

Commit message: fixup! Change variable usage

File: irobot_create_description/urdf/create3.urdf.xacro (robot description, xacro)
@@ -84,5 +84,5 @@
   </xacro:optical_mouse>
   <!-- IR intensity sensors -->
-  <xacro:property name="ir_intensity_z_pos" value="-0.7*cm2m"/>
+  <xacro:property name="ir_intensity_z_pos" value="${-0.7*cm2m}"/>
   <!--
   The robot uses 7 IR sensors in the front to execute a wall-following action

Commit message: Add mouse sensor (#5)
* diffdrive control package

* code cleanup

* address review comments

* included into irobot_create_gazebo and launched from there

* Address comments

* republish node

* Address comments

* Add resource directory

* creates irobot_create_toolbox package

* changes order of node execution

* correct flake8 errors

* new line at end of gitignore

* add dependency rcl_interfaces

* add test_depends

* adds uncrustify

* fix flake 8

* diffdrive control package

* address review comments

* included into irobot_create_gazebo and launched from there

* boilerplate code for mouse sensor

* Adds mouse sensor plugin

* updates publish rate

* Adds plugins package to CI

* integrated position

* mouse returns integrated position

* Update irobot_gazebo_plugins/include/irobot_gazebo_plugins/gazebo_ros_optical_mouse.h

* rebased on top of irobot_create_control

* alpha sort includes

* r and l to radius and length

* removes package irobot_gazebo_plugins and move files to irobot_create_gazebo_plugins

* Fixes dependency order

* adds uncrustify

* Fix copyright error

* applies mouse improvements

* removes unwanted files

* Fix Merge conflict

* Adds missing file

* Remove uncrustify

* Reverts changes by mistake

* Fix ci issues

* Fix clang_format issues

* rename optical mouse in xacros

* Address comments

* Uses inertial_dummy

* Addresses last bit of comments

* remaps topic

* clang_format fix

* default values for update rate and parent link

* renames mouse xacro to optical_mouse

* Update irobot_create_description/urdf/sensors/mouse.urdf.xacro

Co-authored-by: Emiliano Borghi <creativa_eborghi@irobot.com>

* removes gazebo_ros_pkgs

* remove srand() call

* Update irobot_create_gazebo_plugins/src/gazebo_ros_optical_mouse.cpp

Co-authored-by: Emiliano Borghi <creativa_eborghi@irobot.com>

* Update irobot_create_gazebo_plugins/src/gazebo_ros_optical_mouse.cpp

Co-authored-by: Emiliano Borghi <creativa_eborghi@irobot.com>

* Update irobot_create_gazebo_plugins/src/gazebo_ros_optical_mouse.cpp

Co-authored-by: Emiliano Borghi <creativa_eborghi@irobot.com>

* Update irobot_create_gazebo_plugins/include/irobot_create_gazebo_plugins/gazebo_ros_optical_mouse.hpp

Co-authored-by: Emiliano Borghi <creativa_eborghi@irobot.com>

* Update irobot_create_gazebo_plugins/src/gazebo_ros_optical_mouse.cpp

Co-authored-by: Emiliano Borghi <creativa_eborghi@irobot.com>

* Update irobot_create_gazebo_plugins/src/gazebo_ros_optical_mouse.cpp

Co-authored-by: Emiliano Borghi <creativa_eborghi@irobot.com>

* Update irobot_create_gazebo_plugins/src/gazebo_ros_optical_mouse.cpp

Co-authored-by: Emiliano Borghi <creativa_eborghi@irobot.com>

* renames link

* Fix linter

* sets frame_id to mouse

* Address comments

* default frame_id and last_squal values

* Update irobot_create_gazebo_plugins/src/gazebo_ros_optical_mouse.cpp

Co-authored-by: Emiliano Borghi <creativa_eborghi@irobot.com>

Co-authored-by: Emiliano Borghi <creativa_eborghi@irobot.com>

File: irobot_create_description/urdf/create3.urdf.xacro (robot description, xacro)
@@ -4,4 +4,5 @@
   <xacro:include filename="$(find irobot_create_description)/urdf/caster.urdf.xacro" />
   <xacro:include filename="$(find irobot_create_description)/urdf/common_properties.urdf.xacro"/>
+  <xacro:include filename="$(find irobot_create_description)/urdf/sensors/optical_mouse.urdf.xacro"/>
   <xacro:include filename="$(find irobot_create_description)/urdf/wheel_with_wheeldrop.urdf.xacro" />
   <!-- MECHANICAL PROPERTIES -->
@@ -21,4 +22,5 @@
   <xacro:property name="inertial_offset_x_cm"       value="1" />
   <xacro:property name="wheel_drop_offset_z_mm"     value="3.5"/>
+  <xacro:property name="wheel_drop_z"               value="${wheel_height_cm*cm2m + wheel_drop_offset_z_mm*mm2m}"/>
   <!-- Create 3 base definitions-->
   <link name="base_footprint"/>
@@ -49,5 +51,4 @@
   <xacro:bumper
       parent_link="base_link"
-      robot_type="create3"
       visual_mesh="file://$(find irobot_create_description)/meshes/bumper_visual.dae"
       collision_mesh="file://$(find irobot_create_description)/meshes/bumper_collision.dae">
@@ -61,5 +62,4 @@
   </xacro:bumper>
   <!-- Wheels with mechanical wheel drop -->
-  <xacro:property name="wheel_drop_z" value="${wheel_height_cm*cm2m + wheel_drop_offset_z_mm*mm2m}"/>
   <xacro:wheel_with_wheeldrop name="left">
     <origin xyz="0 ${distance_between_wheels_cm*cm2m/2} ${wheel_drop_z}" rpy="${-pi/2} 0 0"/>
@@ -78,3 +78,7 @@
     </plugin>
   </gazebo>
+  <!-- Mouse -->
+  <xacro:optical_mouse>
+    <origin xyz="0.1015 0.087 -0.055" rpy="0 0 ${-pi/4}"/>
+  </xacro:optical_mouse>
 </robot>

Commit message: Update irobot_create_description/urdf/create3.urdf.xacro
Co-authored-by: Emiliano Borghi <creativa_eborghi@irobot.com>

File: irobot_create_description/urdf/create3.urdf.xacro (robot description, xacro)
@@ -85,5 +85,5 @@
   </xacro:optical_mouse>
   <!-- Cliffs sensors -->
-  <xacro:property name="cliff_z"        value="${-4.5*cm2m}" />
+  <xacro:property name="cliff_z"  value="${-4.5*cm2m}" />
   <xacro:property name="cliff_center_x" value="${5.9*cm2m}"/>
   <xacro:property name="cliff_center_y" value="${14.6*cm2m}"/>

Commit message: Adds IMU (#17)
* Adds IMU sensor

* fix clang format

* minor changes

* removes gravity component from IMU reading

* makes joint fixed

* removes spaces

* inertial dummy to link

* Fix CMakeLists error

* Fix clang_format

* Fix cppcheck errors

* Update irobot_create_gazebo_plugins/src/gazebo_ros_imu.cpp

Co-authored-by: Emiliano Borghi <creativa_eborghi@irobot.com>

* Update irobot_create_gazebo_plugins/src/gazebo_ros_imu.cpp

Co-authored-by: Emiliano Borghi <creativa_eborghi@irobot.com>

* Update irobot_create_gazebo_plugins/src/gazebo_ros_imu.cpp

Co-authored-by: Emiliano Borghi <creativa_eborghi@irobot.com>

* Update irobot_create_gazebo_plugins/include/irobot_create_gazebo_plugins/gazebo_ros_imu.hpp

Co-authored-by: Emiliano Borghi <creativa_eborghi@irobot.com>

* Update irobot_create_gazebo_plugins/src/gazebo_ros_imu.cpp

Co-authored-by: Emiliano Borghi <creativa_eborghi@irobot.com>

* Apply some suggestions

* remove unnecessary code

* Add missing documentation line

* moves include to hpp file

* Extra line for clarity

* message is shared ptr

* Fix clang_format

* order includes alphabetically

Co-authored-by: Emiliano Borghi <creativa_eborghi@irobot.com>

File: irobot_create_description/urdf/create3.urdf.xacro (robot description, xacro)
@@ -4,4 +4,5 @@
   <xacro:include filename="$(find irobot_create_description)/urdf/caster.urdf.xacro" />
   <xacro:include filename="$(find irobot_create_description)/urdf/common_properties.urdf.xacro"/>
+  <xacro:include filename="$(find irobot_create_description)/urdf/sensors/imu.urdf.xacro" />
   <xacro:include filename="$(find irobot_create_description)/urdf/sensors/ir_intensity.urdf.xacro" />
   <xacro:include filename="$(find irobot_create_description)/urdf/sensors/optical_mouse.urdf.xacro"/>
@@ -74,4 +75,8 @@
       rpy="${-pi/2} 0 0"/>
   </xacro:caster>
+  <!-- IMU -->
+  <xacro:imu_sensor>
+    <origin xyz="0.050613 0.043673 0.0202"/>
+  </xacro:imu_sensor>
   <gazebo>
     <plugin name="gazebo_ros2_control" filename="libgazebo_ros2_control.so">

Commit message: Address Alexis comments

File: irobot_create_description/urdf/create3.urdf.xacro (robot description, xacro)
@@ -88,25 +88,25 @@
   <xacro:property name="cliff_center_x" value="${5.9*cm2m}"/>
   <xacro:property name="cliff_center_y" value="${14.6*cm2m}"/>
-  <xacro:property name="cliff_center_P" value="${80*deg2rad}"/>
-  <xacro:property name="cliff_center_Y" value="${65.3*deg2rad}"/>
+  <xacro:property name="cliff_center_pitch" value="${80*deg2rad}"/>
+  <xacro:property name="cliff_center_yaw" value="${65.3*deg2rad}"/>
   <xacro:property name="cliff_back_x" value="${-6.5*cm2m}"/>
   <xacro:property name="cliff_back_y" value="${14.5*cm2m}"/>
-  <xacro:property name="cliff_back_P" value="${80*deg2rad}"/>
-  <xacro:property name="cliff_back_Y" value="${167.4*deg2rad}"/>
+  <xacro:property name="cliff_back_pitch" value="${80*deg2rad}"/>
+  <xacro:property name="cliff_back_yaw" value="${167.4*deg2rad}"/>
   <xacro:cliff_sensor name="side_left">
     <origin xyz="${cliff_back_x} ${cliff_back_y} ${cliff_z}"
-            rpy="0 ${cliff_back_P} ${cliff_back_Y}"/>
+            rpy="0 ${cliff_back_pitch} ${cliff_back_yaw}"/>
   </xacro:cliff_sensor>
   <xacro:cliff_sensor name="side_right">
     <origin xyz="${cliff_back_x} ${- cliff_back_y} ${cliff_z}"
-            rpy="0 ${cliff_back_P} ${- cliff_back_Y}"/>
+            rpy="0 ${cliff_back_pitch} ${- cliff_back_yaw}"/>
   </xacro:cliff_sensor>
   <xacro:cliff_sensor name="front_left">
     <origin xyz="${cliff_center_x} ${cliff_center_y} ${cliff_z}"
-            rpy="0 ${cliff_center_P} ${cliff_center_Y}"/>
+            rpy="0 ${cliff_center_pitch} ${cliff_center_yaw}"/>
   </xacro:cliff_sensor>
   <xacro:cliff_sensor name="front_right">
     <origin xyz="${cliff_center_x} ${- cliff_center_y} ${cliff_z}"
-            rpy="0 ${cliff_center_P} ${- cliff_center_Y}"/>
+            rpy="0 ${cliff_center_pitch} ${- cliff_center_yaw}"/>
   </xacro:cliff_sensor>
   <!-- IR intensity sensors -->

File: irobot_create_description/urdf/sensors/cliff_sensor.urdf.xacro (robot description, xacro)
@@ -1,6 +1,6 @@
 <?xml version="1.0"?>
 <robot xmlns:xacro="http://ros.org/wiki/xacro">
-<xacro:macro name="cliff_sensor" params="name parent:=base_link detection_threshold:=${8*cm2m}
-                                           visualize:=false *origin">
+<xacro:macro name="cliff_sensor" params="name parent:=base_link
+                                         visualize:=false *origin">
   <!-- Sensor settings -->
   <xacro:property name="update_rate" value="62"/>
@@ -47,8 +47,8 @@
       <plugin name="${sensor_name}" filename="libgazebo_ros_create_cliff_sensor.so">
         <ros>
-          <namespace>cliff</namespace>
-          <remapping>~/out:=${name}/event</remapping>
+          <namespace>/</namespace>
+          <remapping>~/out:=${sensor_name}/event</remapping>
         </ros>
-        <detection_threshold>${detection_threshold}</detection_threshold>
+        <detection_threshold>${8*cm2m}</detection_threshold>
       </plugin>
     </sensor>

Commit message: Add cliff sensors (#9)
* Use realistic wheel drop model (#8)

* Use realistic wheeldrop model

* Rename parent argument to parent_link

* Add wheel drop plugin

* Enable C++ linter

* Fix linter

* Create irobot_create_gazebo_plugins

* Add env hooks

* Fix reminiscents of irobot_create_gazebo_plugins

* Address Alexis' comments

* Use 62 Hz by default

* Fix body inclination offset

* Fix plugin installation

* Remove env-hooks

* Address Rodri's comment

Add urdf cliff sensor to create3

Add cliff plugin

Addressed Emi and Rodr's comments

Enable linter

Address Emi Rodri and Alexis comments

Update irobot_create_description/urdf/cliffs_sensor.urdf.xacro

Co-authored-by: Emiliano Borghi <emiliano.borghi@gmail.com>

Address more comments

Update cliff sensor links and added to the create3

Fix remapping warning

Update ament checks  and emi comments

Addressed Emi's comments

Address more Emi's commment

Update cliff topic

Address Emi's functions

Improve the code with Emi comments

* Fix rebase issue

* Address Rodri comments

* Update argument to be camel_cased

* Add always_on flag

* Update irobot_create_description/urdf/create3.urdf.xacro

Co-authored-by: Emiliano Borghi <creativa_eborghi@irobot.com>

* Update irobot_create_description/urdf/sensors/cliff_sensor.urdf.xacro

Co-authored-by: Emiliano Borghi <creativa_eborghi@irobot.com>

* Update irobot_create_gazebo_plugins/CMakeLists.txt

Co-authored-by: Emiliano Borghi <creativa_eborghi@irobot.com>

* Update irobot_create_gazebo_plugins/src/gazebo_ros_cliff_sensor.cpp

Co-authored-by: Emiliano Borghi <creativa_eborghi@irobot.com>

* Last Emi comments

* Missing comments

* Update irobot_create_description/urdf/sensors/cliff_sensor.urdf.xacro

Co-authored-by: Rodrigo Causarano <46730379+rjcausarano@users.noreply.github.com>

* Update rodri comments

* Address Alexis comments

* Address Alexis comments

* Address Alexis comments

* Fix clang format

Co-authored-by: Emiliano Borghi <creativa_eborghi@irobot.com>
Co-authored-by: Luis Chico <lchico@ekumenlabs.com>
Co-authored-by: Rodrigo Causarano <46730379+rjcausarano@users.noreply.github.com>

File: irobot_create_description/urdf/create3.urdf.xacro (robot description, xacro)
@@ -4,4 +4,5 @@
   <xacro:include filename="$(find irobot_create_description)/urdf/caster.urdf.xacro" />
   <xacro:include filename="$(find irobot_create_description)/urdf/common_properties.urdf.xacro"/>
+  <xacro:include filename="$(find irobot_create_description)/urdf/sensors/cliff_sensor.urdf.xacro"/>
   <xacro:include filename="$(find irobot_create_description)/urdf/sensors/imu.urdf.xacro" />
   <xacro:include filename="$(find irobot_create_description)/urdf/sensors/ir_intensity.urdf.xacro" />
@@ -88,4 +89,30 @@
     <origin xyz="0.1015 0.087 -0.055" rpy="0 0 ${-pi/4}"/>
   </xacro:optical_mouse>
+  <!-- Cliffs sensors -->
+  <xacro:property name="cliff_z"  value="${-4.5*cm2m}" />
+  <xacro:property name="cliff_center_x" value="${5.9*cm2m}"/>
+  <xacro:property name="cliff_center_y" value="${14.6*cm2m}"/>
+  <xacro:property name="cliff_center_pitch" value="${80*deg2rad}"/>
+  <xacro:property name="cliff_center_yaw" value="${65.3*deg2rad}"/>
+  <xacro:property name="cliff_back_x" value="${-6.5*cm2m}"/>
+  <xacro:property name="cliff_back_y" value="${14.5*cm2m}"/>
+  <xacro:property name="cliff_back_pitch" value="${80*deg2rad}"/>
+  <xacro:property name="cliff_back_yaw" value="${167.4*deg2rad}"/>
+  <xacro:cliff_sensor name="side_left">
+    <origin xyz="${cliff_back_x} ${cliff_back_y} ${cliff_z}"
+            rpy="0 ${cliff_back_pitch} ${cliff_back_yaw}"/>
+  </xacro:cliff_sensor>
+  <xacro:cliff_sensor name="side_right">
+    <origin xyz="${cliff_back_x} ${- cliff_back_y} ${cliff_z}"
+            rpy="0 ${cliff_back_pitch} ${- cliff_back_yaw}"/>
+  </xacro:cliff_sensor>
+  <xacro:cliff_sensor name="front_left">
+    <origin xyz="${cliff_center_x} ${cliff_center_y} ${cliff_z}"
+            rpy="0 ${cliff_center_pitch} ${cliff_center_yaw}"/>
+  </xacro:cliff_sensor>
+  <xacro:cliff_sensor name="front_right">
+    <origin xyz="${cliff_center_x} ${- cliff_center_y} ${cliff_z}"
+            rpy="0 ${cliff_center_pitch} ${- cliff_center_yaw}"/>
+  </xacro:cliff_sensor>
   <!-- IR intensity sensors -->
   <xacro:property name="ir_intensity_z_pos" value="${-0.7*cm2m}"/>
