Commit message: Improve bumper and body inertias -- Cleaned up code

File: irobot_create_description/urdf/create3.urdf.xacro (robot description, xacro)
@@ -10,20 +10,19 @@
   <xacro:include filename="$(find irobot_create_description)/urdf/wheel_with_wheeldrop.urdf.xacro" />
   <!-- MECHANICAL PROPERTIES -->
-  <xacro:property name="body_z_offset_cm"           value="-2.5" />
-  <xacro:property name="body_collision_z_offset_cm" value="-1" />
-  <xacro:property name="body_mass_kg"               value="2.300" />
-  <xacro:property name="body_radius_cm"             value="16.4" />
-  <xacro:property name="body_length_cm"             value="6" />
-  <xacro:property name="bumper_mass_kg"             value="0.1" />
-  <xacro:property name="bumper_offset_z_cm"         value="-2.5" />
-  <xacro:property name="bumber_inertial_x_cm"       value="8" />
-  <xacro:property name="wheel_height_cm"            value="-2.75" />
-  <xacro:property name="distance_between_wheels_cm" value="23.3" />
-  <xacro:property name="caster_position_x_cm"       value="12.5" />
-  <xacro:property name="caster_position_y_cm"       value="0" />
-  <xacro:property name="caster_position_z_cm"       value="-5.4" />
-  <xacro:property name="inertial_offset_x_cm"       value="1" />
-  <xacro:property name="wheel_drop_offset_z_mm"     value="3.5"/>
-  <xacro:property name="wheel_drop_z"               value="${wheel_height_cm*cm2m + wheel_drop_offset_z_mm*mm2m}"/>
+  <xacro:property name="body_z_offset"           value="${-2.5*cm2m}" />
+  <xacro:property name="body_collision_z_offset" value="${-1*cm2m}" />
+  <xacro:property name="body_mass"               value="2.300" />
+  <xacro:property name="body_radius"             value="${16.4*cm2m}" />
+  <xacro:property name="body_length"             value="${6*cm2m}" />
+  <xacro:property name="bumper_mass"             value="0.1" />
+  <xacro:property name="bumper_offset_z"         value="${-2.5*cm2m}" />
+  <xacro:property name="bumber_inertial_x"       value="${8*cm2m}" />
+  <xacro:property name="bumper_inertial_z"       value="${2*cm2m}"/>
+  <xacro:property name="wheel_height"            value="${-2.75*cm2m}" />
+  <xacro:property name="distance_between_wheels" value="${23.3*cm2m}" />
+  <xacro:property name="caster_position_x"       value="${12.5*cm2m}" />
+  <xacro:property name="caster_position_z"       value="${-5.4*cm2m}" />
+  <xacro:property name="wheel_drop_offset_z"     value="${3.5*mm2m}"/>
+  <xacro:property name="wheel_drop_z"            value="${wheel_height + wheel_drop_offset_z}"/>
   <!-- Create 3 base definitions-->
   <link name="base_footprint"/>
@@ -35,5 +34,5 @@
   <link name="base_link">
     <visual>
-      <origin xyz="0 0 ${body_z_offset_cm*cm2m}" rpy="0 0 ${pi/2}"/>
+      <origin xyz="0 0 ${body_z_offset}" rpy="0 0 ${pi/2}"/>
       <geometry>
         <mesh filename="file://$(find irobot_create_description)/meshes/body_visual.dae" />
@@ -41,12 +40,11 @@
     </visual>
     <collision name="create3_base_collision">
-      <origin xyz="0 0 ${body_collision_z_offset_cm*cm2m}" rpy="0 0 ${pi/2}"/>
+      <origin xyz="0 0 ${body_collision_z_offset}" rpy="0 0 ${pi/2}"/>
       <geometry>
-        <cylinder length="${body_length_cm*cm2m}" radius="${body_radius_cm*cm2m}"/>
+        <cylinder length="${body_length}" radius="${body_radius}"/>
       </geometry>
     </collision>
-    <xacro:inertial_cylinder_with_pose mass="${body_mass_kg}" radius="${body_radius_cm*cm2m}"
-      length="${body_length_cm*cm2m}">
-      <origin xyz="${inertial_offset_x_cm*cm2m} 0 ${body_collision_z_offset_cm*cm2m}"/>
+    <xacro:inertial_cylinder_with_pose mass="${body_mass}" radius="${body_radius}" length="${body_length}">
+      <origin xyz="0 0 ${body_collision_z_offset}"/>
     </xacro:inertial_cylinder_with_pose>
   </link>
@@ -56,23 +54,22 @@
       visual_mesh="file://$(find irobot_create_description)/meshes/bumper_visual.dae"
       collision_mesh="file://$(find irobot_create_description)/meshes/bumper_collision.dae">
-    <origin xyz="0 0 ${bumper_offset_z_cm*cm2m}" rpy="0 0 ${pi/2}"/>
+    <origin xyz="0 0 ${bumper_offset_z}"/>
     <inertial>
-        <origin xyz="${bumber_inertial_x_cm*cm2m} 0 ${bumper_offset_z_cm*cm2m}"/>
-        <mass value="${bumper_mass_kg}"/>
-        <inertia ixx="0.0013483753405" ixy="0.0000000454352" ixz="0.0000014434849" iyy="0.0002521736852"
-          iyz="-0.0000000006721" izz="0.0015442525386"/>
-      </inertial>
+      <origin xyz="${bumber_inertial_x} 0 ${bumper_inertial_z}"/>
+      <mass value="${bumper_mass}"/>
+      <inertia ixx="0.0013483753405" ixy="0.0000000454352" ixz="0.0000014434849"
+               iyy="0.0002521736852" iyz="-0.0000000006721" izz="0.0015442525386"/>
+    </inertial>
   </xacro:bumper>
   <!-- Wheels with mechanical wheel drop -->
   <xacro:wheel_with_wheeldrop name="left">
-    <origin xyz="0 ${distance_between_wheels_cm*cm2m/2} ${wheel_drop_z}" rpy="${-pi/2} 0 0"/>
+    <origin xyz="0 ${distance_between_wheels/2} ${wheel_drop_z}" rpy="${-pi/2} 0 0"/>
   </xacro:wheel_with_wheeldrop>
   <xacro:wheel_with_wheeldrop name="right">
-    <origin xyz="0 ${-distance_between_wheels_cm*cm2m/2} ${wheel_drop_z}" rpy="${-pi/2} 0 0"/>
+    <origin xyz="0 ${-distance_between_wheels/2} ${wheel_drop_z}" rpy="${-pi/2} 0 0"/>
   </xacro:wheel_with_wheeldrop>
   <!-- Caster wheel -->
   <xacro:caster name="front_caster" parent_link="base_link">
-    <origin xyz="${caster_position_x_cm*cm2m} ${caster_position_y_cm*cm2m} ${caster_position_z_cm*cm2m}"
-      rpy="${-pi/2} 0 0"/>
+    <origin xyz="${caster_position_x} 0 ${caster_position_z}" rpy="${-pi/2} 0 0"/>
   </xacro:caster>
   <!-- IMU -->

Commit message: Docking status
Fix rebase conflicts

WARN_ONCE

model and link names via xacro parameters

Fix linters

All review comments addressed

updates gitignore

File: irobot_create_description/urdf/create3.urdf.xacro (robot description, xacro)
@@ -11,5 +11,5 @@
   <xacro:include filename="$(find irobot_create_description)/urdf/sensors/optical_mouse.urdf.xacro"/>
   <xacro:include filename="$(find irobot_create_description)/urdf/wheel_with_wheeldrop.urdf.xacro" />
-  <!-- MECHANICAL PROPERTIES -->
+  <!-- Mechanical properties -->
   <xacro:property name="body_z_offset"           value="${-2.5*cm2m}" />
   <xacro:property name="body_collision_z_offset" value="${1*cm2m}" />
@@ -27,4 +27,9 @@
   <xacro:property name="wheel_drop_offset_z"     value="${3.5*mm2m}"/>
   <xacro:property name="wheel_drop_z"            value="${wheel_height + wheel_drop_offset_z}"/>
+  <!-- Docking properties -->
+  <xacro:property name="robot_model_name" value="create3"/>
+  <xacro:property name="receiver_link_name" value="ir_omni"/>
+  <xacro:property name="dock_model_name" value="standard_dock"/>
+  <xacro:property name="emitter_link_name" value="halo_link"/>
   <!-- Create 3 base definition-->
   <origin xyz="0 0 0.064171"/>
@@ -160,7 +165,21 @@
   <xacro:property name="ir_omni_fov_rad" value="${220.0*deg2rad}"/>
   <xacro:property name="ir_front_facing_fov_rad" value="${pi/2}"/>
-  <xacro:ir_opcode_receivers sensor_0_range="0.01" sensor_0_fov="${ir_omni_fov_rad}"
+  <xacro:ir_opcode_receivers robot_model_name="${robot_model_name}" dock_model_name="${dock_model_name}" emitter_link_name="${emitter_link_name}" sensor_0_range="0.01" sensor_0_fov="${ir_omni_fov_rad}"
     sensor_1_range="0.5" sensor_1_fov="${ir_front_facing_fov_rad}" visualize="true" >
     <origin xyz="0.153 0 0.035"/>
   </xacro:ir_opcode_receivers>
+  <!-- Dock status -->
+  <gazebo>
+    <plugin name="dock_status_publisher" filename="libgazebo_ros_create_docking_status.so">
+      <ros>
+        <namespace>/</namespace>
+        <remapping>~/out:=dock</remapping>
+      </ros>
+      <update_rate>1.0</update_rate>
+      <robot_model_name>${robot_model_name}</robot_model_name>
+      <receiver_link_name>${receiver_link_name}</receiver_link_name>
+      <dock_model_name>${dock_model_name}</dock_model_name>
+      <emitter_link_name>${emitter_link_name}</emitter_link_name>
+    </plugin>
+  </gazebo>
 </robot>

File: irobot_create_description/urdf/sensors/ir_opcode_receivers.urdf.xacro (robot description, xacro)
@@ -2,4 +2,7 @@
 <robot xmlns:xacro="http://ros.org/wiki/xacro">
   <xacro:macro name="ir_opcode_receivers" params="name:=ir_omni
+                                                  robot_model_name
+                                                  dock_model_name
+                                                  emitter_link_name
                                                   parent:=base_link
                                                   sensor_0_fov
@@ -13,11 +16,11 @@
                                                   *origin" >
     <xacro:property name="joint_name" value="${name}_joint" />
-    <xacro:property name="link_name" value="${name}" />
+    <xacro:property name="receiver_link_name" value="${name}" />
     <joint name="${joint_name}" type="fixed">
       <xacro:insert_block name="origin" />
       <parent link="${parent}"/>
-      <child link="${link_name}"/>
+      <child link="${receiver_link_name}"/>
     </joint>
-    <link name="${link_name}">
+    <link name="${receiver_link_name}">
       <xacro:inertial_dummy />
     </link>
@@ -26,5 +29,5 @@
     <xacro:if value="${visualize}">
       <!-- Sensor 0 visualization -->
-      <gazebo reference="${link_name}">
+      <gazebo reference="${receiver_link_name}">
         <sensor type="ray" name="sensor_0">
             <always_on>true</always_on>
@@ -49,5 +52,5 @@
       </gazebo>
       <!-- Sensor 1 visualization -->
-      <gazebo reference="${link_name}">
+      <gazebo reference="${receiver_link_name}">
         <sensor type="ray" name="sensor_1">
             <always_on>true</always_on>
@@ -79,5 +82,8 @@
         </ros>
         <update_rate>${update_rate}</update_rate>
-        <link_name>${link_name}</link_name>
+        <robot_model_name>${robot_model_name}</robot_model_name>
+        <receiver_link_name>${receiver_link_name}</receiver_link_name>
+        <dock_model_name>${dock_model_name}</dock_model_name>
+        <emitter_link_name>${emitter_link_name}</emitter_link_name>
         <sensor_0_fov>${sensor_0_fov}</sensor_0_fov>
         <sensor_0_range>${sensor_0_range}</sensor_0_range>

Commit message: IR opcode
fixed plugin

dock with links

Halo detection

Force field detection working

Buoy detection working

Publishing IR opcodes for both Force field and buoys detection

Fix clang format

Improved Red, Green and Yellow Buoys detection

Update gazebo_ros_ir_opcode.cpp

Fixes red and green buoy detection

Fix corner case when buoys are detected when they shouldn't

Update irobot_create_description/urdf/create3.urdf.xacro

Co-authored-by: Emiliano Borghi <creativa_eborghi@irobot.com>

Update irobot_create_description/urdf/dock/ir_emitter.urdf.xacro

Co-authored-by: Emiliano Borghi <creativa_eborghi@irobot.com>

Update irobot_create_description/urdf/dock/standard.urdf.xacro

Co-authored-by: Emiliano Borghi <creativa_eborghi@irobot.com>

Update irobot_create_description/urdf/dock/standard.urdf.xacro

Co-authored-by: Emiliano Borghi <creativa_eborghi@irobot.com>

Update irobot_create_gazebo_plugins/src/gazebo_ros_ir_opcode.cpp

Co-authored-by: Emiliano Borghi <creativa_eborghi@irobot.com>

Fix update_rate

Created docking_manager class

Improvements to class

renames file

Both sensors in a single plugin to ensure publish rate

self review

Address peer review comments

Unused includes removed, fixed clang_format

Address comments

Stop using Vector2d to represent polar coordinates

const references for docking manager

Adding const where needed

Address code style comments

New opcodes logic

Updates IR opcode logic

publish rate at 31 Hz

corrects comment

Debug message instead of WARN

fix base_link

Lint errors

Fix lint

restore file

File: irobot_create_description/urdf/create3.urdf.xacro (robot description, xacro)
@@ -8,21 +8,22 @@
   <xacro:include filename="$(find irobot_create_description)/urdf/sensors/imu.urdf.xacro" />
   <xacro:include filename="$(find irobot_create_description)/urdf/sensors/ir_intensity.urdf.xacro" />
+  <xacro:include filename="$(find irobot_create_description)/urdf/sensors/ir_opcode_receivers.urdf.xacro" />
   <xacro:include filename="$(find irobot_create_description)/urdf/sensors/optical_mouse.urdf.xacro"/>
   <xacro:include filename="$(find irobot_create_description)/urdf/wheel_with_wheeldrop.urdf.xacro" />
   <!-- MECHANICAL PROPERTIES -->
-  <xacro:property name="body_z_offset"           value="${4.1*cm2m}" />
-  <xacro:property name="body_collision_z_offset" value="${1*cm2m}" />
+  <xacro:property name="body_z_offset"           value="${-2.5*cm2m}" />
+  <xacro:property name="body_collision_z_offset" value="${-1*cm2m}" />
   <xacro:property name="body_mass"               value="2.300" />
   <xacro:property name="body_radius"             value="${16.4*cm2m}" />
   <xacro:property name="body_length"             value="${6*cm2m}" />
   <xacro:property name="bumper_mass"             value="0.1" />
-  <xacro:property name="bumper_offset_z"         value="${4.1*cm2m}" />
+  <xacro:property name="bumper_offset_z"         value="${-2.5*cm2m}" />
   <xacro:property name="bumber_inertial_x"       value="${8*cm2m}" />
   <xacro:property name="bumper_inertial_z"       value="${2*cm2m}"/>
-  <xacro:property name="wheel_height"            value="${3.85*cm2m}" />
+  <xacro:property name="wheel_height"            value="${-2.75*cm2m}" />
   <xacro:property name="distance_between_wheels" value="${23.3*cm2m}" />
   <xacro:property name="caster_position_x"       value="${12.5*cm2m}" />
-  <xacro:property name="caster_position_z"       value="${1.2*cm2m}" />
-  <xacro:property name="wheel_drop_offset_z"     value="${3.1*mm2m}"/>
+  <xacro:property name="caster_position_z"       value="${-5.4*cm2m}" />
+  <xacro:property name="wheel_drop_offset_z"     value="${3.5*mm2m}"/>
   <xacro:property name="wheel_drop_z"            value="${wheel_height + wheel_drop_offset_z}"/>
   <!-- Create 3 base definition-->
@@ -155,3 +156,11 @@
       <origin xyz="0.06 0 0.08" rpy="0 ${-pi/2} 0"/>
   </xacro:button>
+  <!-- Omni IR receiver (sensor 0) parameters and Front-facing IR receiver (sensor 1) parameters -->
+  <xacro:property name="ir_omni_fov_rad" value="${360*deg2rad}"/>
+  <xacro:property name="ir_front_facing_fov_rad" value="${90*deg2rad}"/>
+  <xacro:property name="ir_samples" value="72"/>
+  <xacro:ir_opcode_receivers sensor_0_range="1" sensor_0_fov="${ir_omni_fov_rad}"
+    sensor_1_range="5" sensor_1_fov="${ir_front_facing_fov_rad}" samples="${ir_samples}" visualize="true" >
+    <origin xyz="0.153 0 0.035"/>
+  </xacro:ir_opcode_receivers>
 </robot>

File: irobot_create_description/urdf/dock/ir_emitter.urdf.xacro (robot description, xacro)
@@ -2,7 +2,8 @@
 <robot xmlns:xacro="http://ros.org/wiki/xacro">
   <xacro:macro name="ir_emitter" params="name parent:=base_link *origin
-                                         range code aperture
-                                         update_rate:=20 broadcast_rate:=64
-                                         ros_topic:=ir_emitter min_range:=0.50
+                                         range
+                                         aperture
+                                         update_rate:=1
+                                         min_range:=${7*cm2m}
                                          visualize:=false" >
     <!-- Physical link properties -->
@@ -27,5 +28,4 @@
     </link>
     <gazebo reference="${name}_link">
-      <preserveFixedJoint>true</preserveFixedJoint>
       <sensor type="ray" name="${name}">
         <always_on>true</always_on>
@@ -48,20 +48,7 @@
         </ray>
       </sensor>
-      <material>Gazebo/Red</material>
-      <static>true</static>
     </gazebo>
-    <gazebo>
-      <static>true</static>
-      <!-- MOVE TO SENSOR PLUGIN -->
-      <!-- <plugin name="${name}_ir_emitter" filename="libgazebo_ros_irobot_ir_emitter.so">
-        <link>${name}_link</link>
-        <topicName>${ros_topic}</topicName>
-        <emitterName>${name}</emitterName>
-        <emitterCode>${code}</emitterCode>
-        <rayAperture>${aperture}</rayAperture>
-        <rayRange>${range}</rayRange>
-        <updateRate>${update_rate}</updateRate>
-        <broadcastRate>${broadcast_rate}</broadcastRate>
-      </plugin> -->
+    <gazebo reference="${name}_joint" >
+      <preserveFixedJoint>true</preserveFixedJoint>
     </gazebo>
   </xacro:macro>

File: irobot_create_description/urdf/dock/standard.urdf.xacro (robot description, xacro)
@@ -3,9 +3,9 @@
   <xacro:include filename="$(find irobot_create_description)/urdf/common_properties.urdf.xacro"/>
   <xacro:include filename="$(find irobot_create_description)/urdf/dock/ir_emitter.urdf.xacro"/>
-  <xacro:property name="z_offset_mm" value="4.6"/>
-  <xacro:property name="link_name" value="std_dock_link"/>
+  <xacro:property name="z_offset" value="${4.6*mm2m}"/>
+  <xacro:property name="link_name"   value="std_dock_link"/>
   <link name="${link_name}">
     <visual>
-      <origin xyz="0 0 ${z_offset_mm*mm2m}"/>
+      <origin xyz="0 0 ${z_offset}"/>
       <geometry>
         <mesh filename="file://$(find irobot_create_description)/meshes/dock/visual.dae"/>
@@ -19,15 +19,9 @@
       </geometry>
     </collision>
+    <xacro:inertial_dummy />
   </link>
-  <gazebo reference="${link_name}">
-    <mu1>1.0</mu1>
-    <mu2>1.0</mu2>
-    <kp>1000000.0</kp>
-    <kd>1.0</kd>
-  </gazebo>
   <!-- Parameters for IR emitters -->
-  <xacro:property name="buoy_x" value="-0.037"/>
-  <xacro:property name="buoy_y" value="0.005"/>
-  <xacro:property name="buoy_z" value="${0.065 - (z_offset_mm*mm2m)}"/>
+  <xacro:property name="buoy_x" value="${-6*cm2m}"/>
+  <xacro:property name="buoy_z" value="${0.065 - z_offset}"/>
   <xacro:property name="halo_name"        value="halo"/>
   <xacro:property name="green_buoy_name"  value="green_buoy"/>
@@ -39,8 +33,8 @@
   <xacro:ir_emitter name="${green_buoy_name}"
                     parent="${link_name}"
-                    code="164"
                     aperture="${buoy_lateral_aperture}"
-                    range="1.524">
-    <origin xyz="${buoy_x} ${- buoy_y} ${buoy_z}"
+                    range="1.524"
+                    visualize="true">
+    <origin xyz="${buoy_x} 0 ${buoy_z}"
             rpy="0 0 ${- buoy_lateral_angle_yaw}"/>
   </xacro:ir_emitter>
@@ -48,8 +42,8 @@
   <xacro:ir_emitter name="${red_buoy_name}"
                     parent="${link_name}"
-                    code="168"
                     aperture="${buoy_lateral_aperture}"
-                    range="1.524">
-    <origin xyz="${buoy_x} ${buoy_y} ${buoy_z}"
+                    range="1.524"
+                    visualize="true">
+    <origin xyz="${buoy_x} 0 ${buoy_z}"
             rpy="0 0 ${buoy_lateral_angle_yaw}"/>
   </xacro:ir_emitter>
@@ -57,7 +51,7 @@
   <xacro:ir_emitter name="${yellow_buoy_name}"
                     parent="${link_name}"
-                    code="172"
                     aperture="${10*deg2rad}"
-                    range="1.2192">
+                    range="1.2192"
+                    visualize="true">
     <origin xyz="${buoy_x} 0 ${buoy_z}"/>
   </xacro:ir_emitter>
@@ -65,19 +59,11 @@
   <xacro:ir_emitter name="${halo_name}"
                     parent="${link_name}"
-                    code="161"
                     aperture="360"
-                    range="0.6096">
-    <origin xyz="-0.052 0 ${0.095 - (z_offset_mm*mm2m)}"/>
+                    range="0.6096"
+                    visualize="true">
+    <origin xyz="${buoy_x} 0 ${0.095 - z_offset}"/>
   </xacro:ir_emitter>
-  <xacro:property name="real_behavior" value="$(arg real_behavior)"/>
   <gazebo>
-      <static>true</static>
-      <!-- <plugin name="gazebo_ros_dock_manager" filename="libgazebo_ros_irobot_dock_manager.so">
-        <halo>${halo_name}</halo>
-        <greenBuoy>${green_buoy_name}</greenBuoy>
-        <redBuoy>${red_buoy_name}</redBuoy>
-        <yellowBuoy>${yellow_buoy_name}</yellowBuoy>
-        <realBehavior>${real_behavior}</realBehavior>
-      </plugin> -->
-    </gazebo>
+    <static>true</static>
+  </gazebo>
 </robot>

Commit message: Updates the positions of the cliff sensors. This also solves the trigger error.

File: irobot_create_description/urdf/create3.urdf.xacro (robot description, xacro)
@@ -81,11 +81,11 @@
   </xacro:optical_mouse>
   <!-- Cliffs sensors -->
-  <xacro:property name="cliff_z"  value="${-4.5*cm2m}" />
-  <xacro:property name="cliff_center_x" value="${5.9*cm2m}"/>
-  <xacro:property name="cliff_center_y" value="${14.6*cm2m}"/>
+  <xacro:property name="cliff_z"  value="${2.1*cm2m}" />
+  <xacro:property name="cliff_center_x" value="${4.5*cm2m}"/>
+  <xacro:property name="cliff_center_y" value="${16*cm2m}"/>
   <xacro:property name="cliff_center_pitch" value="${80*deg2rad}"/>
   <xacro:property name="cliff_center_yaw" value="${65.3*deg2rad}"/>
-  <xacro:property name="cliff_back_x" value="${-6.5*cm2m}"/>
-  <xacro:property name="cliff_back_y" value="${14.5*cm2m}"/>
+  <xacro:property name="cliff_back_x" value="${-14.5*cm2m}"/>
+  <xacro:property name="cliff_back_y" value="${6*cm2m}"/>
   <xacro:property name="cliff_back_pitch" value="${80*deg2rad}"/>
   <xacro:property name="cliff_back_yaw" value="${167.4*deg2rad}"/>

Commit message: Corrects the cliff sensors position.

File: irobot_create_description/urdf/create3.urdf.xacro (robot description, xacro)
@@ -82,10 +82,10 @@
   <!-- Cliffs sensors -->
   <xacro:property name="cliff_z"  value="${2.1*cm2m}" />
-  <xacro:property name="cliff_center_x" value="${4.5*cm2m}"/>
-  <xacro:property name="cliff_center_y" value="${16*cm2m}"/>
+  <xacro:property name="cliff_center_x" value="${16*cm2m}"/>
+  <xacro:property name="cliff_center_y" value="${4.5*cm2m}"/>
   <xacro:property name="cliff_center_pitch" value="${80*deg2rad}"/>
   <xacro:property name="cliff_center_yaw" value="${65.3*deg2rad}"/>
-  <xacro:property name="cliff_back_x" value="${-14.5*cm2m}"/>
-  <xacro:property name="cliff_back_y" value="${6*cm2m}"/>
+  <xacro:property name="cliff_back_x" value="${6*cm2m}"/>
+  <xacro:property name="cliff_back_y" value="${-14.5*cm2m}"/>
   <xacro:property name="cliff_back_pitch" value="${80*deg2rad}"/>
   <xacro:property name="cliff_back_yaw" value="${167.4*deg2rad}"/>
