Commit message: Luis' comments

File: irobot_create_description/urdf/create3.urdf.xacro (robot description, xacro)
@@ -159,7 +159,6 @@
   <xacro:property name="ir_omni_fov_rad" value="${360*deg2rad}"/>
   <xacro:property name="ir_front_facing_fov_rad" value="${90*deg2rad}"/>
-  <xacro:property name="ir_samples" value="72"/>
   <xacro:ir_opcode_receivers sensor_0_range="1" sensor_0_fov="${ir_omni_fov_rad}"
-    sensor_1_range="5" sensor_1_fov="${ir_front_facing_fov_rad}" samples="${ir_samples}" visualize="true" >
+    sensor_1_range="5" sensor_1_fov="${ir_front_facing_fov_rad}" visualize="true" >
     <origin xyz="0.153 0 0.035"/>
   </xacro:ir_opcode_receivers>

File: irobot_create_description/urdf/dock/ir_emitter.urdf.xacro (robot description, xacro)
@@ -4,5 +4,5 @@
                                          range
                                          aperture
-                                         update_rate:=1
+                                         update_rate:=1.0
                                          min_range:=${7*cm2m}
                                          visualize:=false" >
@@ -18,35 +18,32 @@
     </joint>
     <link name="${name}_link">
-      <xacro:if value="${visualize}">
-        <visual>
-          <geometry>
-            <box size="${x} ${y} ${z}" />
-          </geometry>
-        </visual>
-      </xacro:if>
       <xacro:inertial_cuboid mass="${mass}" x="${x}" y="${y}" z="${z}" />
     </link>
-    <gazebo reference="${name}_link">
-      <sensor type="ray" name="${name}">
-        <always_on>true</always_on>
-        <update_rate>${update_rate}</update_rate>
-        <visualize>${visualize}</visualize>
-        <ray>
-          <scan>
-            <horizontal>
-              <samples>50</samples>
-              <resolution>1</resolution>
-              <min_angle>-${aperture/2}</min_angle>
-              <max_angle>${aperture/2}</max_angle>
-              </horizontal>
-          </scan>
-            <range>
-            <min>${min_range}</min>
-            <max>${range}</max>
-            <resolution>0.01</resolution>
-          </range>
-        </ray>
-      </sensor>
-    </gazebo>
+    <!-- This ray is not attached to any plugin, it is only used for aesthetic and debugging purposes
+    only when the visualize flag is set. No need for high update rates. -->
+    <xacro:if value="${visualize}">
+      <gazebo reference="${name}_link">
+        <sensor type="ray" name="${name}">
+          <always_on>true</always_on>
+          <update_rate>${update_rate}</update_rate>
+          <visualize>${visualize}</visualize>
+          <ray>
+            <scan>
+              <horizontal>
+                <samples>50</samples>
+                <resolution>1</resolution>
+                <min_angle>-${aperture/2}</min_angle>
+                <max_angle>${aperture/2}</max_angle>
+                </horizontal>
+            </scan>
+              <range>
+              <min>${min_range}</min>
+              <max>${range}</max>
+              <resolution>0.01</resolution>
+            </range>
+          </ray>
+        </sensor>
+      </gazebo>
+    </xacro:if>
     <gazebo reference="${name}_joint" >
       <preserveFixedJoint>true</preserveFixedJoint>

File: irobot_create_description/urdf/sensors/ir_opcode_receivers.urdf.xacro (robot description, xacro)
@@ -7,5 +7,5 @@
                                                   sensor_1_fov
                                                   sensor_1_range
-                                                  samples
+                                                  samples:=50
                                                   min_range:=0.015
                                                   update_rate:=31
@@ -22,50 +22,54 @@
       <xacro:inertial_dummy />
     </link>
-    <!-- Sensor 0 visualization -->
-    <gazebo reference="${link_name}">
-      <sensor type="ray" name="sensor_0">
-          <always_on>true</always_on>
-          <update_rate>1</update_rate>
-          <visualize>${visualize}</visualize>
-          <ray>
-              <scan>
-                  <horizontal>
-                      <samples>${samples}</samples>
-                      <resolution>1</resolution>
-                      <min_angle>${-sensor_0_fov/2}</min_angle>
-                      <max_angle>${sensor_0_fov/2}</max_angle>
-                  </horizontal>
-              </scan>
-              <range>
-                  <min>${min_range}</min>
-                  <max>${sensor_0_range}</max>
-                  <resolution>0.01</resolution>
-              </range>
-          </ray>
-      </sensor>
-    </gazebo>
-    <!-- Sensor 1 visualization -->
-    <gazebo reference="${link_name}">
-      <sensor type="ray" name="sensor_1">
-          <always_on>true</always_on>
-          <update_rate>1</update_rate>
-          <visualize>${visualize}</visualize>
-          <ray>
-              <scan>
-                  <horizontal>
-                      <samples>${samples}</samples>
-                      <resolution>1</resolution>
-                      <min_angle>${-sensor_1_fov/2}</min_angle>
-                      <max_angle>${sensor_1_fov/2}</max_angle>
-                  </horizontal>
-              </scan>
-              <range>
-                  <min>${min_range}</min>
-                  <max>${sensor_1_range}</max>
-                  <resolution>0.01</resolution>
-              </range>
-          </ray>
-      </sensor>
-    </gazebo>
+    <!-- These rays are only used for aesthetic and debugging purposes only when the visualize flag is set.
+    This there is no need for high update rates. -->
+    <xacro:if value="${visualize}">
+      <!-- Sensor 0 visualization -->
+      <gazebo reference="${link_name}">
+        <sensor type="ray" name="sensor_0">
+            <always_on>true</always_on>
+            <update_rate>1</update_rate>
+            <visualize>${visualize}</visualize>
+            <ray>
+                <scan>
+                    <horizontal>
+                        <samples>${samples}</samples>
+                        <resolution>1</resolution>
+                        <min_angle>${-sensor_0_fov/2}</min_angle>
+                        <max_angle>${sensor_0_fov/2}</max_angle>
+                    </horizontal>
+                </scan>
+                <range>
+                    <min>${min_range}</min>
+                    <max>${sensor_0_range}</max>
+                    <resolution>0.01</resolution>
+                </range>
+            </ray>
+        </sensor>
+      </gazebo>
+      <!-- Sensor 1 visualization -->
+      <gazebo reference="${link_name}">
+        <sensor type="ray" name="sensor_1">
+            <always_on>true</always_on>
+            <update_rate>1</update_rate>
+            <visualize>${visualize}</visualize>
+            <ray>
+                <scan>
+                    <horizontal>
+                        <samples>${samples}</samples>
+                        <resolution>1</resolution>
+                        <min_angle>${-sensor_1_fov/2}</min_angle>
+                        <max_angle>${sensor_1_fov/2}</max_angle>
+                    </horizontal>
+                </scan>
+                <range>
+                    <min>${min_range}</min>
+                    <max>${sensor_1_range}</max>
+                    <resolution>0.01</resolution>
+                </range>
+            </ray>
+        </sensor>
+      </gazebo>
+    </xacro:if>
     <gazebo>
       <plugin name="${name}_plugin" filename="libgazebo_ros_create_ir_opcodes.so">

Commit message: Address comments

File: irobot_create_description/urdf/create3.urdf.xacro (robot description, xacro)
@@ -24,8 +24,9 @@
   <xacro:property name="distance_between_wheels" value="${23.3*cm2m}" />
   <xacro:property name="caster_position_x"       value="${12.5*cm2m}" />
-  <xacro:property name="caster_position_z"       value="${-5.4*cm2m}" />
+  <xacro:property name="caster_position_z"       value="${-5.55*cm2m}" />
   <xacro:property name="wheel_drop_offset_z"     value="${3.5*mm2m}"/>
   <xacro:property name="wheel_drop_z"            value="${wheel_height + wheel_drop_offset_z}"/>
   <!-- Create 3 base definition-->
+  <origin xyz="0 0 0.064171"/>
   <link name="base_link">
     <visual>
@@ -157,6 +158,6 @@
   </xacro:button>
   <!-- Omni IR receiver (sensor 0) parameters and Front-facing IR receiver (sensor 1) parameters -->
-  <xacro:property name="ir_omni_fov_rad" value="${360*deg2rad}"/>
-  <xacro:property name="ir_front_facing_fov_rad" value="${90*deg2rad}"/>
+  <xacro:property name="ir_omni_fov_rad" value="${2*pi}"/>
+  <xacro:property name="ir_front_facing_fov_rad" value="${pi/2}"/>
   <xacro:ir_opcode_receivers sensor_0_range="1" sensor_0_fov="${ir_omni_fov_rad}"
     sensor_1_range="5" sensor_1_fov="${ir_front_facing_fov_rad}" visualize="true" >

File: irobot_create_description/urdf/dock/standard.urdf.xacro (robot description, xacro)
@@ -3,6 +3,6 @@
   <xacro:include filename="$(find irobot_create_description)/urdf/common_properties.urdf.xacro"/>
   <xacro:include filename="$(find irobot_create_description)/urdf/dock/ir_emitter.urdf.xacro"/>
-  <xacro:property name="z_offset" value="${4.6*mm2m}"/>
-  <xacro:property name="link_name"   value="std_dock_link"/>
+  <xacro:property name="z_offset"  value="${4.6*mm2m}"/>
+  <xacro:property name="link_name" value="std_dock_link"/>
   <link name="${link_name}">
     <visual>

Commit message: Fix collision offset

File: irobot_create_description/urdf/create3.urdf.xacro (robot description, xacro)
@@ -13,5 +13,5 @@
   <!-- MECHANICAL PROPERTIES -->
   <xacro:property name="body_z_offset"           value="${-2.5*cm2m}" />
-  <xacro:property name="body_collision_z_offset" value="${-1*cm2m}" />
+  <xacro:property name="body_collision_z_offset" value="${1*cm2m}" />
   <xacro:property name="body_mass"               value="2.300" />
   <xacro:property name="body_radius"             value="${16.4*cm2m}" />

Commit message: Publish IR Opcodes (#66)
* IR opcode

fixed plugin

dock with links

Halo detection

Force field detection working

Buoy detection working

Publishing IR opcodes for both Force field and buoys detection

Fix clang format

Improved Red, Green and Yellow Buoys detection

Update gazebo_ros_ir_opcode.cpp

Fixes red and green buoy detection

Fix corner case when buoys are detected when they shouldn't

Update irobot_create_description/urdf/create3.urdf.xacro

Co-authored-by: Emiliano Borghi <creativa_eborghi@irobot.com>

Update irobot_create_description/urdf/dock/ir_emitter.urdf.xacro

Co-authored-by: Emiliano Borghi <creativa_eborghi@irobot.com>

Update irobot_create_description/urdf/dock/standard.urdf.xacro

Co-authored-by: Emiliano Borghi <creativa_eborghi@irobot.com>

Update irobot_create_description/urdf/dock/standard.urdf.xacro

Co-authored-by: Emiliano Borghi <creativa_eborghi@irobot.com>

Update irobot_create_gazebo_plugins/src/gazebo_ros_ir_opcode.cpp

Co-authored-by: Emiliano Borghi <creativa_eborghi@irobot.com>

Fix update_rate

Created docking_manager class

Improvements to class

renames file

Both sensors in a single plugin to ensure publish rate

self review

Address peer review comments

Unused includes removed, fixed clang_format

Address comments

Stop using Vector2d to represent polar coordinates

const references for docking manager

Adding const where needed

Address code style comments

New opcodes logic

Updates IR opcode logic

publish rate at 31 Hz

corrects comment

Debug message instead of WARN

fix base_link

Lint errors

Fix lint

restore file

* Luis' comments

* Another review address round

* Rename functions

* modify SensorParams

* Fix lint

* rename variable

* Address comments

* Fix collision offset

File: irobot_create_description/urdf/create3.urdf.xacro (robot description, xacro)
@@ -8,8 +8,9 @@
   <xacro:include filename="$(find irobot_create_description)/urdf/sensors/imu.urdf.xacro" />
   <xacro:include filename="$(find irobot_create_description)/urdf/sensors/ir_intensity.urdf.xacro" />
+  <xacro:include filename="$(find irobot_create_description)/urdf/sensors/ir_opcode_receivers.urdf.xacro" />
   <xacro:include filename="$(find irobot_create_description)/urdf/sensors/optical_mouse.urdf.xacro"/>
   <xacro:include filename="$(find irobot_create_description)/urdf/wheel_with_wheeldrop.urdf.xacro" />
   <!-- MECHANICAL PROPERTIES -->
-  <xacro:property name="body_z_offset"           value="${4.1*cm2m}" />
+  <xacro:property name="body_z_offset"           value="${-2.5*cm2m}" />
   <xacro:property name="body_collision_z_offset" value="${1*cm2m}" />
   <xacro:property name="body_mass"               value="2.300" />
@@ -17,14 +18,15 @@
   <xacro:property name="body_length"             value="${6*cm2m}" />
   <xacro:property name="bumper_mass"             value="0.1" />
-  <xacro:property name="bumper_offset_z"         value="${4.1*cm2m}" />
+  <xacro:property name="bumper_offset_z"         value="${-2.5*cm2m}" />
   <xacro:property name="bumber_inertial_x"       value="${8*cm2m}" />
   <xacro:property name="bumper_inertial_z"       value="${2*cm2m}"/>
-  <xacro:property name="wheel_height"            value="${3.85*cm2m}" />
+  <xacro:property name="wheel_height"            value="${-2.75*cm2m}" />
   <xacro:property name="distance_between_wheels" value="${23.3*cm2m}" />
   <xacro:property name="caster_position_x"       value="${12.5*cm2m}" />
-  <xacro:property name="caster_position_z"       value="${1.2*cm2m}" />
-  <xacro:property name="wheel_drop_offset_z"     value="${3.1*mm2m}"/>
+  <xacro:property name="caster_position_z"       value="${-5.55*cm2m}" />
+  <xacro:property name="wheel_drop_offset_z"     value="${3.5*mm2m}"/>
   <xacro:property name="wheel_drop_z"            value="${wheel_height + wheel_drop_offset_z}"/>
   <!-- Create 3 base definition-->
+  <origin xyz="0 0 0.064171"/>
   <link name="base_link">
     <visual>
@@ -155,3 +157,10 @@
       <origin xyz="0.06 0 0.08" rpy="0 ${-pi/2} 0"/>
   </xacro:button>
+  <!-- Omni IR receiver (sensor 0) parameters and Front-facing IR receiver (sensor 1) parameters -->
+  <xacro:property name="ir_omni_fov_rad" value="${2*pi}"/>
+  <xacro:property name="ir_front_facing_fov_rad" value="${pi/2}"/>
+  <xacro:ir_opcode_receivers sensor_0_range="1" sensor_0_fov="${ir_omni_fov_rad}"
+    sensor_1_range="5" sensor_1_fov="${ir_front_facing_fov_rad}" visualize="true" >
+    <origin xyz="0.153 0 0.035"/>
+  </xacro:ir_opcode_receivers>
 </robot>

File: irobot_create_description/urdf/dock/ir_emitter.urdf.xacro (robot description, xacro)
@@ -2,7 +2,8 @@
 <robot xmlns:xacro="http://ros.org/wiki/xacro">
   <xacro:macro name="ir_emitter" params="name parent:=base_link *origin
-                                         range code aperture
-                                         update_rate:=20 broadcast_rate:=64
-                                         ros_topic:=ir_emitter min_range:=0.50
+                                         range
+                                         aperture
+                                         update_rate:=1.0
+                                         min_range:=${7*cm2m}
                                          visualize:=false" >
     <!-- Physical link properties -->
@@ -17,51 +18,34 @@
     </joint>
     <link name="${name}_link">
-      <xacro:if value="${visualize}">
-        <visual>
-          <geometry>
-            <box size="${x} ${y} ${z}" />
-          </geometry>
-        </visual>
-      </xacro:if>
       <xacro:inertial_cuboid mass="${mass}" x="${x}" y="${y}" z="${z}" />
     </link>
-    <gazebo reference="${name}_link">
+    <!-- This ray is not attached to any plugin, it is only used for aesthetic and debugging purposes
+    only when the visualize flag is set. No need for high update rates. -->
+    <xacro:if value="${visualize}">
+      <gazebo reference="${name}_link">
+        <sensor type="ray" name="${name}">
+          <always_on>true</always_on>
+          <update_rate>${update_rate}</update_rate>
+          <visualize>${visualize}</visualize>
+          <ray>
+            <scan>
+              <horizontal>
+                <samples>50</samples>
+                <resolution>1</resolution>
+                <min_angle>-${aperture/2}</min_angle>
+                <max_angle>${aperture/2}</max_angle>
+                </horizontal>
+            </scan>
+              <range>
+              <min>${min_range}</min>
+              <max>${range}</max>
+              <resolution>0.01</resolution>
+            </range>
+          </ray>
+        </sensor>
+      </gazebo>
+    </xacro:if>
+    <gazebo reference="${name}_joint" >
       <preserveFixedJoint>true</preserveFixedJoint>
-      <sensor type="ray" name="${name}">
-        <always_on>true</always_on>
-        <update_rate>${update_rate}</update_rate>
-        <visualize>${visualize}</visualize>
-        <ray>
-          <scan>
-            <horizontal>
-              <samples>50</samples>
-              <resolution>1</resolution>
-              <min_angle>-${aperture/2}</min_angle>
-              <max_angle>${aperture/2}</max_angle>
-              </horizontal>
-          </scan>
-            <range>
-            <min>${min_range}</min>
-            <max>${range}</max>
-            <resolution>0.01</resolution>
-          </range>
-        </ray>
-      </sensor>
-      <material>Gazebo/Red</material>
-      <static>true</static>
-    </gazebo>
-    <gazebo>
-      <static>true</static>
-      <!-- MOVE TO SENSOR PLUGIN -->
-      <!-- <plugin name="${name}_ir_emitter" filename="libgazebo_ros_irobot_ir_emitter.so">
-        <link>${name}_link</link>
-        <topicName>${ros_topic}</topicName>
-        <emitterName>${name}</emitterName>
-        <emitterCode>${code}</emitterCode>
-        <rayAperture>${aperture}</rayAperture>
-        <rayRange>${range}</rayRange>
-        <updateRate>${update_rate}</updateRate>
-        <broadcastRate>${broadcast_rate}</broadcastRate>
-      </plugin> -->
     </gazebo>
   </xacro:macro>

File: irobot_create_description/urdf/dock/standard.urdf.xacro (robot description, xacro)
@@ -3,9 +3,9 @@
   <xacro:include filename="$(find irobot_create_description)/urdf/common_properties.urdf.xacro"/>
   <xacro:include filename="$(find irobot_create_description)/urdf/dock/ir_emitter.urdf.xacro"/>
-  <xacro:property name="z_offset_mm" value="4.6"/>
+  <xacro:property name="z_offset"  value="${4.6*mm2m}"/>
   <xacro:property name="link_name" value="std_dock_link"/>
   <link name="${link_name}">
     <visual>
-      <origin xyz="0 0 ${z_offset_mm*mm2m}"/>
+      <origin xyz="0 0 ${z_offset}"/>
       <geometry>
         <mesh filename="file://$(find irobot_create_description)/meshes/dock/visual.dae"/>
@@ -19,15 +19,9 @@
       </geometry>
     </collision>
+    <xacro:inertial_dummy />
   </link>
-  <gazebo reference="${link_name}">
-    <mu1>1.0</mu1>
-    <mu2>1.0</mu2>
-    <kp>1000000.0</kp>
-    <kd>1.0</kd>
-  </gazebo>
   <!-- Parameters for IR emitters -->
-  <xacro:property name="buoy_x" value="-0.037"/>
-  <xacro:property name="buoy_y" value="0.005"/>
-  <xacro:property name="buoy_z" value="${0.065 - (z_offset_mm*mm2m)}"/>
+  <xacro:property name="buoy_x" value="${-6*cm2m}"/>
+  <xacro:property name="buoy_z" value="${0.065 - z_offset}"/>
   <xacro:property name="halo_name"        value="halo"/>
   <xacro:property name="green_buoy_name"  value="green_buoy"/>
@@ -39,8 +33,8 @@
   <xacro:ir_emitter name="${green_buoy_name}"
                     parent="${link_name}"
-                    code="164"
                     aperture="${buoy_lateral_aperture}"
-                    range="1.524">
-    <origin xyz="${buoy_x} ${- buoy_y} ${buoy_z}"
+                    range="1.524"
+                    visualize="true">
+    <origin xyz="${buoy_x} 0 ${buoy_z}"
             rpy="0 0 ${- buoy_lateral_angle_yaw}"/>
   </xacro:ir_emitter>
@@ -48,8 +42,8 @@
   <xacro:ir_emitter name="${red_buoy_name}"
                     parent="${link_name}"
-                    code="168"
                     aperture="${buoy_lateral_aperture}"
-                    range="1.524">
-    <origin xyz="${buoy_x} ${buoy_y} ${buoy_z}"
+                    range="1.524"
+                    visualize="true">
+    <origin xyz="${buoy_x} 0 ${buoy_z}"
             rpy="0 0 ${buoy_lateral_angle_yaw}"/>
   </xacro:ir_emitter>
@@ -57,7 +51,7 @@
   <xacro:ir_emitter name="${yellow_buoy_name}"
                     parent="${link_name}"
-                    code="172"
                     aperture="${10*deg2rad}"
-                    range="1.2192">
+                    range="1.2192"
+                    visualize="true">
     <origin xyz="${buoy_x} 0 ${buoy_z}"/>
   </xacro:ir_emitter>
@@ -65,19 +59,11 @@
   <xacro:ir_emitter name="${halo_name}"
                     parent="${link_name}"
-                    code="161"
                     aperture="360"
-                    range="0.6096">
-    <origin xyz="-0.052 0 ${0.095 - (z_offset_mm*mm2m)}"/>
+                    range="0.6096"
+                    visualize="true">
+    <origin xyz="${buoy_x} 0 ${0.095 - z_offset}"/>
   </xacro:ir_emitter>
-  <xacro:property name="real_behavior" value="$(arg real_behavior)"/>
   <gazebo>
-      <static>true</static>
-      <!-- <plugin name="gazebo_ros_dock_manager" filename="libgazebo_ros_irobot_dock_manager.so">
-        <halo>${halo_name}</halo>
-        <greenBuoy>${green_buoy_name}</greenBuoy>
-        <redBuoy>${red_buoy_name}</redBuoy>
-        <yellowBuoy>${yellow_buoy_name}</yellowBuoy>
-        <realBehavior>${real_behavior}</realBehavior>
-      </plugin> -->
-    </gazebo>
+    <static>true</static>
+  </gazebo>
 </robot>
