Commit message: Tune sensor and emitter params to give both sensors shorter range with omni shorter than directional sensor.  Decrease omni FOV to account for Create3 shell.

File: irobot_create_description/urdf/create3.urdf.xacro (robot description, xacro)
@@ -158,8 +158,8 @@
   </xacro:button>
   <!-- Omni IR receiver (sensor 0) parameters and Front-facing IR receiver (sensor 1) parameters -->
-  <xacro:property name="ir_omni_fov_rad" value="${2*pi}"/>
+  <xacro:property name="ir_omni_fov_rad" value="${220.0*pi/180.0}"/>
   <xacro:property name="ir_front_facing_fov_rad" value="${pi/2}"/>
-  <xacro:ir_opcode_receivers sensor_0_range="1" sensor_0_fov="${ir_omni_fov_rad}"
-    sensor_1_range="5" sensor_1_fov="${ir_front_facing_fov_rad}" visualize="true" >
+  <xacro:ir_opcode_receivers sensor_0_range="0.01" sensor_0_fov="${ir_omni_fov_rad}"
+    sensor_1_range="0.5" sensor_1_fov="${ir_front_facing_fov_rad}" visualize="true" >
     <origin xyz="0.153 0 0.035"/>
   </xacro:ir_opcode_receivers>

File: irobot_create_description/urdf/dock/standard.urdf.xacro (robot description, xacro)
@@ -34,5 +34,5 @@
                     parent="${link_name}"
                     aperture="${buoy_lateral_aperture}"
-                    range="1.524"
+                    range="1.0"
                     visualize="true">
     <origin xyz="${buoy_x} 0 ${buoy_z}"
@@ -43,5 +43,5 @@
                     parent="${link_name}"
                     aperture="${buoy_lateral_aperture}"
-                    range="1.524"
+                    range="1.0"
                     visualize="true">
     <origin xyz="${buoy_x} 0 ${buoy_z}"
@@ -52,5 +52,5 @@
                     parent="${link_name}"
                     aperture="${10*deg2rad}"
-                    range="1.2192"
+                    range="1.0"
                     visualize="true">
     <origin xyz="${buoy_x} 0 ${buoy_z}"/>

Commit message: update math with constant

File: irobot_create_description/urdf/create3.urdf.xacro (robot description, xacro)
@@ -158,5 +158,5 @@
   </xacro:button>
   <!-- Omni IR receiver (sensor 0) parameters and Front-facing IR receiver (sensor 1) parameters -->
-  <xacro:property name="ir_omni_fov_rad" value="${220.0*pi/180.0}"/>
+  <xacro:property name="ir_omni_fov_rad" value="${220.0*deg2rad}"/>
   <xacro:property name="ir_front_facing_fov_rad" value="${pi/2}"/>
   <xacro:ir_opcode_receivers sensor_0_range="0.01" sensor_0_fov="${ir_omni_fov_rad}"

Commit message: tune opcodes / add placeholder safety params (#94)
* Tune sensor and emitter params to give both sensors shorter range with omni shorter than directional sensor.  Decrease omni FOV to account for Create3 shell.

* Add safety_override and max_speed placeholder params.  Not able to update for now

File: irobot_create_description/urdf/create3.urdf.xacro (robot description, xacro)
@@ -158,8 +158,8 @@
   </xacro:button>
   <!-- Omni IR receiver (sensor 0) parameters and Front-facing IR receiver (sensor 1) parameters -->
-  <xacro:property name="ir_omni_fov_rad" value="${2*pi}"/>
+  <xacro:property name="ir_omni_fov_rad" value="${220.0*deg2rad}"/>
   <xacro:property name="ir_front_facing_fov_rad" value="${pi/2}"/>
-  <xacro:ir_opcode_receivers sensor_0_range="1" sensor_0_fov="${ir_omni_fov_rad}"
-    sensor_1_range="5" sensor_1_fov="${ir_front_facing_fov_rad}" visualize="true" >
+  <xacro:ir_opcode_receivers sensor_0_range="0.01" sensor_0_fov="${ir_omni_fov_rad}"
+    sensor_1_range="0.5" sensor_1_fov="${ir_front_facing_fov_rad}" visualize="true" >
     <origin xyz="0.153 0 0.035"/>
   </xacro:ir_opcode_receivers>

Commit message: merge conflict after rebase

File: irobot_create_description/urdf/create3.urdf.xacro (robot description, xacro)
@@ -168,4 +168,6 @@
     emitter_link_name="${emitter_link_name}" sensor_0_range="0.01" sensor_0_fov="${ir_omni_fov_rad}"
     sensor_1_range="0.5" sensor_1_fov="${ir_front_facing_fov_rad}" >
+    <origin xyz="0.153 0 0.035"/>
+  </xacro:ir_opcode_receivers>
   <!-- Dock status -->
   <gazebo>

Commit message: Fix cliffs and bumper (#99)
* fix bumper and cliffs

* merge conflict after rebase

File: irobot_create_description/urdf/create3.urdf.xacro (robot description, xacro)
@@ -88,5 +88,5 @@
   </xacro:optical_mouse>
   <!-- Cliffs sensors -->
-  <xacro:property name="cliff_z"  value="${2.1*cm2m}" />
+  <xacro:property name="cliff_z"  value="${-4.5*cm2m}" />
   <xacro:property name="cliff_center_x" value="${16*cm2m}"/>
   <xacro:property name="cliff_center_y" value="${4.5*cm2m}"/>
@@ -165,6 +165,7 @@
   <xacro:property name="ir_omni_fov_rad" value="${220.0*deg2rad}"/>
   <xacro:property name="ir_front_facing_fov_rad" value="${pi/2}"/>
-  <xacro:ir_opcode_receivers robot_model_name="${robot_model_name}" dock_model_name="${dock_model_name}" emitter_link_name="${emitter_link_name}" sensor_0_range="0.01" sensor_0_fov="${ir_omni_fov_rad}"
-    sensor_1_range="0.5" sensor_1_fov="${ir_front_facing_fov_rad}" visualize="true" >
+  <xacro:ir_opcode_receivers robot_model_name="${robot_model_name}" dock_model_name="${dock_model_name}"
+    emitter_link_name="${emitter_link_name}" sensor_0_range="0.01" sensor_0_fov="${ir_omni_fov_rad}"
+    sensor_1_range="0.5" sensor_1_fov="${ir_front_facing_fov_rad}" >
     <origin xyz="0.153 0 0.035"/>
   </xacro:ir_opcode_receivers>

Commit message: Remove base_link offset; Added it to each of its children

File: irobot_create_description/urdf/create3.urdf.xacro (robot description, xacro)
@@ -27,4 +27,5 @@
   <xacro:property name="wheel_drop_offset_z"     value="${3.5*mm2m}"/>
   <xacro:property name="wheel_drop_z"            value="${wheel_height + wheel_drop_offset_z}"/>
+  <xacro:property name="base_link_z_offset"     value="${6.42*cm2m}"/>
   <!-- Docking properties -->
   <xacro:property name="robot_model_name" value="create3"/>
@@ -33,8 +34,7 @@
   <xacro:property name="emitter_link_name" value="halo_link"/>
   <!-- Create 3 base definition-->
-  <origin xyz="0 0 0.064171"/>
   <link name="base_link">
     <visual>
-      <origin xyz="0 0 ${body_z_offset}" rpy="0 0 ${pi/2}"/>
+      <origin xyz="0 0 ${body_z_offset + base_link_z_offset}" rpy="0 0 ${pi/2}"/>
       <geometry>
         <mesh filename="file://$(find irobot_create_description)/meshes/body_visual.dae" />
@@ -42,5 +42,5 @@
     </visual>
     <collision name="create3_base_collision">
-      <origin xyz="0 0 ${body_z_offset + body_collision_z_offset}" rpy="0 0 ${pi/2}"/>
+      <origin xyz="0 0 ${body_z_offset + body_collision_z_offset  + base_link_z_offset}" rpy="0 0 ${pi/2}"/>
       <geometry>
         <cylinder length="${body_length}" radius="${body_radius}"/>
@@ -48,5 +48,5 @@
     </collision>
     <xacro:inertial_cylinder_with_pose mass="${body_mass}" radius="${body_radius}" length="${body_length}">
-      <origin xyz="0 0 ${body_collision_z_offset}"/>
+      <origin xyz="0 0 ${body_collision_z_offset + base_link_z_offset}"/>
     </xacro:inertial_cylinder_with_pose>
   </link>
@@ -55,5 +55,5 @@
       visual_mesh="file://$(find irobot_create_description)/meshes/bumper_visual.dae"
       collision_mesh="file://$(find irobot_create_description)/meshes/bumper_collision.dae">
-    <origin xyz="0 0 ${bumper_offset_z}"/>
+    <origin xyz="0 0 ${bumper_offset_z  + base_link_z_offset}"/>
     <inertial>
       <origin xyz="${bumber_inertial_x} 0 ${bumper_inertial_z}"/>
@@ -65,16 +65,16 @@
   <!-- Wheels with mechanical wheel drop -->
   <xacro:wheel_with_wheeldrop name="left">
-    <origin xyz="0 ${distance_between_wheels/2} ${wheel_drop_z}" rpy="${-pi/2} 0 0"/>
+    <origin xyz="0 ${distance_between_wheels/2} ${wheel_drop_z  + base_link_z_offset}" rpy="${-pi/2} 0 0"/>
   </xacro:wheel_with_wheeldrop>
   <xacro:wheel_with_wheeldrop name="right">
-    <origin xyz="0 ${-distance_between_wheels/2} ${wheel_drop_z}" rpy="${-pi/2} 0 0"/>
+    <origin xyz="0 ${-distance_between_wheels/2} ${wheel_drop_z  + base_link_z_offset}" rpy="${-pi/2} 0 0"/>
   </xacro:wheel_with_wheeldrop>
   <!-- Caster wheel -->
   <xacro:caster name="front_caster" parent_link="base_link">
-    <origin xyz="${caster_position_x} 0 ${caster_position_z}" rpy="${-pi/2} 0 0"/>
+    <origin xyz="${caster_position_x} 0 ${caster_position_z  + base_link_z_offset}" rpy="${-pi/2} 0 0"/>
   </xacro:caster>
   <!-- IMU -->
   <xacro:imu_sensor>
-    <origin xyz="0.050613 0.043673 0.0202"/>
+    <origin xyz="0.050613 0.043673 ${0.0202 + base_link_z_offset}"/>
   </xacro:imu_sensor>
   <gazebo>
@@ -85,5 +85,5 @@
   <!-- Mouse -->
   <xacro:optical_mouse>
-    <origin xyz="0.1015 0.087 -0.055" rpy="0 0 ${-pi/4}"/>
+    <origin xyz="0.1015 0.087 ${-0.055 + base_link_z_offset}" rpy="0 0 ${-pi/4}"/>
   </xacro:optical_mouse>
   <!-- Cliffs sensors -->
@@ -98,17 +98,17 @@
   <xacro:property name="cliff_back_yaw" value="${167.4*deg2rad}"/>
   <xacro:cliff_sensor name="side_left">
-    <origin xyz="${cliff_back_x} ${cliff_back_y} ${cliff_z}"
+    <origin xyz="${cliff_back_x} ${cliff_back_y} ${cliff_z + base_link_z_offset}"
             rpy="0 ${cliff_back_pitch} ${cliff_back_yaw}"/>
   </xacro:cliff_sensor>
   <xacro:cliff_sensor name="side_right">
-    <origin xyz="${cliff_back_x} ${- cliff_back_y} ${cliff_z}"
+    <origin xyz="${cliff_back_x} ${- cliff_back_y} ${cliff_z + base_link_z_offset}"
             rpy="0 ${cliff_back_pitch} ${- cliff_back_yaw}"/>
   </xacro:cliff_sensor>
   <xacro:cliff_sensor name="front_left">
-    <origin xyz="${cliff_center_x} ${cliff_center_y} ${cliff_z}"
+    <origin xyz="${cliff_center_x} ${cliff_center_y} ${cliff_z + base_link_z_offset}"
             rpy="0 ${cliff_center_pitch} ${cliff_center_yaw}"/>
   </xacro:cliff_sensor>
   <xacro:cliff_sensor name="front_right">
-    <origin xyz="${cliff_center_x} ${- cliff_center_y} ${cliff_z}"
+    <origin xyz="${cliff_center_x} ${- cliff_center_y} ${cliff_z + base_link_z_offset}"
             rpy="0 ${cliff_center_pitch} ${- cliff_center_yaw}"/>
   </xacro:cliff_sensor>
@@ -129,36 +129,36 @@
   -->
   <xacro:ir_intensity name="front_center_left">
-    <origin xyz="0.1540 0 ${ir_intensity_z_pos}"/>
+    <origin xyz="0.1540 0 ${ir_intensity_z_pos + base_link_z_offset}"/>
   </xacro:ir_intensity>
   <xacro:ir_intensity name="front_center_right">
-    <origin xyz="0.1396 -0.0651 ${ir_intensity_z_pos}" rpy="0 0 -0.436"/>
+    <origin xyz="0.1396 -0.0651 ${ir_intensity_z_pos + base_link_z_offset}" rpy="0 0 -0.436"/>
   </xacro:ir_intensity>
   <xacro:ir_intensity name="front_left">
-    <origin xyz="0.1396 0.0651 ${ir_intensity_z_pos}" rpy="0 0 0.436"/>
+    <origin xyz="0.1396 0.0651 ${ir_intensity_z_pos + base_link_z_offset}" rpy="0 0 0.436"/>
   </xacro:ir_intensity>
   <xacro:ir_intensity name="front_right">
-    <origin xyz="0.0990 -0.1180 ${ir_intensity_z_pos}" rpy="0 0 -0.873"/>
+    <origin xyz="0.0990 -0.1180 ${ir_intensity_z_pos + base_link_z_offset}" rpy="0 0 -0.873"/>
   </xacro:ir_intensity>
   <xacro:ir_intensity name="left">
-    <origin xyz="0.0990 0.1180 ${ir_intensity_z_pos}" rpy="0 0 0.873"/>
+    <origin xyz="0.0990 0.1180 ${ir_intensity_z_pos + base_link_z_offset}" rpy="0 0 0.873"/>
   </xacro:ir_intensity>
   <xacro:ir_intensity name="right">
-    <origin xyz="0.0399 -0.1488 ${ir_intensity_z_pos}" rpy="0 0 -1.309"/>
+    <origin xyz="0.0399 -0.1488 ${ir_intensity_z_pos + base_link_z_offset}" rpy="0 0 -1.309"/>
   </xacro:ir_intensity>
   <xacro:ir_intensity name="side_left">
-    <origin xyz="0.0399 0.1488 ${ir_intensity_z_pos}" rpy="0 0 1.309"/>
+    <origin xyz="0.0399 0.1488 ${ir_intensity_z_pos + base_link_z_offset}" rpy="0 0 1.309"/>
   </xacro:ir_intensity>
   <!-- Buttons -->
   <xacro:button
       name="button_1">
-      <origin xyz="0.06 0.37 0.08" rpy="0 ${-pi/2} 0"/>
+      <origin xyz="0.06 0.37 ${0.08 + base_link_z_offset}" rpy="0 ${-pi/2} 0"/>
   </xacro:button>
   <xacro:button
       name="button_2">
-      <origin xyz="0.06 -0.37 0.08" rpy="0 ${-pi/2} 0"/>
+      <origin xyz="0.06 -0.37 ${0.08 + base_link_z_offset}" rpy="0 ${-pi/2} 0"/>
   </xacro:button>
   <xacro:button
       name="button_power">
-      <origin xyz="0.06 0 0.08" rpy="0 ${-pi/2} 0"/>
+      <origin xyz="0.06 0 ${0.08 + base_link_z_offset}" rpy="0 ${-pi/2} 0"/>
   </xacro:button>
   <!-- Omni IR receiver (sensor 0) parameters and Front-facing IR receiver (sensor 1) parameters -->
@@ -168,5 +168,5 @@
     emitter_link_name="${emitter_link_name}" sensor_0_range="0.01" sensor_0_fov="${ir_omni_fov_rad}"
     sensor_1_range="0.5" sensor_1_fov="${ir_front_facing_fov_rad}" >
-    <origin xyz="0.153 0 0.035"/>
+    <origin xyz="0.153 0 ${0.035 + base_link_z_offset}"/>
   </xacro:ir_opcode_receivers>
   <!-- Dock status -->

Commit message: Remove base_link offset; Added it to each of its children (#105)

File: irobot_create_description/urdf/create3.urdf.xacro (robot description, xacro)
@@ -27,4 +27,5 @@
   <xacro:property name="wheel_drop_offset_z"     value="${3.5*mm2m}"/>
   <xacro:property name="wheel_drop_z"            value="${wheel_height + wheel_drop_offset_z}"/>
+  <xacro:property name="base_link_z_offset"     value="${6.42*cm2m}"/>
   <!-- Docking properties -->
   <xacro:property name="robot_model_name" value="create3"/>
@@ -33,8 +34,7 @@
   <xacro:property name="emitter_link_name" value="halo_link"/>
   <!-- Create 3 base definition-->
-  <origin xyz="0 0 0.064171"/>
   <link name="base_link">
     <visual>
-      <origin xyz="0 0 ${body_z_offset}" rpy="0 0 ${pi/2}"/>
+      <origin xyz="0 0 ${body_z_offset + base_link_z_offset}" rpy="0 0 ${pi/2}"/>
       <geometry>
         <mesh filename="file://$(find irobot_create_description)/meshes/body_visual.dae" />
@@ -42,5 +42,5 @@
     </visual>
     <collision name="create3_base_collision">
-      <origin xyz="0 0 ${body_z_offset + body_collision_z_offset}" rpy="0 0 ${pi/2}"/>
+      <origin xyz="0 0 ${body_z_offset + body_collision_z_offset  + base_link_z_offset}" rpy="0 0 ${pi/2}"/>
       <geometry>
         <cylinder length="${body_length}" radius="${body_radius}"/>
@@ -48,5 +48,5 @@
     </collision>
     <xacro:inertial_cylinder_with_pose mass="${body_mass}" radius="${body_radius}" length="${body_length}">
-      <origin xyz="0 0 ${body_collision_z_offset}"/>
+      <origin xyz="0 0 ${body_collision_z_offset + base_link_z_offset}"/>
     </xacro:inertial_cylinder_with_pose>
   </link>
@@ -55,5 +55,5 @@
       visual_mesh="file://$(find irobot_create_description)/meshes/bumper_visual.dae"
       collision_mesh="file://$(find irobot_create_description)/meshes/bumper_collision.dae">
-    <origin xyz="0 0 ${bumper_offset_z}"/>
+    <origin xyz="0 0 ${bumper_offset_z  + base_link_z_offset}"/>
     <inertial>
       <origin xyz="${bumber_inertial_x} 0 ${bumper_inertial_z}"/>
@@ -65,16 +65,16 @@
   <!-- Wheels with mechanical wheel drop -->
   <xacro:wheel_with_wheeldrop name="left">
-    <origin xyz="0 ${distance_between_wheels/2} ${wheel_drop_z}" rpy="${-pi/2} 0 0"/>
+    <origin xyz="0 ${distance_between_wheels/2} ${wheel_drop_z  + base_link_z_offset}" rpy="${-pi/2} 0 0"/>
   </xacro:wheel_with_wheeldrop>
   <xacro:wheel_with_wheeldrop name="right">
-    <origin xyz="0 ${-distance_between_wheels/2} ${wheel_drop_z}" rpy="${-pi/2} 0 0"/>
+    <origin xyz="0 ${-distance_between_wheels/2} ${wheel_drop_z  + base_link_z_offset}" rpy="${-pi/2} 0 0"/>
   </xacro:wheel_with_wheeldrop>
   <!-- Caster wheel -->
   <xacro:caster name="front_caster" parent_link="base_link">
-    <origin xyz="${caster_position_x} 0 ${caster_position_z}" rpy="${-pi/2} 0 0"/>
+    <origin xyz="${caster_position_x} 0 ${caster_position_z  + base_link_z_offset}" rpy="${-pi/2} 0 0"/>
   </xacro:caster>
   <!-- IMU -->
   <xacro:imu_sensor>
-    <origin xyz="0.050613 0.043673 0.0202"/>
+    <origin xyz="0.050613 0.043673 ${0.0202 + base_link_z_offset}"/>
   </xacro:imu_sensor>
   <gazebo>
@@ -85,5 +85,5 @@
   <!-- Mouse -->
   <xacro:optical_mouse>
-    <origin xyz="0.1015 0.087 -0.055" rpy="0 0 ${-pi/4}"/>
+    <origin xyz="0.1015 0.087 ${-0.055 + base_link_z_offset}" rpy="0 0 ${-pi/4}"/>
   </xacro:optical_mouse>
   <!-- Cliffs sensors -->
@@ -98,17 +98,17 @@
   <xacro:property name="cliff_back_yaw" value="${167.4*deg2rad}"/>
   <xacro:cliff_sensor name="side_left">
-    <origin xyz="${cliff_back_x} ${cliff_back_y} ${cliff_z}"
+    <origin xyz="${cliff_back_x} ${cliff_back_y} ${cliff_z + base_link_z_offset}"
             rpy="0 ${cliff_back_pitch} ${cliff_back_yaw}"/>
   </xacro:cliff_sensor>
   <xacro:cliff_sensor name="side_right">
-    <origin xyz="${cliff_back_x} ${- cliff_back_y} ${cliff_z}"
+    <origin xyz="${cliff_back_x} ${- cliff_back_y} ${cliff_z + base_link_z_offset}"
             rpy="0 ${cliff_back_pitch} ${- cliff_back_yaw}"/>
   </xacro:cliff_sensor>
   <xacro:cliff_sensor name="front_left">
-    <origin xyz="${cliff_center_x} ${cliff_center_y} ${cliff_z}"
+    <origin xyz="${cliff_center_x} ${cliff_center_y} ${cliff_z + base_link_z_offset}"
             rpy="0 ${cliff_center_pitch} ${cliff_center_yaw}"/>
   </xacro:cliff_sensor>
   <xacro:cliff_sensor name="front_right">
-    <origin xyz="${cliff_center_x} ${- cliff_center_y} ${cliff_z}"
+    <origin xyz="${cliff_center_x} ${- cliff_center_y} ${cliff_z + base_link_z_offset}"
             rpy="0 ${cliff_center_pitch} ${- cliff_center_yaw}"/>
   </xacro:cliff_sensor>
@@ -129,36 +129,36 @@
   -->
   <xacro:ir_intensity name="front_center_left">
-    <origin xyz="0.1540 0 ${ir_intensity_z_pos}"/>
+    <origin xyz="0.1540 0 ${ir_intensity_z_pos + base_link_z_offset}"/>
   </xacro:ir_intensity>
   <xacro:ir_intensity name="front_center_right">
-    <origin xyz="0.1396 -0.0651 ${ir_intensity_z_pos}" rpy="0 0 -0.436"/>
+    <origin xyz="0.1396 -0.0651 ${ir_intensity_z_pos + base_link_z_offset}" rpy="0 0 -0.436"/>
   </xacro:ir_intensity>
   <xacro:ir_intensity name="front_left">
-    <origin xyz="0.1396 0.0651 ${ir_intensity_z_pos}" rpy="0 0 0.436"/>
+    <origin xyz="0.1396 0.0651 ${ir_intensity_z_pos + base_link_z_offset}" rpy="0 0 0.436"/>
   </xacro:ir_intensity>
   <xacro:ir_intensity name="front_right">
-    <origin xyz="0.0990 -0.1180 ${ir_intensity_z_pos}" rpy="0 0 -0.873"/>
+    <origin xyz="0.0990 -0.1180 ${ir_intensity_z_pos + base_link_z_offset}" rpy="0 0 -0.873"/>
   </xacro:ir_intensity>
   <xacro:ir_intensity name="left">
-    <origin xyz="0.0990 0.1180 ${ir_intensity_z_pos}" rpy="0 0 0.873"/>
+    <origin xyz="0.0990 0.1180 ${ir_intensity_z_pos + base_link_z_offset}" rpy="0 0 0.873"/>
   </xacro:ir_intensity>
   <xacro:ir_intensity name="right">
-    <origin xyz="0.0399 -0.1488 ${ir_intensity_z_pos}" rpy="0 0 -1.309"/>
+    <origin xyz="0.0399 -0.1488 ${ir_intensity_z_pos + base_link_z_offset}" rpy="0 0 -1.309"/>
   </xacro:ir_intensity>
   <xacro:ir_intensity name="side_left">
-    <origin xyz="0.0399 0.1488 ${ir_intensity_z_pos}" rpy="0 0 1.309"/>
+    <origin xyz="0.0399 0.1488 ${ir_intensity_z_pos + base_link_z_offset}" rpy="0 0 1.309"/>
   </xacro:ir_intensity>
   <!-- Buttons -->
   <xacro:button
       name="button_1">
-      <origin xyz="0.06 0.37 0.08" rpy="0 ${-pi/2} 0"/>
+      <origin xyz="0.06 0.37 ${0.08 + base_link_z_offset}" rpy="0 ${-pi/2} 0"/>
   </xacro:button>
   <xacro:button
       name="button_2">
-      <origin xyz="0.06 -0.37 0.08" rpy="0 ${-pi/2} 0"/>
+      <origin xyz="0.06 -0.37 ${0.08 + base_link_z_offset}" rpy="0 ${-pi/2} 0"/>
   </xacro:button>
   <xacro:button
       name="button_power">
-      <origin xyz="0.06 0 0.08" rpy="0 ${-pi/2} 0"/>
+      <origin xyz="0.06 0 ${0.08 + base_link_z_offset}" rpy="0 ${-pi/2} 0"/>
   </xacro:button>
   <!-- Omni IR receiver (sensor 0) parameters and Front-facing IR receiver (sensor 1) parameters -->
@@ -168,5 +168,5 @@
     emitter_link_name="${emitter_link_name}" sensor_0_range="0.01" sensor_0_fov="${ir_omni_fov_rad}"
     sensor_1_range="0.5" sensor_1_fov="${ir_front_facing_fov_rad}" >
-    <origin xyz="0.153 0 0.035"/>
+    <origin xyz="0.153 0 ${0.035 + base_link_z_offset}"/>
   </xacro:ir_opcode_receivers>
   <!-- Ground truth pose -->

Commit message: Use joint_state_publisher for both ignition and classic Cleaned up gazebo launch arg Adjusted front caster position

File: irobot_create_description/urdf/create3.urdf.xacro (robot description, xacro)
@@ -26,5 +26,5 @@
   <xacro:property name="distance_between_wheels" value="${23.3*cm2m}" />
   <xacro:property name="caster_position_x"       value="${12.5*cm2m}" />
-  <xacro:property name="caster_position_z"       value="${-5.25*cm2m}" />
+  <xacro:property name="caster_position_z"       value="${-5.2*cm2m}" />
   <xacro:property name="wheel_drop_offset_z"     value="${3.5*mm2m}"/>
   <xacro:property name="wheel_drop_z"            value="${wheel_height + wheel_drop_offset_z}"/>
@@ -222,12 +222,4 @@
     </gazebo>
     <gazebo>
-      <plugin filename="libignition-gazebo-joint-state-publisher-system.so" name="ignition::gazebo::systems::JointStatePublisher">
-        <joint_name>wheel_drop_left_joint</joint_name>
-        <joint_name>wheel_drop_right_joint</joint_name>
-        <joint_name>left_wheel_joint</joint_name>
-        <joint_name>right_wheel_joint</joint_name>
-      </plugin>
-    </gazebo>
-    <gazebo>
       <plugin filename="ignition-gazebo-diff-drive-system" name="ignition::gazebo::systems::DiffDrive">
         <left_joint>left_wheel_joint</left_joint>

File: irobot_create_description/urdf/dock/ir_emitter.urdf.xacro (robot description, xacro)
@@ -7,5 +7,5 @@
                                          update_rate:=1.0
                                          min_range:=${7*cm2m}
-                                         visualize:=true" >
+                                         visualize:=false" >
     <!-- Physical link properties -->
     <xacro:property name="mass" value="0.15" />
