Commit message: Simplify IR emitter Xacro

File: irobot_create_description/urdf/dock/ir_emitter.urdf.xacro (robot description, xacro)
@@ -1,7 +1,9 @@
 <?xml version="1.0"?>
 <robot xmlns:xacro="http://ros.org/wiki/xacro">
-  <xacro:macro name="ir_emitter" params="name updateRate broadcastRate parent *origin
-                                         ros_topic device_type code aperture
-                                         min_range:=0.50 range visualize" >
+  <xacro:macro name="ir_emitter" params="name parent:=base_link *origin
+                                         range code aperture
+                                         update_rate:=20 broadcast_rate:=64
+                                         ros_topic:=ir_emitter min_range:=0.50
+                                         visualize:=false" >
     <!-- Physical link properties -->
     <xacro:property name="mass" value="0.15" />
@@ -9,10 +11,10 @@
     <xacro:property name="y"    value="0.02" />
     <xacro:property name="z"    value="0.008" />
-    <joint name="sensor_emitter_${name}_joint" type="fixed">
+    <joint name="${name}_joint" type="fixed">
       <xacro:insert_block name="origin" />
       <parent link="${parent}"/>
-      <child link="sensor_emitter_${name}_link"/>
+      <child link="${name}_link"/>
     </joint>
-    <link name="sensor_emitter_${name}_link">
+    <link name="${name}_link">
       <xacro:if value="${visualize}">
         <visual>
@@ -24,9 +26,9 @@
       <xacro:inertial_cuboid mass="${mass}" x="${x}" y="${y}" z="${z}" />
     </link>
-    <gazebo reference="sensor_emitter_${name}_link">
+    <gazebo reference="${name}_link">
       <preserveFixedJoint>true</preserveFixedJoint>
       <sensor type="ray" name="${name}">
         <always_on>true</always_on>
-        <update_rate>10</update_rate>
+        <update_rate>${update_rate}</update_rate>
         <visualize>${visualize}</visualize>
         <ray>
@@ -51,14 +53,14 @@
     <gazebo>
       <static>true</static>
-      <!-- <plugin name="${name}_sensor_emitter" filename="libgazebo_ros_irobot_sensor_emitter.so">
-        <link>sensor_emitter_${name}_link</link>
+      <!-- MOVE TO SENSOR PLUGIN -->
+      <!-- <plugin name="${name}_ir_emitter" filename="libgazebo_ros_irobot_ir_emitter.so">
+        <link>${name}_link</link>
         <topicName>${ros_topic}</topicName>
         <emitterName>${name}</emitterName>
-        <emitterType>${device_type}</emitterType>
         <emitterCode>${code}</emitterCode>
         <rayAperture>${aperture}</rayAperture>
         <rayRange>${range}</rayRange>
-        <updateRate>${updateRate}</updateRate>
-        <broadcastRate>${broadcastRate}</broadcastRate>
+        <updateRate>${update_rate}</updateRate>
+        <broadcastRate>${broadcast_rate}</broadcastRate>
       </plugin> -->
     </gazebo>

File: irobot_create_description/urdf/dock/standard.urdf.xacro (robot description, xacro)
@@ -3,5 +3,5 @@
   <xacro:include filename="$(find irobot_create_description)/urdf/common_properties.urdf.xacro"/>
   <xacro:include filename="$(find irobot_create_description)/urdf/dock/ir_emitter.urdf.xacro"/>
-  <xacro:property name="z_offset_mm"   value="4.6"/>
+  <xacro:property name="z_offset_mm" value="4.6"/>
   <link name="base_link">
     <visual>
@@ -45,13 +45,7 @@
   <!-- Green IR emitter -->
   <xacro:ir_emitter name="${green_buoy_name}"
-                    updateRate="20"
-                    broadcastRate="64"
-                    parent="base_link"
-                    ros_topic="ir_emitter"
                     code="164"
                     aperture="${buoy_lateral_aperture}"
-                    range="1.524"
-                    device_type="dock"
-                    visualize="$(arg visual_debug)">
+                    range="1.524">
     <origin xyz="${buoy_x} ${- buoy_y} ${buoy_z}"
             rpy="0 0 ${- buoy_lateral_angle_yaw}"/>
@@ -59,13 +53,7 @@
   <!-- Red IR emitter -->
   <xacro:ir_emitter name="${red_buoy_name}"
-                    updateRate="20"
-                    broadcastRate="64"
-                    parent="base_link"
-                    ros_topic="ir_emitter"
                     code="168"
                     aperture="${buoy_lateral_aperture}"
-                    range="1.524"
-                    device_type="dock"
-                    visualize="$(arg visual_debug)">
+                    range="1.524">
     <origin xyz="${buoy_x} ${buoy_y} ${buoy_z}"
             rpy="0 0 ${buoy_lateral_angle_yaw}"/>
@@ -73,26 +61,14 @@
   <!-- Yellow IR emitter -->
   <xacro:ir_emitter name="${yellow_buoy_name}"
-                    updateRate="20"
-                    broadcastRate="64"
-                    parent="base_link"
-                    ros_topic="ir_emitter"
                     code="172"
                     aperture="${buoy_central_aperture}"
-                    range="1.2192"
-                    device_type="dock"
-                    visualize="$(arg visual_debug)">
+                    range="1.2192">
     <origin xyz="${buoy_x} 0 ${buoy_z}"/>
   </xacro:ir_emitter>
   <!-- Halo IR emitter -->
   <xacro:ir_emitter name="${halo_name}"
-                    updateRate="20"
-                    broadcastRate="64"
-                    parent="base_link"
-                    ros_topic="ir_emitter"
                     code="161"
                     aperture="360"
-                    range="0.6096"
-                    device_type="dock"
-                    visualize="$(arg visual_debug)">
+                    range="0.6096">
     <origin xyz="${halo_x} 0 ${halo_z}"/>
   </xacro:ir_emitter>
