Commit message: Use primitive instead of mesh for dock's collision model

File: irobot_create_description/urdf/dock/standard.urdf.xacro (robot description, xacro)
@@ -12,12 +12,10 @@
     </visual>
     <collision>
-      <origin xyz="0 0 ${z_offset_mm*mm2m}"/>
+      <!-- Using a simple box as collision model -->
+      <origin xyz="-0.045 0 0.05"/>
       <geometry>
-        <mesh filename="file://$(find irobot_create_description)/meshes/dock/collision.stl"/>
+        <box size="0.04 0.13 0.1"/>
       </geometry>
     </collision>
-    <xacro:inertial_cuboid_with_pose mass="2.5" x="0.15" y="0.13" z="0.19">
-      <origin xyz="-0.073 0 0"/>
-    </xacro:inertial_cuboid_with_pose>
   </link>
   <gazebo reference="base_link">
@@ -26,7 +24,4 @@
     <kp>1000000.0</kp>
     <kd>1.0</kd>
-  </gazebo>
-  <gazebo>
-    <static>true</static>
   </gazebo>
   <!-- Parameters for IR emitters -->

Commit message: Adds Dock and TF visualization

File: irobot_create_description/urdf/dock/standard.urdf.xacro (robot description, xacro)
@@ -4,5 +4,5 @@
   <xacro:include filename="$(find irobot_create_description)/urdf/dock/ir_emitter.urdf.xacro"/>
   <xacro:property name="z_offset_mm" value="4.6"/>
-  <link name="base_link">
+  <link name="std_dock_link">
     <visual>
       <origin xyz="0 0 ${z_offset_mm*mm2m}"/>
@@ -19,5 +19,5 @@
     </collision>
   </link>
-  <gazebo reference="base_link">
+  <gazebo reference="std_dock_link">
     <mu1>1.0</mu1>
     <mu2>1.0</mu2>
@@ -37,4 +37,5 @@
   <!-- Green IR emitter -->
   <xacro:ir_emitter name="${green_buoy_name}"
+                    parent="std_dock_link"
                     code="164"
                     aperture="${buoy_lateral_aperture}"
@@ -45,4 +46,5 @@
   <!-- Red IR emitter -->
   <xacro:ir_emitter name="${red_buoy_name}"
+                    parent="std_dock_link"
                     code="168"
                     aperture="${buoy_lateral_aperture}"
@@ -53,4 +55,5 @@
   <!-- Yellow IR emitter -->
   <xacro:ir_emitter name="${yellow_buoy_name}"
+                    parent="std_dock_link"
                     code="172"
                     aperture="${10*deg2rad}"
@@ -60,4 +63,5 @@
   <!-- Halo IR emitter -->
   <xacro:ir_emitter name="${halo_name}"
+                    parent="std_dock_link"
                     code="161"
                     aperture="360"

Commit message: link_name property for std dock link

File: irobot_create_description/urdf/dock/standard.urdf.xacro (robot description, xacro)
@@ -4,5 +4,6 @@
   <xacro:include filename="$(find irobot_create_description)/urdf/dock/ir_emitter.urdf.xacro"/>
   <xacro:property name="z_offset_mm" value="4.6"/>
-  <link name="std_dock_link">
+  <xacro:property name="link_name" value="std_dock_link"/>
+  <link name="${link_name}">
     <visual>
       <origin xyz="0 0 ${z_offset_mm*mm2m}"/>
@@ -19,5 +20,5 @@
     </collision>
   </link>
-  <gazebo reference="std_dock_link">
+  <gazebo reference="${link_name}">
     <mu1>1.0</mu1>
     <mu2>1.0</mu2>
@@ -37,5 +38,5 @@
   <!-- Green IR emitter -->
   <xacro:ir_emitter name="${green_buoy_name}"
-                    parent="std_dock_link"
+                    parent="${link_name}"
                     code="164"
                     aperture="${buoy_lateral_aperture}"
@@ -46,5 +47,5 @@
   <!-- Red IR emitter -->
   <xacro:ir_emitter name="${red_buoy_name}"
-                    parent="std_dock_link"
+                    parent="${link_name}"
                     code="168"
                     aperture="${buoy_lateral_aperture}"
@@ -55,5 +56,5 @@
   <!-- Yellow IR emitter -->
   <xacro:ir_emitter name="${yellow_buoy_name}"
-                    parent="std_dock_link"
+                    parent="${link_name}"
                     code="172"
                     aperture="${10*deg2rad}"
@@ -63,5 +64,5 @@
   <!-- Halo IR emitter -->
   <xacro:ir_emitter name="${halo_name}"
-                    parent="std_dock_link"
+                    parent="${link_name}"
                     code="161"
                     aperture="360"
