Commit message: r and l to radius and length

File: irobot_create_description/urdf/sensors/optical_mouse.urdf.xacro (robot description, xacro)
@@ -5,6 +5,6 @@
     <!-- Sensor settings -->
     <xacro:property name="mass" value="0.1" />
-    <xacro:property name="l" value="0.008" /> <!-- Length -->
-    <xacro:property name="r" value="0.01" /> <!-- Radius -->
+    <xacro:property name="length" value="0.008" /> <!-- Length -->
+    <xacro:property name="radius" value="0.01" /> <!-- Radius -->
     <!-- Visualization settings -->
     <xacro:property name="color" value="Red" />
@@ -20,9 +20,9 @@
         <visual>
           <geometry>
-            <cylinder length="${l}" radius="${r}" />
+            <cylinder length="${length}" radius="${radius}" />
           </geometry>
         </visual>
       </xacro:if>
-      <xacro:inertial_cylinder mass="${mass}" length="${l}" radius="${r}" />
+      <xacro:inertial_cylinder mass="${mass}" length="${length}" radius="${radius}" />
     </link>
     <gazebo>

Commit message: renames link

File: irobot_create_description/urdf/sensors/optical_mouse.urdf.xacro (robot description, xacro)
@@ -17,5 +17,5 @@
           </ros>
         <update_rate>${update_rate}</update_rate>
-        <link>${name}</link>
+        <link_name>${name}</link_name>
       </plugin>
     </gazebo>
