Commit message: Update irobot_create_description/urdf/sensors/cliff_sensor.urdf.xacro
Co-authored-by: Emiliano Borghi <creativa_eborghi@irobot.com>

File: irobot_create_description/urdf/sensors/cliff_sensor.urdf.xacro (robot description, xacro)
@@ -5,9 +5,9 @@
   <!-- Sensor settings -->
   <xacro:property name="update_rate" value="62"/>
-  <xacro:property name="fov_deg" value="5"/>
-  <xacro:property name="fov_rad" value="${fov_deg*deg2rad}"/>
-  <xacro:property name="min_range" value="${0*cm2m}"/>
-  <xacro:property name="max_range" value="${15*cm2m}"/>
-  <xacro:property name="samples" value="${fov_deg/5}"/>
+  <xacro:property name="fov_deg"     value="5"/>
+  <xacro:property name="fov_rad"     value="${fov_deg*deg2rad}"/>
+  <xacro:property name="min_range"   value="${0*cm2m}"/>
+  <xacro:property name="max_range"   value="${15*cm2m}"/>
+  <xacro:property name="samples"     value="${fov_deg/5}"/>
   <xacro:property name="sensor_name" value="cliff_${name}"/>
   <joint name="${sensor_name}_joint" type="fixed">

Commit message: Address Alexis comments

File: irobot_create_description/urdf/sensors/cliff_sensor.urdf.xacro (robot description, xacro)
@@ -4,11 +4,12 @@
                                          visualize:=false *origin">
   <!-- Sensor settings -->
-  <xacro:property name="update_rate" value="62"/>
-  <xacro:property name="fov_deg"     value="5"/>
-  <xacro:property name="fov_rad"     value="${fov_deg*deg2rad}"/>
-  <xacro:property name="min_range"   value="${0*cm2m}"/>
-  <xacro:property name="max_range"   value="${15*cm2m}"/>
-  <xacro:property name="samples"     value="${fov_deg/5}"/>
-  <xacro:property name="sensor_name" value="cliff_${name}"/>
+  <xacro:property name="update_rate"         value="62"/>
+  <xacro:property name="fov_deg"             value="5"/>
+  <xacro:property name="fov_rad"             value="${fov_deg*deg2rad}"/>
+  <xacro:property name="min_range"           value="${0*cm2m}"/>
+  <xacro:property name="max_range"           value="${15*cm2m}"/>
+  <xacro:property name="samples"             value="${fov_deg/5}"/>
+  <xacro:property name="sensor_name"         value="cliff_${name}"/>
+  <xacro:property name="detection_threshold" value="${8*cm2m}"/>
   <joint name="${sensor_name}_joint" type="fixed">
     <xacro:insert_block name="origin"/>
@@ -50,5 +51,5 @@
           <remapping>~/out:=${sensor_name}/event</remapping>
         </ros>
-        <detection_threshold>${8*cm2m}</detection_threshold>
+        <detection_threshold>${detection_threshold}</detection_threshold>
       </plugin>
     </sensor>

Commit message: Changes the min range of the cliff sensors.

File: irobot_create_description/urdf/sensors/cliff_sensor.urdf.xacro (robot description, xacro)
@@ -7,5 +7,5 @@
   <xacro:property name="fov_deg"             value="5"/>
   <xacro:property name="fov_rad"             value="${fov_deg*deg2rad}"/>
-  <xacro:property name="min_range"           value="${0*cm2m}"/>
+  <xacro:property name="min_range"           value="${0.01*cm2m}"/>
   <xacro:property name="max_range"           value="${15*cm2m}"/>
   <xacro:property name="samples"             value="${fov_deg/5}"/>
