Commit message: - Reorganized packages - Shifted center of gravity of create3 forwards by 22.8 mm - Added min/max velocity and acceleration to diff drive plugin

File: irobot_create_common/irobot_create_description/urdf/create3.urdf.xacro (robot description, xacro)
@@ -16,4 +16,5 @@
   <xacro:property name="body_z_offset"           value="${-2.5*cm2m}" />
   <xacro:property name="body_collision_z_offset" value="${1*cm2m}" />
+  <xacro:property name="body_cog_x_offset"       value="${2.28*cm2m}" />
   <xacro:property name="body_mass"               value="2.300" />
   <xacro:property name="body_radius"             value="${16.4*cm2m}" />
@@ -26,5 +27,10 @@
   <xacro:property name="distance_between_wheels" value="${23.3*cm2m}" />
   <xacro:property name="caster_position_x"       value="${12.5*cm2m}" />
-  <xacro:property name="caster_position_z"       value="${-5.2*cm2m}" />
+  <xacro:if value="${'$(arg gazebo)' == 'ignition'}">
+    <xacro:property name="caster_position_z"       value="${-5.03*cm2m}" />
+  </xacro:if>
+  <xacro:if value="${'$(arg gazebo)' == 'classic'}">
+    <xacro:property name="caster_position_z"       value="${-5.2*cm2m}" />
+  </xacro:if>
   <xacro:property name="wheel_drop_offset_z"     value="${3.5*mm2m}"/>
   <xacro:property name="wheel_drop_z"            value="${wheel_height + wheel_drop_offset_z}"/>
@@ -50,5 +56,5 @@
     </collision>
     <xacro:inertial_cylinder_with_pose mass="${body_mass}" radius="${body_radius}" length="${body_length}">
-      <origin xyz="0 0 ${body_collision_z_offset + base_link_z_offset}"/>
+      <origin xyz="${body_cog_x_offset} 0 ${body_collision_z_offset + base_link_z_offset}"/>
     </xacro:inertial_cylinder_with_pose>
   </link>
@@ -230,6 +236,12 @@
         <child_frame_id>base_link</child_frame_id>
         <odom_publish_frequency>50</odom_publish_frequency>
-        <min_acceleration>-1</min_acceleration>
-        <max_acceleration>1</max_acceleration>
+        <min_linear_velocity>-0.46</min_linear_velocity>
+        <max_linear_velocity>0.46</max_linear_velocity>
+        <min_linear_acceleration>-0.9</min_linear_acceleration>
+        <max_linear_acceleration>0.9</max_linear_acceleration>
+        <min_angular_velocity>-1.9</min_angular_velocity>
+        <max_angular_velocity>1.9</max_angular_velocity>
+        <min_angular_acceleration>-7.725</min_angular_acceleration>
+        <max_angular_acceleration>7.725</max_angular_acceleration>
       </plugin>
     </gazebo>

Commit message: Renamed dock to standard_dock Center of gravity offset only applied in ignition for now

File: irobot_create_common/irobot_create_description/urdf/create3.urdf.xacro (robot description, xacro)
@@ -16,8 +16,13 @@
   <xacro:property name="body_z_offset"           value="${-2.5*cm2m}" />
   <xacro:property name="body_collision_z_offset" value="${1*cm2m}" />
-  <xacro:property name="body_cog_x_offset"       value="${2.28*cm2m}" />
   <xacro:property name="body_mass"               value="2.300" />
   <xacro:property name="body_radius"             value="${16.4*cm2m}" />
   <xacro:property name="body_length"             value="${6*cm2m}" />
+  <xacro:if value="${'$(arg gazebo)' == 'ignition'}">
+    <xacro:property name="body_cog_x_offset"       value="${2.28*cm2m}" />
+  </xacro:if>
+  <xacro:if value="${'$(arg gazebo)' == 'classic'}">
+    <xacro:property name="body_cog_x_offset"       value="${0*cm2m}" />
+  </xacro:if>
   <xacro:property name="bumper_mass"             value="0.1" />
   <xacro:property name="bumper_offset_z"         value="${-2.5*cm2m}" />
