Commit message: Multi robot support (#207)
* Working multi robot sim

* Use wildcards for param files
Added robot name to Create 3 buttons

* Dock model is now called <robot_name>/standard_dock
Namespaced dock frame id in pose republisher

* Added namespacing support to Rviz config
Rviz now launches for each robot spawn
Added static transform for prefixed odom and base_link frames
Added offset launch module in irobot_create_common_bringup
Fixed spawning robots with different x, y, and yaw positions

* Linter fixes

* Added namespace launch arg. Defaults to 'robot_name' in create3_spawn
create3_ignition defaults to spawning 'create3' robot without namespace

* Frame id fixes

* Changed robot name to be <namespace>/create3, rather than using a robot_name arg
Changed dock name to be <namespace>/standard_dock
Remove robot_name arg, use just namespace for everything

* Fixed bumper
Use ogre2 as sensor render engine
Reduce max_step_size to 3ms

* Linter fixes

* Fixed import order

* Multi robot support for gazebo classic

* Updated README

* Fixed import order

File: irobot_create_common/irobot_create_description/urdf/bumper.urdf.xacro (robot description, xacro)
@@ -13,5 +13,5 @@
   <link name="${link_name}"/>
 </xacro:macro>
-<xacro:macro name="bumper" params="name:=bumper parent_link:=base_link update_rate:=62.0 gazebo visual_mesh collision_mesh
+<xacro:macro name="bumper" params="name:=bumper namespace parent_link:=base_link update_rate:=62.0 gazebo visual_mesh collision_mesh
   *origin *inertial">
   <xacro:property name="link_name" value="${name}"/>
@@ -47,9 +47,17 @@
       <contact>
         <collision>${link_name}_collision</collision>
+        <xacro:if value="${gazebo == 'ignition'}">
+          <xacro:if value="${namespace == ''}">
+            <topic>/bumper_contact</topic>
+          </xacro:if>
+          <xacro:if value="${namespace != ''}">
+            <topic>${namespace}/bumper_contact</topic>
+          </xacro:if>
+        </xacro:if>
       </contact>
       <xacro:if value="${gazebo == 'classic'}">
         <plugin name="${name}_plugin" filename="libgazebo_ros_create_bumper.so">
           <ros>
-            <namespace>/</namespace>
+            <namespace>${namespace}</namespace>
             <remapping>~/out:=_internal/bumper/event</remapping>
           </ros>

File: irobot_create_common/irobot_create_description/urdf/create3.urdf.xacro (robot description, xacro)
@@ -13,4 +13,6 @@
   <!-- Gazebo version -->
   <xacro:arg name="gazebo"                       default="classic" />
+  <!-- Namespace -->
+  <xacro:arg name="namespace"                    default=""/>
   <!-- Mechanical properties -->
   <xacro:property name="body_z_offset"           value="${-2.5*cm2m}" />
@@ -73,4 +75,5 @@
   <xacro:bumper
       gazebo="$(arg gazebo)"
+      namespace="$(arg namespace)"
       visual_mesh="package://irobot_create_description/meshes/bumper_visual.dae"
       collision_mesh="package://irobot_create_description/meshes/bumper_collision.dae">
@@ -84,8 +87,8 @@
   </xacro:bumper>
   <!-- Wheels with mechanical wheel drop -->
-  <xacro:wheel_with_wheeldrop name="left" gazebo="$(arg gazebo)">
+  <xacro:wheel_with_wheeldrop name="left" gazebo="$(arg gazebo)" namespace="$(arg namespace)">
     <origin xyz="0 ${distance_between_wheels/2} ${wheel_drop_z  + base_link_z_offset}" rpy="${-pi/2} 0 0"/>
   </xacro:wheel_with_wheeldrop>
-  <xacro:wheel_with_wheeldrop name="right" gazebo="$(arg gazebo)">
+  <xacro:wheel_with_wheeldrop name="right" gazebo="$(arg gazebo)" namespace="$(arg namespace)">
     <origin xyz="0 ${-distance_between_wheels/2} ${wheel_drop_z  + base_link_z_offset}" rpy="${-pi/2} 0 0"/>
   </xacro:wheel_with_wheeldrop>
@@ -95,5 +98,5 @@
   </xacro:caster>
   <!-- IMU -->
-  <xacro:imu_sensor gazebo="$(arg gazebo)">
+  <xacro:imu_sensor gazebo="$(arg gazebo)" namespace="$(arg namespace)">
     <origin xyz="0.050613 0.043673 ${0.0202 + base_link_z_offset}"/>
   </xacro:imu_sensor>
@@ -101,7 +104,11 @@
     <gazebo>
       <plugin name="gazebo_ros2_control" filename="libgazebo_ros2_control.so">
-        <parameters> $(find irobot_create_control)/config/control.yaml </parameters>
+        <parameters>$(find irobot_create_control)/config/control.yaml</parameters>
         <ros>
           <remapping>~/odom:=odom</remapping>
+          <remapping>/tf:=tf</remapping>
+          <remapping>/tf_static:=tf_static</remapping>
+          <remapping>/diagnostics:=diagnostics</remapping>
+          <namespace>$(arg namespace)</namespace>
         </ros>
       </plugin>
@@ -111,7 +118,11 @@
     <gazebo>
       <plugin filename="libign_ros2_control-system.so" name="ign_ros2_control::IgnitionROS2ControlPlugin">
-        <parameters> $(find irobot_create_control)/config/control.yaml </parameters>
+        <parameters>$(find irobot_create_control)/config/control.yaml</parameters>
         <ros>
           <remapping>~/odom:=odom</remapping>
+          <remapping>/tf:=tf</remapping>
+          <remapping>/tf_static:=tf_static</remapping>
+          <remapping>/diagnostics:=diagnostics</remapping>
+          <namespace>$(arg namespace)</namespace>
         </ros>
       </plugin>
@@ -119,5 +130,5 @@
   </xacro:if>
   <!-- Mouse -->
-  <xacro:optical_mouse gazebo="$(arg gazebo)">
+  <xacro:optical_mouse gazebo="$(arg gazebo)" namespace="$(arg namespace)">
     <origin xyz="0.1015 0.087 ${-0.055 + base_link_z_offset}" rpy="0 0 ${-pi/4}"/>
   </xacro:optical_mouse>
@@ -132,17 +143,17 @@
   <xacro:property name="cliff_back_pitch" value="${80*deg2rad}"/>
   <xacro:property name="cliff_back_yaw" value="${167.4*deg2rad}"/>
-  <xacro:cliff_sensor name="side_left" gazebo="$(arg gazebo)" visualize="$(arg visualize_rays)">
+  <xacro:cliff_sensor name="side_left" gazebo="$(arg gazebo)" visualize="$(arg visualize_rays)" namespace="$(arg namespace)">
     <origin xyz="${cliff_back_x} ${cliff_back_y} ${cliff_z + base_link_z_offset}"
             rpy="0 ${cliff_back_pitch} ${cliff_back_yaw}"/>
   </xacro:cliff_sensor>
-  <xacro:cliff_sensor name="side_right" gazebo="$(arg gazebo)" visualize="$(arg visualize_rays)">
+  <xacro:cliff_sensor name="side_right" gazebo="$(arg gazebo)" visualize="$(arg visualize_rays)" namespace="$(arg namespace)">
     <origin xyz="${cliff_back_x} ${- cliff_back_y} ${cliff_z + base_link_z_offset}"
             rpy="0 ${cliff_back_pitch} ${- cliff_back_yaw}"/>
   </xacro:cliff_sensor>
-  <xacro:cliff_sensor name="front_left" gazebo="$(arg gazebo)" visualize="$(arg visualize_rays)">
+  <xacro:cliff_sensor name="front_left" gazebo="$(arg gazebo)" visualize="$(arg visualize_rays)" namespace="$(arg namespace)">
     <origin xyz="${cliff_center_x} ${cliff_center_y} ${cliff_z + base_link_z_offset}"
             rpy="0 ${cliff_center_pitch} ${cliff_center_yaw}"/>
   </xacro:cliff_sensor>
-  <xacro:cliff_sensor name="front_right" gazebo="$(arg gazebo)" visualize="$(arg visualize_rays)">
+  <xacro:cliff_sensor name="front_right" gazebo="$(arg gazebo)" visualize="$(arg visualize_rays)" namespace="$(arg namespace)">
     <origin xyz="${cliff_center_x} ${- cliff_center_y} ${cliff_z + base_link_z_offset}"
             rpy="0 ${cliff_center_pitch} ${- cliff_center_yaw}"/>
@@ -163,23 +174,23 @@
   side_left                                                   right
   -->
-  <xacro:ir_intensity name="front_center_left" gazebo="$(arg gazebo)">
+  <xacro:ir_intensity name="front_center_left" gazebo="$(arg gazebo)" namespace="$(arg namespace)">
     <origin xyz="0.1540 0 ${ir_intensity_z_pos + base_link_z_offset}"/>
   </xacro:ir_intensity>
-  <xacro:ir_intensity name="front_center_right" gazebo="$(arg gazebo)">
+  <xacro:ir_intensity name="front_center_right" gazebo="$(arg gazebo)" namespace="$(arg namespace)">
     <origin xyz="0.1396 -0.0651 ${ir_intensity_z_pos + base_link_z_offset}" rpy="0 0 -0.436"/>
   </xacro:ir_intensity>
-  <xacro:ir_intensity name="front_left" gazebo="$(arg gazebo)">
+  <xacro:ir_intensity name="front_left" gazebo="$(arg gazebo)" namespace="$(arg namespace)">
     <origin xyz="0.1396 0.0651 ${ir_intensity_z_pos + base_link_z_offset}" rpy="0 0 0.436"/>
   </xacro:ir_intensity>
-  <xacro:ir_intensity name="front_right" gazebo="$(arg gazebo)">
+  <xacro:ir_intensity name="front_right" gazebo="$(arg gazebo)" namespace="$(arg namespace)">
     <origin xyz="0.0990 -0.1180 ${ir_intensity_z_pos + base_link_z_offset}" rpy="0 0 -0.873"/>
   </xacro:ir_intensity>
-  <xacro:ir_intensity name="left" gazebo="$(arg gazebo)">
+  <xacro:ir_intensity name="left" gazebo="$(arg gazebo)" namespace="$(arg namespace)">
     <origin xyz="0.0990 0.1180 ${ir_intensity_z_pos + base_link_z_offset}" rpy="0 0 0.873"/>
   </xacro:ir_intensity>
-  <xacro:ir_intensity name="right" gazebo="$(arg gazebo)">
+  <xacro:ir_intensity name="right" gazebo="$(arg gazebo)" namespace="$(arg namespace)">
     <origin xyz="0.0399 -0.1488 ${ir_intensity_z_pos + base_link_z_offset}" rpy="0 0 -1.309"/>
   </xacro:ir_intensity>
-  <xacro:ir_intensity name="side_left" gazebo="$(arg gazebo)">
+  <xacro:ir_intensity name="side_left" gazebo="$(arg gazebo)" namespace="$(arg namespace)">
     <origin xyz="0.0399 0.1488 ${ir_intensity_z_pos + base_link_z_offset}" rpy="0 0 1.309"/>
   </xacro:ir_intensity>
@@ -200,5 +211,6 @@
   <xacro:property name="ir_omni_fov_rad" value="${220.0*deg2rad}"/>
   <xacro:property name="ir_front_facing_fov_rad" value="${pi/2}"/>
-  <xacro:ir_opcode_receivers gazebo="$(arg gazebo)" robot_model_name="${robot_model_name}" dock_model_name="${dock_model_name}"
+  <xacro:ir_opcode_receivers gazebo="$(arg gazebo)" namespace="$(arg namespace)"
+    robot_model_name="${robot_model_name}" dock_model_name="${dock_model_name}"
     emitter_link_name="${emitter_link_name}" sensor_0_range="0.01" sensor_0_fov="${ir_omni_fov_rad}"
     sensor_1_range="0.5" sensor_1_fov="${ir_front_facing_fov_rad}" >
@@ -211,5 +223,5 @@
       <plugin name="gazebo_ros_p3d_robot" filename="libgazebo_ros_p3d.so">
         <ros>
-          <namespace>/</namespace>
+          <namespace>$(arg namespace)</namespace>
           <remapping>odom:=sim_ground_truth_pose</remapping>
         </ros>
@@ -226,5 +238,5 @@
       <plugin name="dock_status_publisher" filename="libgazebo_ros_create_docking_status.so">
         <ros>
-          <namespace>/</namespace>
+          <namespace>$(arg namespace)</namespace>
           <remapping>~/out:=dock_status</remapping>
         </ros>
